File: CSeventeen.kicad_pcb (KiCad board)
At the start: 2 copper layers, 320 x 135 mm, 98 parts, among them CN2 KEYBOARD_HEADER, CN9 LED_CONNECTOR, Q1 2SC1815, Q2 2SC1815, Q3 2SC1815, Q5 2SD880, U1 MOS_7360_TED, U10 NE555, U11 74LS125, U12 74LS02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

Commit message: Add diodes
Parts:
- added D11: 1N914, Diode_THT:D_DO-41_SOD81_P5.08mm_Vertical_KathodeUp, F.Cu at (316.2, 124.2)
- added D12: 6.8V, Diode_THT:D_DO-35_SOD27_P5.08mm_Vertical_KathodeUp, F.Cu at (316.7, 147.3)
- D1, D10, D2, D3, D4, D5, D6, D7, D8, D9: footprint Diode_THT:D_DO-35_SOD27_P7.62mm_Horizontal -> Diode_THT:D_DO-35_SOD27_P5.08mm_Vertical_KathodeUp
- Q1, Q2, Q3: footprint Package_TO_SOT_THT:TO-92_Inline -> Package_TO_SOT_THT:TO-92_Inline_Wide
- Q5: footprint Package_TO_SOT_THT:TO-126-3_Vertical -> Package_TO_SOT_THT:TO-220-3_Horizontal_TabDown
- moved D2 358.8 mm to (337.0, 177.4), turned to 180 degrees
- moved D5 355.5 mm to (337.0, 167.3), turned to 180 degrees
- moved D4 353.5 mm to (337.0, 172.4), turned to 180 degrees
- moved D10 352.9 mm to (337.0, 142.0), turned to 180 degrees
- moved D3 347.3 mm to (337.0, 162.2), turned to 180 degrees
- moved D8 346.4 mm to (337.0, 136.9), turned to 180 degrees
- moved D7 345.8 mm to (337.0, 152.1), turned to 180 degrees
- moved D1 343.4 mm to (337.0, 157.2), turned to 180 degrees
- moved D6 336.0 mm to (337.0, 131.8), turned to 180 degrees
- moved D9 335.4 mm to (337.0, 147.0), turned to 180 degrees
- moved Q5 313.0 mm to (300.0, 163.3), turned to 270 degrees

Commit message: Fix board dimensions
Parts:
- moved C1 3.00 mm to (311.4, 127.5)
- moved C10 3.00 mm to (91.7, 140.1)
- moved C11 3.00 mm to (183.1, 100.7)
- moved C12 3.00 mm to (170.7, 177.5)
- moved C13 3.00 mm to (200.9, 187.7)
- moved C14 3.00 mm to (205.9, 193.0)
- moved C15 3.00 mm to (225.8, 182.8)
- moved C16 3.00 mm to (63.3, 103.1)
- moved C17 3.00 mm to (72.9, 103.1)
- moved C18 3.00 mm to (150.9, 96.1)
- moved C19 3.00 mm to (158.7, 96.1)
- moved C2 3.00 mm to (310.4, 137.9)
- moved C20 3.00 mm to (158.7, 108.7)
- moved C200 3.00 mm to (353.3, 89.1)
- moved C21 3.00 mm to (170.7, 172.9)
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Other:
- board size 320 x 135 mm -> 320 x 136.2 mm
