File: CSeventeen.kicad_pcb (KiCad board)
At the start: 2 copper layers, 320 x 136.2 mm, 100 parts, among them CN2 KEYBOARD_HEADER, CN9 LED_CONNECTOR, Q1 2SC1815, Q2 2SC1815, Q3 2SC1815, Q5 2SD880, U1 MOS_7360_TED, U10 NE555, U11 74LS125, U12 74LS02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

Commit message: Add crystal
Parts:
- added EM1: EMI_Filter_LCL, CSeventeen:EMI_Filter, F.Cu at (346.8, 185.1)
- added EM2: EMI_Filter_LCL, CSeventeen:EMI_Filter, F.Cu at (346.8, 152.7)
- added EM3: EMI_Filter_LCL, CSeventeen:EMI_Filter, F.Cu at (163.8, 92.8)
- added EM4: EMI_Filter_LCL, CSeventeen:EMI_Filter, F.Cu at (173.4, 90.3)
- added EM5: EMI_Filter_LCL, CSeventeen:EMI_Filter, F.Cu at (168.6, 90.3)
- added FB1: Ferrite_Bead_Small, CSeventeen:Ferrite, F.Cu at (126.4, 91.7)
- added FB12: Ferrite_Bead_Small, CSeventeen:Ferrite, F.Cu at (183.1, 90.3)
- added FB13: Ferrite_Bead_Small, CSeventeen:Ferrite, F.Cu at (178.2, 90.3)
- added FB14: Ferrite_Bead_Small, CSeventeen:Ferrite, F.Cu at (102.2, 80.5)
- added FB15: Ferrite_Bead_Small, CSeventeen:Ferrite, F.Cu at (87.6, 80.5)
- added FB16: Ferrite_Bead_Small, CSeventeen:Ferrite, F.Cu at (97.3, 80.5)
- added FB17: Ferrite_Bead_Small, CSeventeen:Ferrite, F.Cu at (82.7, 80.5)
- added FB18: Ferrite_Bead_Small, CSeventeen:Ferrite, F.Cu at (92.4, 80.5)
- added FB19: Ferrite_Bead_Small, CSeventeen:Ferrite, F.Cu at (77.8, 80.5)
- added FB2: Ferrite_Bead_Small, CSeventeen:Ferrite, F.Cu at (136.0, 91.7)
- added FB22: Ferrite_Bead_Small, CSeventeen:Ferrite, F.Cu at (346.8, 189.2)
- added FB24: Ferrite_Bead_Small, CSeventeen:Ferrite, F.Cu at (346.8, 164.9)
- added FB25: Ferrite_Bead_Small, CSeventeen:Ferrite, F.Cu at (344.3, 193.2)
- added FB26: Ferrite_Bead_Small, CSeventeen:Ferrite, F.Cu at (346.8, 168.9)
- added FB27: Ferrite_Bead_Small, CSeventeen:Ferrite, F.Cu at (346.8, 177.0)
- added FB28: Ferrite_Bead_Small, CSeventeen:Ferrite, F.Cu at (346.8, 173.0)
- added FB29: Ferrite_Bead_Small, CSeventeen:Ferrite, F.Cu at (346.8, 181.1)
- added FB3: Ferrite_Bead_Small, CSeventeen:Ferrite, F.Cu at (145.5, 91.7)
- added FB30: Ferrite_Bead_Small, CSeventeen:Ferrite, F.Cu at (346.8, 156.8)
- added FB31: Ferrite_Bead_Small, CSeventeen:Ferrite, F.Cu at (346.8, 132.5)
- added FB32: Ferrite_Bead_Small, CSeventeen:Ferrite, F.Cu at (346.8, 160.8)
- added FB33: Ferrite_Bead_Small, CSeventeen:Ferrite, F.Cu at (346.8, 136.5)
- added FB34: Ferrite_Bead_Small, CSeventeen:Ferrite, F.Cu at (346.8, 144.6)
- added FB35: Ferrite_Bead_Small, CSeventeen:Ferrite, F.Cu at (346.8, 140.6)
- added FB37: Ferrite_Bead_Small, CSeventeen:Ferrite, F.Cu at (346.8, 148.7)
- added FB38: Ferrite_Bead_Small, CSeventeen:Ferrite, F.Cu at (251.8, 101.9)
- added FB39: Ferrite_Bead_Small, CSeventeen:Ferrite, F.Cu at (251.8, 106.8)
- added FB4: Ferrite_Bead_Small, CSeventeen:Ferrite, F.Cu at (140.7, 91.7)
- added FB40: Ferrite_Bead_Small, CSeventeen:Ferrite, F.Cu at (251.8, 118.0)
- added FB41: Ferrite_Bead_Small, CSeventeen:Ferrite, F.Cu at (321.6, 177.5)
- added FB42: Ferrite_Bead_Small, CSeventeen:Ferrite, F.Cu at (267.6, 177.5)
- added FB43: Ferrite_Bead_Small, CSeventeen:Ferrite, F.Cu at (287.2, 177.5)
- added FB44: Ferrite_Bead_Small, CSeventeen:Ferrite, F.Cu at (282.3, 177.5)
- added FB45: Ferrite_Bead_Small, CSeventeen:Ferrite, F.Cu at (292.2, 177.5)
- added FB46: Ferrite_Bead_Small, CSeventeen:Ferrite, F.Cu at (252.9, 177.5)
- added FB47: Ferrite_Bead_Small, CSeventeen:Ferrite, F.Cu at (306.9, 177.5)
- added FB48: Ferrite_Bead_Small, CSeventeen:Ferrite, F.Cu at (257.8, 177.5)
- added FB49: Ferrite_Bead_Small, CSeventeen:Ferrite, F.Cu at (316.7, 177.5)
- added FB5: Ferrite_Bead_Small, CSeventeen:Ferrite, F.Cu at (131.2, 91.7)
- added FB50: Ferrite_Bead_Small, CSeventeen:Ferrite, F.Cu at (302.0, 177.5)
- added FB51: Ferrite_Bead_Small, CSeventeen:Ferrite, F.Cu at (297.1, 177.5)
- added FB52: Ferrite_Bead_Small, CSeventeen:Ferrite, F.Cu at (311.8, 177.5)
- added FB53: Ferrite_Bead_Small, CSeventeen:Ferrite, F.Cu at (262.7, 177.5)
- added FB54: Ferrite_Bead_Small, CSeventeen:Ferrite, F.Cu at (272.5, 177.5)
- added FB55: Ferrite_Bead_Small, CSeventeen:Ferrite, F.Cu at (277.4, 177.5)
- added FB56: Ferrite_Bead_Small, CSeventeen:Ferrite, F.Cu at (248.0, 177.5)
- added FB58: Ferrite_Bead_Small, CSeventeen:Ferrite, F.Cu at (187.4, 90.3)
- added Y1: Crystal, Crystal:Crystal_HC49-U_Horizontal_1EP_style2, F.Cu at (194.7, 183.3)
- C18, C19: footprint Capacitor_THT:CP_Radial_D6.3mm_P2.50mm -> Capacitor_THT:CP_Radial_D5.0mm_P2.50mm
- moved Q1 4.50 mm to (205.9, 181.1)
- moved Q3 1.27 mm to (173.5, 104.9)
- moved R23 0.70 mm to (163.8, 103.6)
- moved RP1 0.50 mm to (126.4, 101.5)
- moved C18 0.40 mm to (151.3, 96.1)
- moved C19 0.14 mm to (158.9, 96.1)
- moved C20 0.13 mm to (158.9, 108.7)
- moved R9 0.06 mm to (154.5, 108.7)
Connections:
- C12 pad 1: (no net) -> Net-(C12-Pad1)
- CN2 pad 1: (no net) -> Net-(CN2-Pad1)
- CN2 pad 10: (no net) -> Net-(CN2-Pad10)
- CN2 pad 11: (no net) -> Net-(CN2-Pad11)
- CN2 pad 12: (no net) -> Net-(CN2-Pad12)
- CN2 pad 13: (no net) -> Net-(CN2-Pad13)
- CN2 pad 14: (no net) -> Net-(CN2-Pad14)
- CN2 pad 15: (no net) -> Net-(CN2-Pad15)
- CN2 pad 16: (no net) -> Net-(CN2-Pad16)
- CN2 pad 17: (no net) -> Net-(CN2-Pad17)
- CN2 pad 18: (no net) -> Net-(CN2-Pad18)
- CN2 pad 19: (no net) -> Net-(CN2-Pad19)
- CN2 pad 3: (no net) -> Net-(CN2-Pad3)
- CN2 pad 6: (no net) -> Net-(CN2-Pad6)
- CN2 pad 7: (no net) -> Net-(CN2-Pad7)
- CN2 pad 8: (no net) -> Net-(CN2-Pad8)
- CN2 pad 9: (no net) -> Net-(CN2-Pad9)
- D10 pad 1: (no net) -> Net-(D10-Pad1)
- D6 pad 1: (no net) -> Net-(D6-Pad1)
- D7 pad 1: (no net) -> Net-(D7-Pad1)
- D8 pad 1: (no net) -> Net-(D8-Pad1)
- D9 pad 1: (no net) -> Net-(D9-Pad1)
- Q5 pad 1: (no net) -> Net-(FB19-Pad2)
- U1 pad 19: (no net) -> k4
- U1 pad 20: (no net) -> k5
- U11 pad 3: (no net) -> Net-(EM1-Pad3)
- U11 pad 6: (no net) -> Net-(EM2-Pad3)
- U13 pad 2: (no net) -> Net-(FB41-Pad2)
- U13 pad 3: (no net) -> Net-(FB42-Pad2)
- U13 pad 4: (no net) -> Net-(FB43-Pad2)
- U13 pad 5: (no net) -> Net-(FB44-Pad2)
- U13 pad 6: (no net) -> Net-(FB45-Pad2)
- U13 pad 7: (no net) -> Net-(FB46-Pad2)
- U13 pad 8: (no net) -> Net-(FB47-Pad2)
- U13 pad 9: (no net) -> Net-(FB48-Pad2)

Commit message: Use 3d models from github.com/StormTrooper/Commodore-Plus4
Parts:
- added CN1: EXPANSION_CONNECTOR, CommodorePlus4:50Pin_Edge_Connector, F.Cu at (283.2, 97.8)
- added CN3: CASSETTE, CommodorePlus4:Connector_Mini-DIN_Female_7Pin_2rows, F.Cu at (93.1, 73.7)
- added CN4: JOY1, CommodorePlus4:Connector_Mini-DIN_Female_8Pin_2rows, F.Cu at (361.4, 165.4)
- added CN5: JOY2, CommodorePlus4:Connector_Mini-DIN_Female_8Pin_2rows, F.Cu at (361.4, 147.4)
- added CN6: AUDIO_VIDEO, CommodorePlus4:Connector_DIN_Female_8Pin_3rows, F.Cu at (173.6, 76.7)
- added CN7: SERIAL_BUS, CommodorePlus4:Connector_DIN_Female_6Pin_3rows, F.Cu at (143.3, 77.3)
- added M1: Modulator, CommodorePlus4:RF_Modulator, F.Cu at (232.0, 68.6)
- added SW1: POWER_SWITCH, CommodorePlus4:Switch-Rocker, F.Cu at (352.0, 98.6)
- added SW2: RESET_SW, CommodorePlus4:Switch-Pushbutton, F.Cu at (354.6, 126.6)
- moved FB41 5.05 mm to (321.6, 182.6), turned to 180 degrees
- moved FB42 5.05 mm to (267.6, 182.6), turned to 180 degrees
- moved FB43 5.05 mm to (287.2, 182.6), turned to 180 degrees
- moved FB44 5.05 mm to (282.3, 182.6), turned to 180 degrees
- moved FB45 5.05 mm to (292.2, 182.6), turned to 180 degrees
- moved FB46 5.05 mm to (252.9, 182.6), turned to 180 degrees
- moved FB47 5.05 mm to (306.9, 182.6), turned to 180 degrees
- moved FB48 5.05 mm to (257.8, 182.6), turned to 180 degrees
- moved FB49 5.05 mm to (316.7, 182.6), turned to 180 degrees
- moved FB50 5.05 mm to (302.0, 182.6), turned to 180 degrees
- moved FB51 5.05 mm to (297.1, 182.6), turned to 180 degrees
- moved FB52 5.05 mm to (311.8, 182.6), turned to 180 degrees
- moved FB53 5.05 mm to (262.7, 182.6), turned to 180 degrees
- moved FB54 5.05 mm to (272.5, 182.6), turned to 180 degrees
- moved FB55 5.05 mm to (277.4, 182.6), turned to 180 degrees
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Connections:
- C11 pad 1: (no net) -> Net-(C11-Pad1)
- EM1 pad 1: (no net) -> Net-(CN4-Pad8)
- EM2 pad 1: (no net) -> Net-(CN5-Pad8)
- EM3 pad 1: (no net) -> Net-(EM3-Pad1)
- EM3 pad 3: (no net) -> Net-(CN6-Pad1)
- EM4 pad 1: (no net) -> Net-(EM4-Pad1)
- EM4 pad 3: (no net) -> Net-(CN6-Pad6)
- EM5 pad 1: (no net) -> Net-(EM5-Pad1)
- EM5 pad 3: (no net) -> Net-(CN6-Pad4)
- FB1 pad 1: (no net) -> Net-(CN7-Pad2)
- FB12 pad 2: (no net) -> Net-(CN6-Pad3)
- FB13 pad 1: (no net) -> Net-(CN6-Pad2)
- FB14 pad 1: (no net) -> Net-(CN3-Pad2)
- FB15 pad 2: (no net) -> Net-(CN3-Pad1)
- FB16 pad 2: (no net) -> Net-(CN3-Pad4)
- FB17 pad 1: (no net) -> Net-(CN3-Pad5)
- FB18 pad 1: (no net) -> Net-(CN3-Pad6)
- FB19 pad 1: (no net) -> Net-(CN3-Pad3)
- FB2 pad 2: (no net) -> Net-(CN7-Pad6)
- FB22 pad 1: (no net) -> Net-(CN4-Pad5)
- FB24 pad 2: (no net) -> Net-(CN4-Pad1)
- FB25 pad 2: (no net) -> Net-(CN4-Pad2)
- FB26 pad 2: (no net) -> Net-(CN4-Pad3)
- FB27 pad 2: (no net) -> Net-(CN4-Pad4)
- FB28 pad 2: (no net) -> Net-(CN4-Pad6)
- FB29 pad 1: (no net) -> Net-(CN4-Pad7)
- FB3 pad 1: (no net) -> Net-(CN7-Pad5)
- FB30 pad 1: (no net) -> Net-(CN5-Pad5)
- FB31 pad 2: (no net) -> Net-(CN5-Pad1)
- FB32 pad 2: (no net) -> Net-(CN5-Pad2)
- FB33 pad 2: (no net) -> Net-(CN5-Pad3)
- FB34 pad 2: (no net) -> Net-(CN5-Pad4)
- FB35 pad 2: (no net) -> Net-(CN5-Pad6)
- FB37 pad 1: (no net) -> Net-(CN5-Pad7)
- FB38 pad 2: (no net) -> Net-(CN1-PadD)
- FB39 pad 2: (no net) -> Net-(CN1-PadE)
- FB4 pad 1: (no net) -> Net-(CN7-Pad4)
- FB40 pad 1: (no net) -> Net-(CN1-Pad11)
- FB5 pad 1: (no net) -> Net-(CN7-Pad3)
- FB58 pad 2: (no net) -> Net-(CN6-Pad5)
- R102 pad 2: (no net) -> Net-(CN7-Pad1)
- U1 pad 13: (no net) -> COLOR
- U1 pad 23: (no net) -> SYNC_LUM
- U14 pad 10: (no net) -> C1_HIGH
- U14 pad 6: (no net) -> C1_LOW
- U14 pad 7: (no net) -> C2_LOW
- U14 pad 9: (no net) -> C2_HIGH
- U16 pad 17: (no net) -> PHI2
Routing:
- net Net-(FB41-Pad2): track 0.00 -> 75.9 mm
- net k7: track 0.00 -> 54.1 mm
- net k6: track 0.00 -> 49.4 mm
- net k5: track 0.00 -> 46.9 mm
- net k4: track 0.00 -> 39.3 mm
- net Net-(FB47-Pad2): track 0.00 -> 38.5 mm
- net Net-(FB44-Pad2): track 0.00 -> 33.0 mm
- net Net-(FB43-Pad2): track 0.00 -> 29.0 mm
- net Net-(FB45-Pad2): track 0.00 -> 28.3 mm
- net Net-(FB46-Pad2): track 0.00 -> 28.1 mm
- net Net-(CN2-Pad3): track 0.00 -> 27.6 mm
- net d4: track 0.00 -> 25.9 mm
- net d2: track 0.00 -> 25.8 mm
- net d3: track 0.00 -> 25.8 mm
- net Net-(FB48-Pad2): track 0.00 -> 24.5 mm, vias 0 -> 1
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