File: kbd+joy.sch (KiCad schematic (older format))
At the start: 50 parts, among them CN2 KEYBOARD_HEADER, CN4 JOY1, CN5 JOY2, U11 74LS125, U13 MOS_6529

Commit message: Add PLA
Parts:
- U11: footprint (none) -> Package_DIP:DIP-14_W7.62mm_Socket_LongPads
- U13: footprint MODULE -> Package_DIP:DIP-20_W7.62mm_Socket_LongPads
Changed lines of the file:
@@
 F 0 "U13" H 5115 2475 50  0000 C CNN
 F 1 "MOS_6529" H 5115 2384 50  0000 C CNN
-F 2 "MODULE" H 5115 1660 50  0001 C CNN
+F 2 "Package_DIP:DIP-20_W7.62mm_Socket_LongPads" H 5115 1660 50  0001 C CNN
 F 3 "DOCUMENTATION" H 5115 1660 50  0001 C CNN
 	1    5115 1660
@@
 F 0 "U13" H 9807 5406 50  0000 R CNN
 F 1 "MOS_6529" H 9807 5315 50  0000 R CNN
-F 2 "MODULE" H 10075 5360 50  0001 C CNN
+F 2 "Package_DIP:DIP-20_W7.62mm_Socket_LongPads" H 10075 5360 50  0001 C CNN
 F 3 "DOCUMENTATION" H 10075 5360 50  0001 C CNN
 	2    10075 5360
@@
 F 0 "U11" H 5295 3237 50  0000 C CNN
 F 1 "74LS125" H 5295 3146 50  0000 C CNN
-F 2 "" H 5295 2920 50  0001 C CNN
+F 2 "Package_DIP:DIP-14_W7.62mm_Socket_LongPads" H 5295 2920 50  0001 C CNN
 F 3 "http://www.ti.com/lit/gpn/sn74LS125" H 5295 2920 50  0001 C CNN
 	1    5295 2920
@@
 F 0 "U11" H 3855 5062 50  0000 C CNN
 F 1 "74LS125" H 3855 4971 50  0000 C CNN
-F 2 "" H 3855 4745 50  0001 C CNN
+F 2 "Package_DIP:DIP-14_W7.62mm_Socket_LongPads" H 3855 4745 50  0001 C CNN
 F 3 "http://www.ti.com/lit/gpn/sn74LS125" H 3855 4745 50  0001 C CNN
 	2    3855 4745

Commit message: Fix schematics here and there
Changed lines of the file:
@@
 $Descr A4 11693 8268
 encoding utf-8
-Sheet 3 11
+Sheet 6 11
 Title "CSeventeen"
-Date "2019-11-26"
+Date "2020-01-03"
 Rev "1git"
 Comp "SukkoPera"
-Comment1 ""
-Comment2 ""
+Comment1 "Licensed under CC BY-NC-SA 4.0"
+Comment2 "WARNING: These schematics might contain errors!"
 Comment3 ""
 Comment4 ""
@@
 	1    0    0    -1
 $EndComp
-Text Notes 665  2090 0    50   ~ 0
+Text Notes 3350 2115 2    50   ~ 0
 According to Wikipedia, "it is rather clear that the 6529 is just a\nrelabeled 74(LS)639 bidirectional three-state/open-Collector-bus\ndriver. [...]\n\nIf Open-Collector-Output at A-Side is NOT necessary (e.g. for input\nonly application like in Commodore C16 Keyboard-Scanner) 74LS245,\nwhich is available much more easily today will also do."
 Entry Wire Line
@@
 	5595 2920 5725 2920
 Wire Wire Line
-	5725 2920 5725 3500
-Wire Wire Line
-	5055 3505 5725 3500
+	5725 2920 5725 3505
+Wire Wire Line
+	5055 3505 5725 3505
 $Comp
 L power:GND #PWR0107
