File: kbd+joy.sch (KiCad schematic (older format))
At the start: 52 parts, among them CN2 KEYBOARD_HEADER, CN4 JOY1, CN5 JOY2, U11 74LS125, U13 MOS_6529

Commit message: CSeventeen -> LittleSixteen (PCB)
Parts:
- EM1, EM2: footprint CSeventeen:EMI_Filter -> LittleSixteen:EMI_Filter
- FB22, FB24, FB25, FB26, FB27, FB28, FB29, FB30, FB31, FB32, FB33, FB34, FB35, FB37, FB41, FB42, FB43, FB44, FB45, FB46, FB47, FB48, FB49, FB50, FB51, FB52, FB53, FB54, FB55, FB56: footprint CSeventeen:Ferrite -> LittleSixteen:Ferrite
Changed lines of the file:
@@
 F 0 "EM1" H 4755 3830 50  0000 C CNN
 F 1 "EMI_Filter_LCL" H 4755 3831 50  0001 C CNN
-F 2 "CSeventeen:EMI_Filter" V 4755 3605 50  0001 C CNN
+F 2 "LittleSixteen:EMI_Filter" V 4755 3605 50  0001 C CNN
 F 3 "http://www.murata.com/~/media/webrenewal/support/library/catalog/products/emc/emifil/c31e.ashx?la=en-gb" V 4755 3605 50  0001 C CNN
 	1    4755 3605
@@
 F 0 "FB24" V 6020 3935 50  0000 C CNN
 F 1 "Ferrite_Bead_Small" V 6019 3935 50  0001 C CNN
-F 2 "CSeventeen:Ferrite" V 6095 3935 50  0001 C CNN
+F 2 "LittleSixteen:Ferrite" V 6095 3935 50  0001 C CNN
 F 3 "~" H 6165 3935 50  0001 C CNN
 	1    6165 3935
@@
 F 0 "FB25" V 6220 4005 50  0000 C CNN
 F 1 "Ferrite_Bead_Small" V 6219 4005 50  0001 C CNN
-F 2 "CSeventeen:Ferrite" V 6295 4005 50  0001 C CNN
+F 2 "LittleSixteen:Ferrite" V 6295 4005 50  0001 C CNN
 F 3 "~" H 6365 4005 50  0001 C CNN
 	1    6365 4005
@@
 F 0 "FB27" V 6510 4150 50  0000 C CNN
 F 1 "Ferrite_Bead_Small" V 6219 4150 50  0001 C CNN
-F 2 "CSeventeen:Ferrite" V 6295 4150 50  0001 C CNN
+F 2 "LittleSixteen:Ferrite" V 6295 4150 50  0001 C CNN
 F 3 "~" H 6365 4150 50  0001 C CNN
 	1    6365 4150
@@
 F 0 "FB26" V 6300 4080 50  0000 C CNN
 F 1 "Ferrite_Bead_Small" V 6019 4080 50  0001 C CNN
-F 2 "CSeventeen:Ferrite" V 6095 4080 50  0001 C CNN
+F 2 "LittleSixteen:Ferrite" V 6095 4080 50  0001 C CNN
 F 3 "~" H 6165 4080 50  0001 C CNN
 	1    6165 4080
@@
 F 0 "FB22" H 4310 4000 50  0000 L CNN
 F 1 "Ferrite_Bead_Small" V 4064 4000 50  0001 C CNN
-F 2 "CSeventeen:Ferrite" V 4140 4000 50  0001 C CNN
+F 2 "LittleSixteen:Ferrite" V 4140 4000 50  0001 C CNN
 F 3 "~" H 4210 4000 50  0001 C CNN
 	1    4210 4000
@@
 F 0 "FB28" V 6300 4470 50  0000 C CNN
 F 1 "Ferrite_Bead_Small" V 6019 4470 50  0001 C CNN
-F 2 "CSeventeen:Ferrite" V 6095 4470 50  0001 C CNN
+F 2 "LittleSixteen:Ferrite" V 6095 4470 50  0001 C CNN
 F 3 "~" H 6165 4470 50  0001 C CNN
 	1    6165 4470
@@
 F 0 "FB29" V 4920 3780 50  0000 C CNN
 F 1 "Ferrite_Bead_Small" V 4889 3780 50  0001 C CNN
-F 2 "CSeventeen:Ferrite" V 4965 3780 50  0001 C CNN
+F 2 "LittleSixteen:Ferrite" V 4965 3780 50  0001 C CNN
 F 3 "~" H 5035 3780 50  0001 C CNN
 	1    5035 3780
@@
 F 0 "EM2" H 3315 5655 50  0000 C CNN
 F 1 "EMI_Filter_LCL" H 3315 5656 50  0001 C CNN
-F 2 "CSeventeen:EMI_Filter" V 3315 5430 50  0001 C CNN
+F 2 "LittleSixteen:EMI_Filter" V 3315 5430 50  0001 C CNN
 F 3 "http://www.murata.com/~/media/webrenewal/support/library/catalog/products/emc/emifil/c31e.ashx?la=en-gb" V 3315 5430 50  0001 C CNN
 	1    3315 5430
@@
 F 0 "FB31" V 4625 5760 50  0000 C CNN
 F 1 "Ferrite_Bead_Small" V 4624 5760 50  0001 C CNN
-F 2 "CSeventeen:Ferrite" V 4700 5760 50  0001 C CNN
+F 2 "LittleSixteen:Ferrite" V 4700 5760 50  0001 C CNN
 F 3 "~" H 4770 5760 50  0001 C CNN
 	1    4770 5760
@@
 F 0 "FB32" V 4825 5830 50  0000 C CNN
 F 1 "Ferrite_Bead_Small" V 4824 5830 50  0001 C CNN
-F 2 "CSeventeen:Ferrite" V 4900 5830 50  0001 C CNN
+F 2 "LittleSixteen:Ferrite" V 4900 5830 50  0001 C CNN
 F 3 "~" H 4970 5830 50  0001 C CNN
 	1    4970 5830
@@
 F 0 "FB34" V 5115 5975 50  0000 C CNN
 F 1 "Ferrite_Bead_Small" V 4824 5975 50  0001 C CNN
-F 2 "CSeventeen:Ferrite" V 4900 5975 50  0001 C CNN
+F 2 "LittleSixteen:Ferrite" V 4900 5975 50  0001 C CNN
 F 3 "~" H 4970 5975 50  0001 C CNN
 	1    4970 5975
@@
 F 0 "FB33" V 4905 5905 50  0000 C CNN
 F 1 "Ferrite_Bead_Small" V 4624 5905 50  0001 C CNN
-F 2 "CSeventeen:Ferrite" V 4700 5905 50  0001 C CNN
+F 2 "LittleSixteen:Ferrite" V 4700 5905 50  0001 C CNN
 F 3 "~" H 4770 5905 50  0001 C CNN
 	1    4770 5905
@@
 F 0 "FB30" H 2870 5825 50  0000 L CNN
 F 1 "Ferrite_Bead_Small" V 2624 5825 50  0001 C CNN
-F 2 "CSeventeen:Ferrite" V 2700 5825 50  0001 C CNN
+F 2 "LittleSixteen:Ferrite" V 2700 5825 50  0001 C CNN
 F 3 "~" H 2770 5825 50  0001 C CNN
 	1    2770 5825
@@
 F 0 "FB35" V 4905 6295 50  0000 C CNN
 F 1 "Ferrite_Bead_Small" V 4624 6295 50  0001 C CNN
-F 2 "CSeventeen:Ferrite" V 4700 6295 50  0001 C CNN
+F 2 "LittleSixteen:Ferrite" V 4700 6295 50  0001 C CNN
 F 3 "~" H 4770 6295 50  0001 C CNN
 	1    4770 6295
@@
 F 0 "FB37" V 3480 5605 50  0000 C CNN
 F 1 "Ferrite_Bead_Small" V 3449 5605 50  0001 C CNN
-F 2 "CSeventeen:Ferrite" V 3525 5605 50  0001 C CNN
+F 2 "LittleSixteen:Ferrite" V 3525 5605 50  0001 C CNN
 F 3 "~" H 3595 5605 50  0001 C CNN
 	1    3595 5605
@@
 F 0 "FB46" V 8475 880 50  0000 C CNN
 F 1 "Ferrite_Bead_Small" V 8474 880 50  0001 C CNN
-F 2 "CSeventeen:Ferrite" V 8550 880 50  0001 C CNN
+F 2 "LittleSixteen:Ferrite" V 8550 880 50  0001 C CNN
 F 3 "~" H 8620 880 50  0001 C CNN
 	1    8620 880
@@
 F 0 "FB56" V 8485 1080 50  0000 C CNN
 F 1 "Ferrite_Bead_Small" V 8484 1080 50  0001 C CNN
-F 2 "CSeventeen:Ferrite" V 8560 1080 50  0001 C CNN
+F 2 "LittleSixteen:Ferrite" V 8560 1080 50  0001 C CNN
 F 3 "~" H 8630 1080 50  0001 C CNN
 	1    8630 1080
@@
 F 0 "FB53" V 8485 1480 50  0000 C CNN
 F 1 "Ferrite_Bead_Small" V 8484 1480 50  0001 C CNN
-F 2 "CSeventeen:Ferrite" V 8560 1480 50  0001 C CNN
+F 2 "LittleSixteen:Ferrite" V 8560 1480 50  0001 C CNN
 F 3 "~" H 8630 1480 50  0001 C CNN
 	1    8630 1480
@@
 F 0 "FB54" V 8495 1680 50  0000 C CNN
 F 1 "Ferrite_Bead_Small" V 8494 1680 50  0001 C CNN
-F 2 "CSeventeen:Ferrite" V 8570 1680 50  0001 C CNN
+F 2 "LittleSixteen:Ferrite" V 8570 1680 50  0001 C CNN
 F 3 "~" H 8640 1680 50  0001 C CNN
 	1    8640 1680
@@
 F 0 "FB44" V 8470 1880 50  0000 C CNN
 F 1 "Ferrite_Bead_Small" V 8469 1880 50  0001 C CNN
-F 2 "CSeventeen:Ferrite" V 8545 1880 50  0001 C CNN
+F 2 "LittleSixteen:Ferrite" V 8545 1880 50  0001 C CNN
 F 3 "~" H 8615 1880 50  0001 C CNN
 	1    8615 1880
@@
 F 0 "FB45" V 8470 2080 50  0000 C CNN
 F 1 "Ferrite_Bead_Small" V 8469 2080 50  0001 C CNN
-F 2 "CSeventeen:Ferrite" V 8545 2080 50  0001 C CNN
+F 2 "LittleSixteen:Ferrite" V 8545 2080 50  0001 C CNN
 F 3 "~" H 8615 2080 50  0001 C CNN
 	1    8615 2080
@@
 F 0 "FB50" V 8480 2280 50  0000 C CNN
 F 1 "Ferrite_Bead_Small" V 8479 2280 50  0001 C CNN
-F 2 "CSeventeen:Ferrite" V 8555 2280 50  0001 C CNN
+F 2 "LittleSixteen:Ferrite" V 8555 2280 50  0001 C CNN
 F 3 "~" H 8625 2280 50  0001 C CNN
 	1    8625 2280
@@
 F 0 "FB52" V 8480 2480 50  0000 C CNN
 F 1 "Ferrite_Bead_Small" V 8479 2480 50  0001 C CNN
-F 2 "CSeventeen:Ferrite" V 8555 2480 50  0001 C CNN
+F 2 "LittleSixteen:Ferrite" V 8555 2480 50  0001 C CNN
 F 3 "~" H 8625 2480 50  0001 C CNN
 	1    8625 2480
@@
 F 0 "FB41" V 8765 2680 50  0000 C CNN
 F 1 "Ferrite_Bead_Small" V 8474 2680 50  0001 C CNN
-F 2 "CSeventeen:Ferrite" V 8550 2680 50  0001 C CNN
+F 2 "LittleSixteen:Ferrite" V 8550 2680 50  0001 C CNN
 F 3 "~" H 8620 2680 50  0001 C CNN
 	1    8620 2680
@@
 F 0 "FB48" V 8695 1380 50  0000 C CNN
 F 1 "Ferrite_Bead_Small" V 8694 1380 50  0001 C CNN
-F 2 "CSeventeen:Ferrite" V 8770 1380 50  0001 C CNN
+F 2 "LittleSixteen:Ferrite" V 8770 1380 50  0001 C CNN
 F 3 "~" H 8840 1380 50  0001 C CNN
 	1    8840 1380
@@
 F 0 "FB42" V 8715 1580 50  0000 C CNN
 F 1 "Ferrite_Bead_Small" V 8714 1580 50  0001 C CNN
-F 2 "CSeventeen:Ferrite" V 8790 1580 50  0001 C CNN
+F 2 "LittleSixteen:Ferrite" V 8790 1580 50  0001 C CNN
 F 3 "~" H 8860 1580 50  0001 C CNN
 	1    8860 1580
@@
 F 0 "FB55" V 8705 1780 50  0000 C CNN
 F 1 "Ferrite_Bead_Small" V 8704 1780 50  0001 C CNN
-F 2 "CSeventeen:Ferrite" V 8780 1780 50  0001 C CNN
+F 2 "LittleSixteen:Ferrite" V 8780 1780 50  0001 C CNN
 F 3 "~" H 8850 1780 50  0001 C CNN
 	1    8850 1780
@@
 F 0 "FB43" V 8685 1980 50  0000 C CNN
 F 1 "Ferrite_Bead_Small" V 8684 1980 50  0001 C CNN
-F 2 "CSeventeen:Ferrite" V 8760 1980 50  0001 C CNN
+F 2 "LittleSixteen:Ferrite" V 8760 1980 50  0001 C CNN
 F 3 "~" H 8830 1980 50  0001 C CNN
 	1    8830 1980
@@
 F 0 "FB51" V 8710 2180 50  0000 C CNN
 F 1 "Ferrite_Bead_Small" V 8709 2180 50  0001 C CNN
-F 2 "CSeventeen:Ferrite" V 8785 2180 50  0001 C CNN
+F 2 "LittleSixteen:Ferrite" V 8785 2180 50  0001 C CNN
 F 3 "~" H 8855 2180 50  0001 C CNN
 	1    8855 2180
@@
 F 0 "FB47" V 8710 2380 50  0000 C CNN
 F 1 "Ferrite_Bead_Small" V 8709 2380 50  0001 C CNN
-F 2 "CSeventeen:Ferrite" V 8785 2380 50  0001 C CNN
+F 2 "LittleSixteen:Ferrite" V 8785 2380 50  0001 C CNN
 F 3 "~" H 8855 2380 50  0001 C CNN
 	1    8855 2380
@@
 F 0 "FB49" V 8960 2580 50  0000 C CNN
 F 1 "Ferrite_Bead_Small" V 8694 2580 50  0001 C CNN
-F 2 "CSeventeen:Ferrite" V 8770 2580 50  0001 C CNN
+F 2 "LittleSixteen:Ferrite" V 8770 2580 50  0001 C CNN
 F 3 "~" H 8840 2580 50  0001 C CNN
 	1    8840 2580

Commit message: Laid out data bus and muuuuch more stuff
Connections:
- net k0: no longer RP5.2 (R1)
- net k1: no longer RP5.6 (R5)
- net k2: no longer RP5.3 (R2)
- net k3: no longer RP5.5 (R4)
- net k7: no longer RP5.4 (R3)
- net at CN4.8: now also EM1.3; no longer EM1.1
- net at U11.3: now also EM1.1; no longer EM1.3
- net at EM2.1: now also U11.6; no longer CN5.8
- net at EM2.3: now also CN5.8; no longer U11.6
- net at D6.1 (K), FB31.1: now also RP5.2 (R1)
- net at D7.1 (K), FB32.1: now also RP5.6 (R5)
- net at D8.1 (K), FB33.1: now also RP5.3 (R2)
- net at D9.1 (K), FB34.1: now also RP5.5 (R4)
- net at D10.1 (K), FB35.1: now also RP5.4 (R3)
Other:
- moved on the sheet: D10, D6, D7, D8, D9, RP5
Changed lines of the file:
@@
 Sheet 6 11
 Title "LittleSixteen"
-Date "2020-01-20"
+Date "2021-07-15"
 Rev "1git"
 Comp "SukkoPera"
@@
 F 3 "http://www.murata.com/~/media/webrenewal/support/library/catalog/products/emc/emifil/c31e.ashx?la=en-gb" V 4755 3605 50  0001 C CNN
 	1    4755 3605
-	1    0    0    -1
+	-1   0    0    -1
 $EndComp
 Wire Wire Line
@@
 F 3 "http://www.murata.com/~/media/webrenewal/support/library/catalog/products/emc/emifil/c31e.ashx?la=en-gb" V 3315 5430 50  0001 C CNN
 	1    3315 5430
-	1    0    0    -1
+	-1   0    0    -1
 $EndComp
 Wire Wire Line
@@
 L Diode:1N914 D6
 U 1 1 5E19A82E
-P 5320 5760
-F 0 "D6" H 5320 5976 50  0000 C CNN
-F 1 "1N914" H 5320 5885 50  0000 C CNN
-F 2 "Diode_THT:D_DO-35_SOD27_P5.08mm_Vertical_KathodeUp" H 5320 5585 50  0001 C CNN
-F 3 "http://www.vishay.com/docs/85622/1n914.pdf" H 5320 5760 50  0001 C CNN
-	1    5320 5760
+P 6605 5760
+F 0 "D6" H 6605 5976 50  0000 C CNN
+F 1 "1N914" H 6605 5885 50  0000 C CNN
+F 2 "Diode_THT:D_DO-35_SOD27_P5.08mm_Vertical_KathodeUp" H 6605 5585 50  0001 C CNN
+F 3 "http://www.vishay.com/docs/85622/1n914.pdf" H 6605 5760 50  0001 C CNN
+	1    6605 5760
 	1    0    0    -1
 $EndComp
@@
 L Diode:1N914 D7
 U 1 1 5E19A838
-P 5620 5830
-F 0 "D7" H 5620 6046 50  0000 C CNN
-F 1 "1N914" H 5620 5955 50  0000 C CNN
-F 2 "Diode_THT:D_DO-35_SOD27_P5.08mm_Vertical_KathodeUp" H 5620 5655 50  0001 C CNN
-F 3 "http://www.vishay.com/docs/85622/1n914.pdf" H 5620 5830 50  0001 C CNN
-	1    5620 5830
+P 6905 5830
+F 0 "D7" H 6905 6046 50  0000 C CNN
+F 1 "1N914" H 6905 5955 50  0000 C CNN
+F 2 "Diode_THT:D_DO-35_SOD27_P5.08mm_Vertical_KathodeUp" H 6905 5655 50  0001 C CNN
+F 3 "http://www.vishay.com/docs/85622/1n914.pdf" H 6905 5830 50  0001 C CNN
+	1    6905 5830
 	1    0    0    -1
 $EndComp
@@
 L Diode:1N914 D8
 U 1 1 5E19A842
-P 5320 5905
-F 0 "D8" H 5320 5775 50  0000 C CNN
-F 1 "1N914" H 5320 5680 50  0000 C CNN
-F 2 "Diode_THT:D_DO-35_SOD27_P5.08mm_Vertical_KathodeUp" H 5320 5730 50  0001 C CNN
-F 3 "http://www.vishay.com/docs/85622/1n914.pdf" H 5320 5905 50  0001 C CNN
-	1    5320 5905
+P 6605 5905
+F 0 "D8" H 6605 5775 50  0000 C CNN
+F 1 "1N914" H 6605 5680 50  0000 C CNN
+F 2 "Diode_THT:D_DO-35_SOD27_P5.08mm_Vertical_KathodeUp" H 6605 5730 50  0001 C CNN
+F 3 "http://www.vishay.com/docs/85622/1n914.pdf" H 6605 5905 50  0001 C CNN
+	1    6605 5905
 	1    0    0    -1
 $EndComp
@@
 L Diode:1N914 D9
 U 1 1 5E19A84C
-P 5620 5975
-F 0 "D9" H 5620 5851 50  0000 C CNN
-F 1 "1N914" H 5620 5760 50  0000 C CNN
-F 2 "Diode_THT:D_DO-35_SOD27_P5.08mm_Vertical_KathodeUp" H 5620 5800 50  0001 C CNN
-F 3 "http://www.vishay.com/docs/85622/1n914.pdf" H 5620 5975 50  0001 C CNN
-	1    5620 5975
+P 6905 5975
+F 0 "D9" H 6905 5851 50  0000 C CNN
+F 1 "1N914" H 6905 5760 50  0000 C CNN
+F 2 "Diode_THT:D_DO-35_SOD27_P5.08mm_Vertical_KathodeUp" H 6905 5800 50  0001 C CNN
+F 3 "http://www.vishay.com/docs/85622/1n914.pdf" H 6905 5975 50  0001 C CNN
+	1    6905 5975
 	1    0    0    -1
 $EndComp
@@
 	4495 5905 4670 5905
 Wire Wire Line
-	5470 5975 5070 5975
+	6755 5975 5770 5975
 Wire Wire Line
 	4575 5975 4575 6490
@@
 L Diode:1N914 D10
 U 1 1 5E19A869
-P 5320 6295
-F 0 "D10" H 5320 6171 50  0000 C CNN
-F 1 "1N914" H 5320 6080 50  0000 C CNN
-F 2 "Diode_THT:D_DO-35_SOD27_P5.08mm_Vertical_KathodeUp" H 5320 6120 50  0001 C CNN
-F 3 "http://www.vishay.com/docs/85622/1n914.pdf" H 5320 6295 50  0001 C CNN
-	1    5320 6295
+P 6605 6295
+F 0 "D10" H 6605 6171 50  0000 C CNN
+F 1 "1N914" H 6605 6080 50  0000 C CNN
+F 2 "Diode_THT:D_DO-35_SOD27_P5.08mm_Vertical_KathodeUp" H 6605 6120 50  0001 C CNN
+F 3 "http://www.vishay.com/docs/85622/1n914.pdf" H 6605 6295 50  0001 C CNN
+	1    6605 6295
 	1    0    0    -1
 $EndComp
@@
 $EndComp
 Wire Wire Line
-	4870 5760 5170 5760
+	4870 5760 5470 5760
 $Comp
 L Device:Ferrite_Bead_Small FB32
@@
 $EndComp
 Wire Wire Line
-	5070 5830 5470 5830
+	5070 5830 5870 5830
 $Comp
 L Device:Ferrite_Bead_Small FB34
@@
 $EndComp
 Wire Wire Line
-	4870 5905 5170 5905
+	4870 5905 5570 5905
 $Comp
 L Device:Ferrite_Bead_Small FB30
@@
 	2770 6110 3575 6110
 Wire Wire Line
-	4870 6295 5170 6295
+	4870 6295 5670 6295
 $Comp
 L Device:Ferrite_Bead_Small FB35
@@
 Wire Wire Line
 	7955 5760 7955 2580
-Wire Wire Line
-	5470 5760 6485 5760
 Connection ~ 7955 2580
 Wire Wire Line
@@
 Wire Wire Line
 	8045 5830 8045 2280
-Wire Wire Line
-	5770 5830 6885 5830
 Connection ~ 8045 2280
 Wire Wire Line
@@
 Wire Wire Line
 	8130 5905 8130 2180
-Wire Wire Line
-	5470 5905 6585 5905
 Connection ~ 8130 2180
 Wire Wire Line
@@
 Wire Wire Line
 	8215 5975 8215 2480
-Wire Wire Line
-	5770 5975 6785 5975
 Connection ~ 8215 2480
 Wire Wire Line
 	8215 2480 8525 2480
-Wire Wire Line
-	5470 6295 6685 6295
 Wire Wire Line
 	8315 6295 8315 1080
@@
 L Device:R_Network05 RP5
 U 1 1 5E3A4C16
-P 6685 5375
-F 0 "RP5" H 6973 5421 50  0000 L CNN
-F 1 "3.3k" H 6973 5330 50  0000 L CNN
-F 2 "Resistor_THT:R_Array_SIP6" V 7060 5375 50  0001 C CNN
-F 3 "http://www.vishay.com/docs/31509/csc.pdf" H 6685 5375 50  0001 C CNN
-	1    6685 5375
+P 5670 5375
+F 0 "RP5" H 5958 5421 50  0000 L CNN
+F 1 "3.3k" H 5958 5330 50  0000 L CNN
+F 2 "Resistor_THT:R_Array_SIP6" V 6045 5375 50  0001 C CNN
+F 3 "http://www.vishay.com/docs/31509/csc.pdf" H 5670 5375 50  0001 C CNN
+	1    5670 5375
 	1    0    0    -1
 $EndComp
@@
 L power:VCC #PWR0112
 U 1 1 5E419B38
-P 6485 5070
-F 0 "#PWR0112" H 6485 4920 50  0001 C CNN
-F 1 "VCC" H 6502 5243 50  0000 C CNN
-F 2 "" H 6485 5070 50  0001 C CNN
-F 3 "" H 6485 5070 50  0001 C CNN
-	1    6485 5070
-	1    0    0    -1
-$EndComp
-Wire Wire Line
-	6485 5070 6485 5175
+P 5470 5070
+F 0 "#PWR0112" H 5470 4920 50  0001 C CNN
+F 1 "VCC" H 5487 5243 50  0000 C CNN
+F 2 "" H 5470 5070 50  0001 C CNN
+F 3 "" H 5470 5070 50  0001 C CNN
+	1    5470 5070
+	1    0    0    -1
+$EndComp
+Wire Wire Line
+	5470 5070 5470 5175
 Wire Wire Line
 	6885 3745 6885 4005
@@
 $EndComp
 Wire Wire Line
-	6485 5575 6485 5760
-Connection ~ 6485 5760
-Wire Wire Line
-	6485 5760 7955 5760
-Wire Wire Line
-	6885 5575 6885 5830
-Connection ~ 6885 5830
-Wire Wire Line
-	6885 5830 8045 5830
-Wire Wire Line
-	6585 5575 6585 5905
-Connection ~ 6585 5905
-Wire Wire Line
-	6585 5905 8130 5905
-Wire Wire Line
-	6785 5575 6785 5975
-Connection ~ 6785 5975
-Wire Wire Line
-	6785 5975 8215 5975
-Wire Wire Line
-	6685 5575 6685 6295
-Connection ~ 6685 6295
-Wire Wire Line
-	6685 6295 8315 6295
+	5470 5575 5470 5760
+Wire Wire Line
+	5870 5575 5870 5830
+Wire Wire Line
+	5570 5575 5570 5905
+Wire Wire Line
+	5770 5575 5770 5975
+Wire Wire Line
+	5670 5575 5670 6295
 Wire Wire Line
 	4765 2920 4995 2920
@@
 	0    -1   -1   0
 $EndComp
+Wire Wire Line
+	6755 5760 7955 5760
+Wire Wire Line
+	7055 5830 8045 5830
+Wire Wire Line
+	6755 5905 8130 5905
+Wire Wire Line
+	7055 5975 8215 5975
+Wire Wire Line
+	6755 6295 8315 6295
+Connection ~ 5470 5760
+Wire Wire Line
+	5470 5760 6455 5760
+Connection ~ 5570 5905
+Wire Wire Line
+	5570 5905 6455 5905
+Connection ~ 5670 6295
+Wire Wire Line
+	5670 6295 6455 6295
+Connection ~ 5770 5975
+Wire Wire Line
+	5770 5975 5070 5975
+Connection ~ 5870 5830
+Wire Wire Line
+	5870 5830 6755 5830
 Wire Bus Line
 	3510 1380 3510 2085
