File: LittleSixteen.kicad_pcb (KiCad board)
At the start: 2 copper layers, 320 x 136.2 mm, 162 parts, among them CN1 EXPANSION_CONNECTOR, CN2 KEYBOARD_HEADER, CN3 CASSETTE, CN4 JOY1, CN5 JOY2, CN6 AUDIO_VIDEO, CN7 SERIAL_BUS, CN9 LED_CONNECTOR, M1 Modulator, Q1 2SC1815, Q2 2SC1815, Q3 2SC1815, Q5 2SD880, SW1 POWER_SWITCH, SW2 RESET_SW, U1 MOS_7360_TED, U10 NE555, U11 74LS125, U12 74LS02, U13 MOS_6529, U14 74LS139, U15 74LS175, U16 MOS_251641_PLA, U2 MOS_8501, U3 23128_BASIC, U4 23128_KERNAL, U5 4416, U6 4416, U7 74LS257, U8 74LS257, U9 74LS06, Y1 Crystal

Commit message: CSeventeen -> LittleSixteen (PCB)
Parts:
- EM1, EM2, EM3, EM4, EM5: footprint CSeventeen:EMI_Filter -> LittleSixteen:EMI_Filter
- FB1, FB12, FB13, FB14, FB15, FB16, FB17, FB18, FB19, FB2, FB22, FB24, FB25, FB26, FB27, FB28, FB29, FB3, FB30, FB31, FB32, FB33, FB34, FB35, FB37, FB38, FB39, FB4, FB40, FB41, FB42, FB43, FB44, FB45, FB46, FB47, FB48, FB49, FB5, FB50, FB51, FB52, FB53, FB54, FB55, FB56, FB58: footprint CSeventeen:Ferrite -> LittleSixteen:Ferrite
- G***: footprint CSeventeen:Top4 -> LittleSixteen:Top4
- G***: footprint CSeventeen:Top3 -> LittleSixteen:Top3
