File: datasette.sch (KiCad schematic (older format))
At the start: 26 parts, among them CN3 CASSETTE, CN7 SERIAL_BUS, Q5 2SD880, U11 74LS125, U9 74LS06

Commit message: Start working on PCB
Parts:
- R102, R12, R13, R29: footprint (none) -> Resistor_THT:R_Axial_DIN0207_L6.3mm_D2.5mm_P5.08mm_Vertical
- RP1: footprint (none) -> Resistor_THT:R_Array_SIP6
Changed lines of the file:
@@
 F 0 "R13" H 8285 1981 50  0000 L CNN
 F 1 "470" H 8285 1890 50  0000 L CNN
-F 2 "" V 8145 1935 50  0001 C CNN
+F 2 "Resistor_THT:R_Axial_DIN0207_L6.3mm_D2.5mm_P5.08mm_Vertical" V 8145 1935 50  0001 C CNN
 F 3 "~" H 8215 1935 50  0001 C CNN
 	1    8215 1935
@@
 F 0 "R29" V 6018 2460 50  0000 C CNN
 F 1 "100" V 6109 2460 50  0000 C CNN
-F 2 "" V 6155 2460 50  0001 C CNN
+F 2 "Resistor_THT:R_Axial_DIN0207_L6.3mm_D2.5mm_P5.08mm_Vertical" V 6155 2460 50  0001 C CNN
 F 3 "~" H 6225 2460 50  0001 C CNN
 	1    6225 2460
@@
 F 0 "R12" H 5420 1401 50  0000 L CNN
 F 1 "3.3k" H 5420 1310 50  0000 L CNN
-F 2 "" V 5280 1355 50  0001 C CNN
+F 2 "Resistor_THT:R_Axial_DIN0207_L6.3mm_D2.5mm_P5.08mm_Vertical" V 5280 1355 50  0001 C CNN
 F 3 "~" H 5350 1355 50  0001 C CNN
 	1    5350 1355
@@
 F 0 "R102" H 3625 5376 50  0000 L CNN
 F 1 "330" H 3625 5285 50  0000 L CNN
-F 2 "" V 3485 5330 50  0001 C CNN
+F 2 "Resistor_THT:R_Axial_DIN0207_L6.3mm_D2.5mm_P5.08mm_Vertical" V 3485 5330 50  0001 C CNN
 F 3 "~" H 3555 5330 50  0001 C CNN
 	1    3555 5330
@@
 F 0 "RP1" H 5475 5075 50  0000 R CNN
 F 1 "1k" H 5593 4885 50  0001 L CNN
-F 2 "" V 5435 4930 50  0001 C CNN
+F 2 "Resistor_THT:R_Array_SIP6" V 5435 4930 50  0001 C CNN
 F 3 "~" H 5505 4930 50  0001 C CNN
 	2    5505 4930
@@
 F 0 "RP1" H 5655 4730 50  0000 L CNN
 F 1 "1k" H 5738 4885 50  0001 L CNN
-F 2 "" V 5580 4930 50  0001 C CNN
+F 2 "Resistor_THT:R_Array_SIP6" V 5580 4930 50  0001 C CNN
 F 3 "~" H 5650 4930 50  0001 C CNN
 	3    5650 4930
@@
 F 0 "RP1" H 5805 5095 50  0000 L CNN
 F 1 "1k" H 5888 4885 50  0001 L CNN
-F 2 "" V 5730 4930 50  0001 C CNN
+F 2 "Resistor_THT:R_Array_SIP6" V 5730 4930 50  0001 C CNN
 F 3 "~" H 5800 4930 50  0001 C CNN
 	4    5800 4930
@@
 F 0 "RP1" H 5960 4730 50  0000 L CNN
 F 1 "1k" H 6030 4930 50  0000 L CNN
-F 2 "" V 5880 4930 50  0001 C CNN
+F 2 "Resistor_THT:R_Array_SIP6" V 5880 4930 50  0001 C CNN
 F 3 "~" H 5950 4930 50  0001 C CNN
 	5    5950 4930

Commit message: Add ceramics
Parts:
- C23, C24, C25, C26: footprint (none) -> Capacitor_THT:C_Disc_D8.0mm_W2.5mm_P5.00mm
Changed lines of the file:
@@
 F 0 "C26" H 3895 2164 50  0000 R CNN
 F 1 "100n" H 3895 2255 50  0000 R CNN
-F 2 "" H 4048 2060 50  0001 C CNN
+F 2 "Capacitor_THT:C_Disc_D8.0mm_W2.5mm_P5.00mm" H 4048 2060 50  0001 C CNN
 F 3 "~" H 4010 2210 50  0001 C CNN
 	1    4010 2210
@@
 F 0 "C23" H 2780 2774 50  0000 R CNN
 F 1 "470p" H 2780 2865 50  0000 R CNN
-F 2 "" H 2933 2670 50  0001 C CNN
+F 2 "Capacitor_THT:C_Disc_D8.0mm_W2.5mm_P5.00mm" H 2933 2670 50  0001 C CNN
 F 3 "~" H 2895 2820 50  0001 C CNN
 	1    2895 2820
@@
 F 0 "C24" H 5735 2804 50  0000 R CNN
 F 1 "470p" H 5735 2895 50  0000 R CNN
-F 2 "" H 5888 2700 50  0001 C CNN
+F 2 "Capacitor_THT:C_Disc_D8.0mm_W2.5mm_P5.00mm" H 5888 2700 50  0001 C CNN
 F 3 "~" H 5850 2850 50  0001 C CNN
 	1    5850 2850
@@
 F 0 "C25" H 5235 2014 50  0000 R CNN
 F 1 "470p" H 5235 2105 50  0000 R CNN
-F 2 "" H 5388 1910 50  0001 C CNN
+F 2 "Capacitor_THT:C_Disc_D8.0mm_W2.5mm_P5.00mm" H 5388 1910 50  0001 C CNN
 F 3 "~" H 5350 2060 50  0001 C CNN
 	1    5350 2060

Commit message: Add diodes
Parts:
- D12: footprint (none) -> Diode_THT:D_DO-35_SOD27_P5.08mm_Vertical_KathodeUp
- Q5: footprint Package_TO_SOT_THT:TO-126-3_Vertical -> Package_TO_SOT_THT:TO-220-3_Horizontal_TabDown
Changed lines of the file:
@@
 F 0 "Q5" H 8007 2296 50  0000 L CNN
 F 1 "2SD880" H 8007 2205 50  0000 L CNN
-F 2 "Package_TO_SOT_THT:TO-126-3_Vertical" H 8015 2175 50  0001 L CIN
+F 2 "Package_TO_SOT_THT:TO-220-3_Horizontal_TabDown" H 8015 2175 50  0001 L CIN
 F 3 "http://pdf.datasheetcatalog.com/datasheet/sanyo/ds_pdf_e/2SB631.pdf" H 7815 2250 50  0001 L CNN
 	1    7815 2250
@@
 F 0 "D12" V 8278 2637 40  0000 R CNN
 F 1 "6.8V" V 8202 2637 40  0000 R CNN
-F 2 "" H 8215 2690 60  0001 C CNN
+F 2 "Diode_THT:D_DO-35_SOD27_P5.08mm_Vertical_KathodeUp" H 8215 2690 60  0001 C CNN
 F 3 "" H 8215 2690 60  0000 C CNN
 	1    8215 2690

Commit message: Add crystal
Parts:
- FB1, FB14, FB15, FB16, FB17, FB18, FB19, FB2, FB3, FB4, FB5: footprint (none) -> CSeventeen:Ferrite
Changed lines of the file:
@@
 F 0 "FB14" H 3795 2200 50  0000 L CNN
 F 1 "Ferrite_Bead_Small" H 3795 2155 50  0001 L CNN
-F 2 "" V 3625 2200 50  0001 C CNN
+F 2 "CSeventeen:Ferrite" V 3625 2200 50  0001 C CNN
 F 3 "~" H 3695 2200 50  0001 C CNN
 	1    3695 2200
@@
 F 0 "FB15" H 4830 2895 50  0000 R CNN
 F 1 "Ferrite_Bead_Small" H 5030 2850 50  0001 L CNN
-F 2 "" V 4860 2895 50  0001 C CNN
+F 2 "CSeventeen:Ferrite" V 4860 2895 50  0001 C CNN
 F 3 "~" H 4930 2895 50  0001 C CNN
 	1    4930 2895
@@
 F 0 "FB16" V 3395 2560 50  0000 C CNN
 F 1 "Ferrite_Bead_Small" H 3350 2515 50  0001 L CNN
-F 2 "" V 3180 2560 50  0001 C CNN
+F 2 "CSeventeen:Ferrite" V 3180 2560 50  0001 C CNN
 F 3 "~" H 3250 2560 50  0001 C CNN
 	1    3250 2560
@@
 F 0 "FB19" V 7535 2560 50  0000 C CNN
 F 1 "Ferrite_Bead_Small" H 7490 2515 50  0001 L CNN
-F 2 "" V 7320 2560 50  0001 C CNN
+F 2 "CSeventeen:Ferrite" V 7320 2560 50  0001 C CNN
 F 3 "~" H 7390 2560 50  0001 C CNN
 	1    7390 2560
@@
 F 0 "FB17" V 5730 2460 50  0000 C CNN
 F 1 "Ferrite_Bead_Small" H 5685 2415 50  0001 L CNN
-F 2 "" V 5515 2460 50  0001 C CNN
+F 2 "CSeventeen:Ferrite" V 5515 2460 50  0001 C CNN
 F 3 "~" H 5585 2460 50  0001 C CNN
 	1    5585 2460
@@
 F 0 "FB18" V 5175 1670 50  0000 C CNN
 F 1 "Ferrite_Bead_Small" H 5130 1625 50  0001 L CNN
-F 2 "" V 4960 1670 50  0001 C CNN
+F 2 "CSeventeen:Ferrite" V 4960 1670 50  0001 C CNN
 F 3 "~" H 5030 1670 50  0001 C CNN
 	1    5030 1670
@@
 F 0 "FB1" H 3580 6015 50  0000 R CNN
 F 1 "Ferrite_Bead_Small" H 3780 5970 50  0001 L CNN
-F 2 "" V 3610 6015 50  0001 C CNN
+F 2 "CSeventeen:Ferrite" V 3610 6015 50  0001 C CNN
 F 3 "~" H 3680 6015 50  0001 C CNN
 	1    3680 6015
@@
 F 0 "FB5" V 4920 5380 50  0000 C CNN
 F 1 "Ferrite_Bead_Small" H 4875 5335 50  0001 L CNN
-F 2 "" V 4705 5380 50  0001 C CNN
+F 2 "CSeventeen:Ferrite" V 4705 5380 50  0001 C CNN
 F 3 "~" H 4775 5380 50  0001 C CNN
 	1    4775 5380
@@
 F 0 "FB4" V 5220 5625 50  0000 C CNN
 F 1 "Ferrite_Bead_Small" H 5175 5580 50  0001 L CNN
-F 2 "" V 5005 5625 50  0001 C CNN
+F 2 "CSeventeen:Ferrite" V 5005 5625 50  0001 C CNN
 F 3 "~" H 5075 5625 50  0001 C CNN
 	1    5075 5625
@@
 F 0 "FB3" V 4630 5825 50  0000 C CNN
 F 1 "Ferrite_Bead_Small" H 4875 5780 50  0001 L CNN
-F 2 "" V 4705 5825 50  0001 C CNN
+F 2 "CSeventeen:Ferrite" V 4705 5825 50  0001 C CNN
 F 3 "~" H 4775 5825 50  0001 C CNN
 	1    4775 5825
@@
 F 0 "FB2" V 5215 6070 50  0000 C CNN
 F 1 "Ferrite_Bead_Small" H 5170 6025 50  0001 L CNN
-F 2 "" V 5000 6070 50  0001 C CNN
+F 2 "CSeventeen:Ferrite" V 5000 6070 50  0001 C CNN
 F 3 "~" H 5070 6070 50  0001 C CNN
 	1    5070 6070

Commit message: Use 3d models from github.com/StormTrooper/Commodore-Plus4
Parts:
- CN3: footprint (none) -> CommodorePlus4:Connector_Mini-DIN_Female_7Pin_2rows
- CN7: footprint (none) -> CommodorePlus4:Connector_DIN_Female_6Pin_3rows
Changed lines of the file:
@@
 F 0 "CN3" H 4490 2285 50  0000 C CNN
 F 1 "CASSETTE" H 4490 2194 50  0000 C CNN
-F 2 "" V 4480 2550 50  0001 C CNN
+F 2 "CommodorePlus4:Connector_Mini-DIN_Female_7Pin_2rows" V 4480 2550 50  0001 C CNN
 F 3 "http://service.powerdynamics.com/ec/Catalog17/Section%2011.pdf" V 4480 2550 50  0001 C CNN
 	1    4490 2560
@@
 F 0 "CN7" H 4140 6330 50  0000 C CNN
 F 1 "SERIAL_BUS" H 4140 6245 50  0000 C CNN
-F 2 "" H 4140 5725 50  0001 C CNN
+F 2 "CommodorePlus4:Connector_DIN_Female_6Pin_3rows" H 4140 5725 50  0001 C CNN
 F 3 "http://www.mouser.com/ds/2/18/40_c091_abd_e-75918.pdf" H 4140 5725 50  0001 C CNN
 	1    4140 5725

Commit message: CSeventeen -> LittleSixteen (PCB)
Parts:
- FB1, FB14, FB15, FB16, FB17, FB18, FB19, FB2, FB3, FB4, FB5: footprint CSeventeen:Ferrite -> LittleSixteen:Ferrite
Changed lines of the file:
@@
 F 0 "FB14" H 3795 2200 50  0000 L CNN
 F 1 "Ferrite_Bead_Small" H 3795 2155 50  0001 L CNN
-F 2 "CSeventeen:Ferrite" V 3625 2200 50  0001 C CNN
+F 2 "LittleSixteen:Ferrite" V 3625 2200 50  0001 C CNN
 F 3 "~" H 3695 2200 50  0001 C CNN
 	1    3695 2200
@@
 F 0 "FB15" H 4830 2895 50  0000 R CNN
 F 1 "Ferrite_Bead_Small" H 5030 2850 50  0001 L CNN
-F 2 "CSeventeen:Ferrite" V 4860 2895 50  0001 C CNN
+F 2 "LittleSixteen:Ferrite" V 4860 2895 50  0001 C CNN
 F 3 "~" H 4930 2895 50  0001 C CNN
 	1    4930 2895
@@
 F 0 "FB16" V 3395 2560 50  0000 C CNN
 F 1 "Ferrite_Bead_Small" H 3350 2515 50  0001 L CNN
-F 2 "CSeventeen:Ferrite" V 3180 2560 50  0001 C CNN
+F 2 "LittleSixteen:Ferrite" V 3180 2560 50  0001 C CNN
 F 3 "~" H 3250 2560 50  0001 C CNN
 	1    3250 2560
@@
 F 0 "FB19" V 7535 2560 50  0000 C CNN
 F 1 "Ferrite_Bead_Small" H 7490 2515 50  0001 L CNN
-F 2 "CSeventeen:Ferrite" V 7320 2560 50  0001 C CNN
+F 2 "LittleSixteen:Ferrite" V 7320 2560 50  0001 C CNN
 F 3 "~" H 7390 2560 50  0001 C CNN
 	1    7390 2560
@@
 F 0 "FB17" V 5730 2460 50  0000 C CNN
 F 1 "Ferrite_Bead_Small" H 5685 2415 50  0001 L CNN
-F 2 "CSeventeen:Ferrite" V 5515 2460 50  0001 C CNN
+F 2 "LittleSixteen:Ferrite" V 5515 2460 50  0001 C CNN
 F 3 "~" H 5585 2460 50  0001 C CNN
 	1    5585 2460
@@
 F 0 "FB18" V 5175 1670 50  0000 C CNN
 F 1 "Ferrite_Bead_Small" H 5130 1625 50  0001 L CNN
-F 2 "CSeventeen:Ferrite" V 4960 1670 50  0001 C CNN
+F 2 "LittleSixteen:Ferrite" V 4960 1670 50  0001 C CNN
 F 3 "~" H 5030 1670 50  0001 C CNN
 	1    5030 1670
@@
 F 0 "FB1" H 3580 6015 50  0000 R CNN
 F 1 "Ferrite_Bead_Small" H 3780 5970 50  0001 L CNN
-F 2 "CSeventeen:Ferrite" V 3610 6015 50  0001 C CNN
+F 2 "LittleSixteen:Ferrite" V 3610 6015 50  0001 C CNN
 F 3 "~" H 3680 6015 50  0001 C CNN
 	1    3680 6015
@@
 F 0 "FB5" V 4920 5380 50  0000 C CNN
 F 1 "Ferrite_Bead_Small" H 4875 5335 50  0001 L CNN
-F 2 "CSeventeen:Ferrite" V 4705 5380 50  0001 C CNN
+F 2 "LittleSixteen:Ferrite" V 4705 5380 50  0001 C CNN
 F 3 "~" H 4775 5380 50  0001 C CNN
 	1    4775 5380
@@
 F 0 "FB4" V 5220 5625 50  0000 C CNN
 F 1 "Ferrite_Bead_Small" H 5175 5580 50  0001 L CNN
-F 2 "CSeventeen:Ferrite" V 5005 5625 50  0001 C CNN
+F 2 "LittleSixteen:Ferrite" V 5005 5625 50  0001 C CNN
 F 3 "~" H 5075 5625 50  0001 C CNN
 	1    5075 5625
@@
 F 0 "FB3" V 4630 5825 50  0000 C CNN
 F 1 "Ferrite_Bead_Small" H 4875 5780 50  0001 L CNN
-F 2 "CSeventeen:Ferrite" V 4705 5825 50  0001 C CNN
+F 2 "LittleSixteen:Ferrite" V 4705 5825 50  0001 C CNN
 F 3 "~" H 4775 5825 50  0001 C CNN
 	1    4775 5825
@@
 F 0 "FB2" V 5215 6070 50  0000 C CNN
 F 1 "Ferrite_Bead_Small" H 5170 6025 50  0001 L CNN
-F 2 "CSeventeen:Ferrite" V 5000 6070 50  0001 C CNN
+F 2 "LittleSixteen:Ferrite" V 5000 6070 50  0001 C CNN
 F 3 "~" H 5070 6070 50  0001 C CNN
 	1    5070 6070

Commit message: Who remembers?
Parts:
- removed FB1, FB19, FB2, FB3, FB4, FB5: Ferrite_Bead_Small, LittleSixteen:Ferrite, symbol Device:Ferrite_Bead_Small
- added FB1, FB19, FB2, FB3, FB4, FB5: Ferrite_3pin, LittleSixteen:Ferrite, symbol Ferrite3Pin:Ferrite_3pin
Connections:
- net GND: now also FB1.2, FB1.3, FB19.3, FB2.3, FB3.3, FB4.3, FB5.3
- net p7: now also FB3.2
- net p[0..7]: now also FB4.2
- net at CN3.3: now also FB19.1
- net at Q5.1 (E): now also FB19.2
- net at CN7.2: now also FB1.1
- net at CN7.3: now also FB5.1
- net at CN7.4: now also FB4.1
- net at CN7.5: now also FB3.1
- net at CN7.6: now also FB2.1
- net at RP1.3, U9.8: now also FB5.2
- net at RP1.4, U9.4: now also FB2.2
Changed lines of the file:
@@
 	-1   0    0    -1
-$EndComp
-$Comp
-L Device:Ferrite_Bead_Small FB19
-U 1 1 5ECC99AD
-P 7390 2560
-F 0 "FB19" V 7535 2560 50  0000 C CNN
-F 1 "Ferrite_Bead_Small" H 7490 2515 50  0001 L CNN
-F 2 "LittleSixteen:Ferrite" V 7320 2560 50  0001 C CNN
-F 3 "~" H 7390 2560 50  0001 C CNN
-	1    7390 2560
-	0    -1   -1   0
 $EndComp
 Wire Wire Line
@@
 	8215 2740 8215 3100
 Wire Wire Line
-	8215 3100 5850 3100
+	8215 3100 7390 3100
 Connection ~ 5850 3100
 Wire Wire Line
@@
 Text Label 9330 2250 2    50   ~ 0
 p3
-$Comp
-L Connector:DIN-6 CN7
-U 1 1 5ED6C96C
-P 4140 5725
-F 0 "CN7" H 4140 6330 50  0000 C CNN
-F 1 "SERIAL_BUS" H 4140 6245 50  0000 C CNN
-F 2 "CommodorePlus4:Connector_DIN_Female_6Pin_3rows" H 4140 5725 50  0001 C CNN
-F 3 "http://www.mouser.com/ds/2/18/40_c091_abd_e-75918.pdf" H 4140 5725 50  0001 C CNN
-	1    4140 5725
-	1    0    0    -1
-$EndComp
-Wire Wire Line
-	3840 5825 3555 5825
 Wire Wire Line
 	3555 5825 3555 5480
@@
 Wire Wire Line
 	3555 5085 3555 5180
-$Comp
-L Device:Ferrite_Bead_Small FB1
-U 1 1 5ED7203F
-P 3680 6015
-F 0 "FB1" H 3580 6015 50  0000 R CNN
-F 1 "Ferrite_Bead_Small" H 3780 5970 50  0001 L CNN
-F 2 "LittleSixteen:Ferrite" V 3610 6015 50  0001 C CNN
-F 3 "~" H 3680 6015 50  0001 C CNN
-	1    3680 6015
-	1    0    0    -1
-$EndComp
-Wire Wire Line
-	3680 5915 3680 5625
-Wire Wire Line
-	3680 5625 3840 5625
-Wire Wire Line
-	3680 6115 3680 6225
-$Comp
-L power:GND #PWR0158
-U 1 1 5ED75A9A
-P 3680 6225
-F 0 "#PWR0158" H 3680 5975 50  0001 C CNN
-F 1 "GND" H 3685 6052 50  0000 C CNN
-F 2 "" H 3680 6225 50  0001 C CNN
-F 3 "" H 3680 6225 50  0001 C CNN
-	1    3680 6225
-	1    0    0    -1
-$EndComp
 Text Notes 4400 5335 2    50   ~ 0
 FEMALE DIN-6
-Wire Wire Line
-	4140 5425 4140 5380
-$Comp
-L Device:Ferrite_Bead_Small FB5
-U 1 1 5ED7946B
-P 4775 5380
-F 0 "FB5" V 4920 5380 50  0000 C CNN
-F 1 "Ferrite_Bead_Small" H 4875 5335 50  0001 L CNN
-F 2 "LittleSixteen:Ferrite" V 4705 5380 50  0001 C CNN
-F 3 "~" H 4775 5380 50  0001 C CNN
-	1    4775 5380
-	0    -1   -1   0
-$EndComp
 Wire Wire Line
 	4140 5380 4675 5380
@@
 Text Label 7690 5380 2    50   ~ 0
 p2
-$Comp
-L Device:Ferrite_Bead_Small FB4
-U 1 1 5ED81D59
-P 5075 5625
-F 0 "FB4" V 5220 5625 50  0000 C CNN
-F 1 "Ferrite_Bead_Small" H 5175 5580 50  0001 L CNN
-F 2 "LittleSixteen:Ferrite" V 5005 5625 50  0001 C CNN
-F 3 "~" H 5075 5625 50  0001 C CNN
-	1    5075 5625
-	0    -1   -1   0
-$EndComp
-Wire Wire Line
-	4440 5625 4975 5625
 Wire Wire Line
 	5175 5625 5800 5625
@@
 	-1   0    0    -1
 $EndComp
-$Comp
-L Device:Ferrite_Bead_Small FB3
-U 1 1 5ED88505
-P 4775 5825
-F 0 "FB3" V 4630 5825 50  0000 C CNN
-F 1 "Ferrite_Bead_Small" H 4875 5780 50  0001 L CNN
-F 2 "LittleSixteen:Ferrite" V 4705 5825 50  0001 C CNN
-F 3 "~" H 4775 5825 50  0001 C CNN
-	1    4775 5825
-	0    -1   -1   0
-$EndComp
-Wire Wire Line
-	4440 5825 4675 5825
 Wire Wire Line
 	4875 5825 5950 5825
@@
 Wire Wire Line
 	7205 5380 7790 5380
-Wire Wire Line
-	4140 6025 4140 6070
-$Comp
-L Device:Ferrite_Bead_Small FB2
-U 1 1 5ED99E91
-P 5070 6070
-F 0 "FB2" V 5215 6070 50  0000 C CNN
-F 1 "Ferrite_Bead_Small" H 5170 6025 50  0001 L CNN
-F 2 "LittleSixteen:Ferrite" V 5000 6070 50  0001 C CNN
-F 3 "~" H 5070 6070 50  0001 C CNN
-	1    5070 6070
-	0    1    1    0
-$EndComp
 Wire Wire Line
 	4140 6070 4970 6070
@@
 Text Notes 6930 2385 2    50   ~ 0
 CST_WRT
+$Comp
+L Ferrite3Pin:Ferrite_3pin FB3
+U 1 1 5E29E46B
+P 4775 5825
+F 0 "FB3" V 4660 5825 50  0000 C CNN
+F 1 "Ferrite_3pin" V 4629 5825 50  0001 C CNN
+F 2 "LittleSixteen:Ferrite" V 4705 5825 50  0001 C CNN
+F 3 "~" H 4775 5825 50  0001 C CNN
+	1    4775 5825
+	0    -1   1    0
+$EndComp
+$Comp
+L Ferrite3Pin:Ferrite_3pin FB2
+U 1 1 5E2AB049
+P 5070 6070
+F 0 "FB2" V 4955 6070 50  0000 C CNN
+F 1 "Ferrite_3pin" V 4924 6070 50  0001 C CNN
+F 2 "LittleSixteen:Ferrite" V 5000 6070 50  0001 C CNN
+F 3 "~" H 5070 6070 50  0001 C CNN
+	1    5070 6070
+	0    -1   1    0
+$EndComp
+$Comp
+L Ferrite3Pin:Ferrite_3pin FB4
+U 1 1 5E2AB69F
+P 5075 5625
+F 0 "FB4" V 4960 5625 50  0000 C CNN
+F 1 "Ferrite_3pin" V 4929 5625 50  0001 C CNN
+F 2 "LittleSixteen:Ferrite" V 5005 5625 50  0001 C CNN
+F 3 "~" H 5075 5625 50  0001 C CNN
+	1    5075 5625
+	0    -1   1    0
+$EndComp
+$Comp
+L Ferrite3Pin:Ferrite_3pin FB5
+U 1 1 5E2AC1A5
+P 4775 5380
+F 0 "FB5" V 4660 5380 50  0000 C CNN
+F 1 "Ferrite_3pin" V 4629 5380 50  0001 C CNN
+F 2 "LittleSixteen:Ferrite" V 4705 5380 50  0001 C CNN
+F 3 "~" H 4775 5380 50  0001 C CNN
+	1    4775 5380
+	0    -1   1    0
+$EndComp
+Wire Wire Line
+	4775 5480 4775 5515
+Wire Wire Line
+	4775 5515 4595 5515
+Wire Wire Line
+	4595 5515 4595 6290
+Wire Wire Line
+	4595 6290 4775 6290
+Wire Wire Line
+	5070 6290 5070 6170
+Wire Wire Line
+	4775 5925 4775 6290
+Wire Wire Line
+	5075 5725 5075 5755
+Wire Wire Line
+	5075 5755 4925 5755
+Wire Wire Line
+	4925 5755 4925 6290
+Connection ~ 4925 6290
+Wire Wire Line
+	4925 6290 5070 6290
+Connection ~ 4775 6290
+$Comp
+L power:GND #PWR0184
+U 1 1 5E2C1840
+P 4850 6345
+F 0 "#PWR0184" H 4850 6095 50  0001 C CNN
+F 1 "GND" H 4855 6172 50  0000 C CNN
+F 2 "" H 4850 6345 50  0001 C CNN
+F 3 "" H 4850 6345 50  0001 C CNN
+	1    4850 6345
+	1    0    0    -1
+$EndComp
+Wire Wire Line
+	4850 6290 4850 6345
+Wire Wire Line
+	4775 6290 4850 6290
+Connection ~ 4850 6290
+Wire Wire Line
+	4850 6290 4925 6290
+Wire Wire Line
+	4140 6025 4140 6070
+Wire Wire Line
+	4440 5825 4675 5825
+Wire Wire Line
+	4440 5625 4975 5625
+Wire Wire Line
+	4140 5425 4140 5380
+Wire Wire Line
+	3680 5625 3840 5625
+Wire Wire Line
+	3840 5825 3555 5825
+Wire Wire Line
+	3680 6290 3680 6345
+Connection ~ 3680 6290
+Wire Wire Line
+	3865 6290 3680 6290
+Wire Wire Line
+	3865 6135 3865 6290
+Wire Wire Line
+	3780 6135 3865 6135
+$Comp
+L Ferrite3Pin:Ferrite_3pin FB1
+U 1 1 5E2BCB55
+P 3680 6135
+F 0 "FB1" H 3580 6135 50  0000 R CNN
+F 1 "Ferrite_3pin" V 3534 6135 50  0001 C CNN
+F 2 "LittleSixteen:Ferrite" V 3610 6135 50  0001 C CNN
+F 3 "~" H 3680 6135 50  0001 C CNN
+	1    3680 6135
+	1    0    0    -1
+$EndComp
+$Comp
+L power:GND #PWR0158
+U 1 1 5ED75A9A
+P 3680 6345
+F 0 "#PWR0158" H 3680 6095 50  0001 C CNN
+F 1 "GND" H 3685 6172 50  0000 C CNN
+F 2 "" H 3680 6345 50  0001 C CNN
+F 3 "" H 3680 6345 50  0001 C CNN
+	1    3680 6345
+	1    0    0    -1
+$EndComp
+Wire Wire Line
+	3680 6235 3680 6290
+Wire Wire Line
+	3680 6035 3680 5625
+$Comp
+L Connector:DIN-6 CN7
+U 1 1 5ED6C96C
+P 4140 5725
+F 0 "CN7" H 4140 6330 50  0000 C CNN
+F 1 "SERIAL_BUS" H 4140 6245 50  0000 C CNN
+F 2 "CommodorePlus4:Connector_DIN_Female_6Pin_3rows" H 4140 5725 50  0001 C CNN
+F 3 "http://www.mouser.com/ds/2/18/40_c091_abd_e-75918.pdf" H 4140 5725 50  0001 C CNN
+	1    4140 5725
+	1    0    0    -1
+$EndComp
+$Comp
+L Ferrite3Pin:Ferrite_3pin FB19
+U 1 1 5E31356C
+P 7390 2560
+F 0 "FB19" V 7245 2560 50  0000 C CNN
+F 1 "Ferrite_3pin" V 7244 2560 50  0001 C CNN
+F 2 "LittleSixteen:Ferrite" V 7320 2560 50  0001 C CNN
+F 3 "~" H 7390 2560 50  0001 C CNN
+	1    7390 2560
+	0    -1   1    0
+$EndComp
+Wire Wire Line
+	7390 2660 7390 3100
+Connection ~ 7390 3100
+Wire Wire Line
+	7390 3100 5850 3100
 Wire Bus Line
 	7890 4845 7890 5725

Commit message: Working on PCB...
Parts:
- Q5: footprint Package_TO_SOT_THT:TO-220-3_Horizontal_TabDown -> Package_TO_SOT_THT:TO-220-3_Horizontal_TabUp
Changed lines of the file:
@@
 F 0 "Q5" H 8007 2296 50  0000 L CNN
 F 1 "2SD880" H 8007 2205 50  0000 L CNN
-F 2 "Package_TO_SOT_THT:TO-220-3_Horizontal_TabDown" H 8015 2175 50  0001 L CIN
+F 2 "Package_TO_SOT_THT:TO-220-3_Horizontal_TabUp" H 8015 2175 50  0001 L CIN
 F 3 "http://pdf.datasheetcatalog.com/datasheet/sanyo/ds_pdf_e/2SB631.pdf" H 7815 2250 50  0001 L CNN
 	1    7815 2250
