File: datasette.sch (KiCad schematic (older format))
At the start: 35 parts, among them CN3 CASSETTE, CN7 SERIAL_BUS, Q5 2SD880, U11 74LS125, U9 74LS06, U91 DT1042

Commit message: Add better ESD protection for Datassette Connector and some notes
Parts:
- added U92: DT1042, Package_SO:TSOP-6_1.65x3.05mm_P0.95mm, symbol DT1042:DT1042
- D93: Notes (none) -> Only mount if using a 6510 CPU
- D94, D95: Notes (none) -> Do not mount if U92 is mounted
- R93: Notes (none) -> Only mount if using a 6510 CPU (But shouldn't hurt anyway)
Connections:
- net GND: now also U92.2 (GND)
- net VCC: now also U92.5 (VCC)
- net cn3_p6: now reaches CN3.6, FB17.1
- net cn3_p6: now also U92.6 (I/O4)
- net cn3_p7: now reaches CN3.7, FB18.1
- net cn3_p7: now also U92.1 (I/O1)
- net prot1 renamed cn3_p5
- net cn3_p5: now also U92.3 (I/O2)
- no-connect marks 0 -> 1
Other:
- note added: "These offer better ESD protection\nthan the retrofitted diodes, but use\nan SMT component. Mount only one\nor the other, at your preference."
- note removed: "This offers better ESD protection\nthan the retrofitted diodes, but it's\nan SMT component. Use only one\nor the other, at your preference."
Changed lines of the file:
@@
 Sheet 7 12
 Title "LittleSixteen"
-Date "2021-11-17"
+Date "2021-11-21"
 Rev "2git"
 Comp "SukkoPera"
@@
 F 2 "Diode_THT:D_DO-35_SOD27_P5.08mm_Vertical_KathodeUp" H 2715 2120 50  0001 C CNN
 F 3 "~" H 2715 2120 50  0001 C CNN
+F 4 "Do not mount if U92 is mounted" H 2715 2120 50  0001 C CNN "Notes"
 	1    2715 2120
 	0    -1   1    0
@@
 F 2 "Diode_THT:D_DO-35_SOD27_P5.08mm_Vertical_KathodeUp" H 2715 2695 50  0001 C CNN
 F 3 "~" H 2715 2695 50  0001 C CNN
+F 4 "Do not mount if U92 is mounted" H 2715 2695 50  0001 C CNN "Notes"
 	1    2715 2695
 	0    -1   1    0
@@
 F 2 "Resistor_THT:R_Axial_DIN0207_L6.3mm_D2.5mm_P5.08mm_Vertical" V 9630 1380 50  0001 C CNN
 F 3 "~" H 9700 1380 50  0001 C CNN
+F 4 "Only mount if using a 6510 CPU (But shouldn't hurt anyway)" H 9700 1380 50  0001 C CNN "Notes"
 	1    9700 1380
 	-1   0    0    1
@@
 F 2 "Diode_THT:D_DO-35_SOD27_P5.08mm_Vertical_KathodeUp" H 9490 1380 50  0001 C CNN
 F 3 "~" H 9490 1380 50  0001 C CNN
+F 4 "Only mount if using a 6510 CPU" H 9490 1380 50  0001 C CNN "Notes"
 	1    9490 1380
 	0    -1   1    0
@@
 Wire Wire Line
 	9375 5295 9045 5295
-Text Label 3750 2425 0    50   ~ 0
-prot1
+Text Label 3710 2425 0    50   ~ 0
+cn3_p5
 Text Label 6670 5620 0    50   ~ 0
 cn7_p5
@@
 Text Label 9045 4995 0    50   ~ 0
 cn7_p6
+Text Notes 9075 6315 0    50   ~ 0
+These offer better ESD protection\nthan the retrofitted diodes, but use\nan SMT component. Mount only one\nor the other, at your preference.
+Text Label 5265 2325 0    50   ~ 0
+cn3_p6
+Text Label 4690 1535 0    50   ~ 0
+cn3_p7
+$Comp
+L DT1042:DT1042 U92
+U 1 1 62324DC8
+P 9975 3360
+F 0 "U92" H 10303 3406 50  0000 L CNN
+F 1 "DT1042" H 10303 3315 50  0000 L CNN
+F 2 "Package_SO:TSOP-6_1.65x3.05mm_P0.95mm" H 9825 2810 50  0001 C CNN
+F 3 "" H 9825 2810 50  0001 C CNN
+F 4 "Optional, protects Serial port from ESD" H 9975 3360 50  0001 C CNN "Notes"
+	1    9975 3360
+	1    0    0    -1
+$EndComp
+Wire Wire Line
+	9975 2910 9975 2840
+Wire Wire Line
+	9975 3810 9975 3885
+$Comp
+L power:VCC #PWR0211
+U 1 1 62325334
+P 9975 2840
+F 0 "#PWR0211" H 9975 2690 50  0001 C CNN
+F 1 "VCC" H 9992 3013 50  0000 C CNN
+F 2 "" H 9975 2840 50  0001 C CNN
+F 3 "" H 9975 2840 50  0001 C CNN
+	1    9975 2840
+	-1   0    0    -1
+$EndComp
+$Comp
+L power:GND #PWR0212
+U 1 1 6232533E
+P 9975 3885
+F 0 "#PWR0212" H 9975 3635 50  0001 C CNN
+F 1 "GND" H 9980 3712 50  0000 C CNN
+F 2 "" H 9975 3885 50  0001 C CNN
+F 3 "" H 9975 3885 50  0001 C CNN
+	1    9975 3885
+	1    0    0    -1
+$EndComp
+Wire Wire Line
+	9375 3210 9045 3210
+Wire Wire Line
+	9375 3310 9045 3310
+Wire Wire Line
+	9375 3510 9045 3510
+Text Label 9045 3510 0    50   ~ 0
+cn3_p6
+Text Label 9045 3310 0    50   ~ 0
+cn3_p5
+Text Label 9045 3210 0    50   ~ 0
+cn3_p7
+NoConn ~ 9375 3410
+Wire Notes Line
+	8925 2565 10795 2565
+Wire Notes Line
+	10795 2565 10795 6410
+Wire Notes Line
+	10795 6410 8925 6410
+Wire Notes Line
+	8925 6410 8925 2565
 Wire Bus Line
 	3075 4640 3075 5520
-Text Notes 9075 6315 0    50   ~ 0
-This offers better ESD protection\nthan the retrofitted diodes, but it's\nan SMT component. Use only one\nor the other, at your preference.
 $EndSCHEMATC

Commit message: Add internal Tape/IEC connector
Parts:
- added J90: CONN_TAPE_DRIVE, Connector_PinHeader_2.54mm:PinHeader_2x07_P2.54mm_Vertical, symbol Connector_Generic:Conn_02x07_Odd_Even
Connections:
- net GND: now also J90.11 (Pin_11), J90.13 (Pin_13), J90.14 (Pin_14)
- net VCC: now also J90.1 (Pin_1), J90.2 (Pin_2)
- net tape_mtr: now reaches CN3.3, FB19.1
- net tape_mtr: now also J90.9 (Pin_9)
- net iec_srq: now reaches CN7.1, R102.2
- net iec_srq: now also J90.4 (Pin_4)
- net cn3_p5 renamed tape_read
- net tape_read: now also J90.7 (Pin_7)
- net cn3_p6 renamed tape_wr
- net tape_wr: now also J90.5 (Pin_5)
- net cn3_p7 renamed tape_sense
- net tape_sense: now also J90.3 (Pin_3)
- net cn7_p3 renamed iec_atn
- net iec_atn: now also J90.6 (Pin_6)
- net cn7_p4 renamed iec_clk
- net iec_clk: now also J90.8 (Pin_8)
- net cn7_p5 renamed iec_dat
- net iec_dat: now also J90.10 (Pin_10)
- net cn7_p6 renamed iec_rst
- net iec_rst: now also J90.12 (Pin_12)
Other:
- note added: "This connector has all the Tape and IEC\nsignals and can be used to implement\nan internal SD2IEC or Tapuino."
- moved on the sheet: U92
Changed lines of the file:
@@
 	9375 5295 9045 5295
 Text Label 3710 2425 0    50   ~ 0
-cn3_p5
+tape_read
 Text Label 6670 5620 0    50   ~ 0
-cn7_p5
+iec_dat
 Text Label 6670 5420 0    50   ~ 0
-cn7_p4
+iec_clk
 Text Label 6670 5175 0    50   ~ 0
-cn7_p3
+iec_atn
 Text Label 6670 5865 0    50   ~ 0
-cn7_p6
+iec_rst
 Text Label 9045 5195 0    50   ~ 0
-cn7_p5
+iec_dat
 Text Label 9045 5295 0    50   ~ 0
-cn7_p3
+iec_atn
 Text Label 9045 5095 0    50   ~ 0
-cn7_p4
+iec_clk
 Text Label 9045 4995 0    50   ~ 0
-cn7_p6
+iec_rst
 Text Notes 9075 6315 0    50   ~ 0
 These offer better ESD protection\nthan the retrofitted diodes, but use\nan SMT component. Mount only one\nor the other, at your preference.
 Text Label 5265 2325 0    50   ~ 0
-cn3_p6
+tape_wr
 Text Label 4690 1535 0    50   ~ 0
-cn3_p7
+tape_sense
 $Comp
 L DT1042:DT1042 U92
 U 1 1 62324DC8
-P 9975 3360
-F 0 "U92" H 10303 3406 50  0000 L CNN
-F 1 "DT1042" H 10303 3315 50  0000 L CNN
-F 2 "Package_SO:TSOP-6_1.65x3.05mm_P0.95mm" H 9825 2810 50  0001 C CNN
-F 3 "" H 9825 2810 50  0001 C CNN
-F 4 "Optional, protects Serial port from ESD" H 9975 3360 50  0001 C CNN "Notes"
-	1    9975 3360
-	1    0    0    -1
-$EndComp
-Wire Wire Line
-	9975 2910 9975 2840
-Wire Wire Line
-	9975 3810 9975 3885
+P 10070 3355
+F 0 "U92" H 10398 3401 50  0000 L CNN
+F 1 "DT1042" H 10398 3310 50  0000 L CNN
+F 2 "Package_SO:TSOP-6_1.65x3.05mm_P0.95mm" H 9920 2805 50  0001 C CNN
+F 3 "" H 9920 2805 50  0001 C CNN
+F 4 "Optional, protects Serial port from ESD" H 10070 3355 50  0001 C CNN "Notes"
+	1    10070 3355
+	1    0    0    -1
+$EndComp
+Wire Wire Line
+	10070 2905 10070 2835
+Wire Wire Line
+	10070 3805 10070 3880
 $Comp
 L power:VCC #PWR0211
 U 1 1 62325334
-P 9975 2840
-F 0 "#PWR0211" H 9975 2690 50  0001 C CNN
-F 1 "VCC" H 9992 3013 50  0000 C CNN
-F 2 "" H 9975 2840 50  0001 C CNN
-F 3 "" H 9975 2840 50  0001 C CNN
-	1    9975 2840
+P 10070 2835
+F 0 "#PWR0211" H 10070 2685 50  0001 C CNN
+F 1 "VCC" H 10087 3008 50  0000 C CNN
+F 2 "" H 10070 2835 50  0001 C CNN
+F 3 "" H 10070 2835 50  0001 C CNN
+	1    10070 2835
 	-1   0    0    -1
 $EndComp
@@
 L power:GND #PWR0212
 U 1 1 6232533E
-P 9975 3885
-F 0 "#PWR0212" H 9975 3635 50  0001 C CNN
-F 1 "GND" H 9980 3712 50  0000 C CNN
-F 2 "" H 9975 3885 50  0001 C CNN
-F 3 "" H 9975 3885 50  0001 C CNN
-	1    9975 3885
-	1    0    0    -1
-$EndComp
-Wire Wire Line
-	9375 3210 9045 3210
-Wire Wire Line
-	9375 3310 9045 3310
-Wire Wire Line
-	9375 3510 9045 3510
-Text Label 9045 3510 0    50   ~ 0
-cn3_p6
-Text Label 9045 3310 0    50   ~ 0
-cn3_p5
-Text Label 9045 3210 0    50   ~ 0
-cn3_p7
-NoConn ~ 9375 3410
+P 10070 3880
+F 0 "#PWR0212" H 10070 3630 50  0001 C CNN
+F 1 "GND" H 10075 3707 50  0000 C CNN
+F 2 "" H 10070 3880 50  0001 C CNN
+F 3 "" H 10070 3880 50  0001 C CNN
+	1    10070 3880
+	1    0    0    -1
+$EndComp
+Wire Wire Line
+	9470 3205 9020 3205
+Wire Wire Line
+	9470 3305 9020 3305
+Wire Wire Line
+	9470 3505 9020 3505
+Text Label 9020 3505 0    50   ~ 0
+tape_wr
+Text Label 9020 3305 0    50   ~ 0
+tape_read
+Text Label 9020 3205 0    50   ~ 0
+tape_sense
+NoConn ~ 9470 3405
 Wire Notes Line
 	8925 2565 10795 2565
@@
 Wire Notes Line
 	8925 6410 8925 2565
+Wire Wire Line
+	1140 6745 685  6745
+Wire Wire Line
+	1140 6845 685  6845
+Wire Wire Line
+	1140 6945 685  6945
+Wire Wire Line
+	1140 7045 685  7045
+Wire Wire Line
+	1140 7145 685  7145
+Wire Wire Line
+	2100 6845 1640 6845
+Wire Wire Line
+	2100 6945 1640 6945
+Wire Wire Line
+	2100 7045 1640 7045
+Wire Wire Line
+	2100 7145 1640 7145
+Wire Wire Line
+	1140 7245 685  7245
+Wire Wire Line
+	685  7245 685  7345
+$Comp
+L power:GND #PWR0213
+U 1 1 623B7B36
+P 685 7515
+F 0 "#PWR0213" H 685 7265 50  0001 C CNN
+F 1 "GND" H 690 7342 50  0000 C CNN
+F 2 "" H 685 7515 50  0001 C CNN
+F 3 "" H 685 7515 50  0001 C CNN
+	1    685  7515
+	1    0    0    -1
+$EndComp
+$Comp
+L power:VCC #PWR0214
+U 1 1 623B7EDA
+P 685 6620
+F 0 "#PWR0214" H 685 6470 50  0001 C CNN
+F 1 "VCC" H 702 6793 50  0000 C CNN
+F 2 "" H 685 6620 50  0001 C CNN
+F 3 "" H 685 6620 50  0001 C CNN
+	1    685  6620
+	1    0    0    -1
+$EndComp
+Text Label 5265 2425 0    50   ~ 0
+tape_mtr
+Text Label 685  6945 0    50   ~ 0
+tape_wr
+Text Label 685  7145 0    50   ~ 0
+tape_mtr
+Text Label 685  6845 0    50   ~ 0
+tape_sense
+Text Label 685  7045 0    50   ~ 0
+tape_read
+Text Label 2100 6945 2    50   ~ 0
+iec_atn
+Text Label 2100 7045 2    50   ~ 0
+iec_clk
+Text Label 2100 7145 2    50   ~ 0
+iec_dat
+Text Label 2100 7245 2    50   ~ 0
+iec_rst
+Text Label 8090 5620 1    50   ~ 0
+iec_srq
+Text Label 2100 6845 2    50   ~ 0
+iec_srq
+Wire Wire Line
+	685  6620 685  6745
+Wire Wire Line
+	1640 6745 2095 6745
+$Comp
+L power:VCC #PWR0215
+U 1 1 62461BF9
+P 2095 6620
+F 0 "#PWR0215" H 2095 6470 50  0001 C CNN
+F 1 "VCC" H 2112 6793 50  0000 C CNN
+F 2 "" H 2095 6620 50  0001 C CNN
+F 3 "" H 2095 6620 50  0001 C CNN
+	1    2095 6620
+	-1   0    0    -1
+$EndComp
+Wire Wire Line
+	2095 6620 2095 6745
+$Comp
+L Connector_Generic:Conn_02x07_Odd_Even J90
+U 1 1 62482A9D
+P 1340 7045
+F 0 "J90" H 1390 7562 50  0000 C CNN
+F 1 "CONN_TAPE_DRIVE" H 1390 7471 50  0000 C CNN
+F 2 "Connector_PinHeader_2.54mm:PinHeader_2x07_P2.54mm_Vertical" H 1340 7045 50  0001 C CNN
+F 3 "~" H 1340 7045 50  0001 C CNN
+	1    1340 7045
+	1    0    0    -1
+$EndComp
+Wire Wire Line
+	1140 7345 685  7345
+Connection ~ 685  7345
+Wire Wire Line
+	685  7345 685  7515
+$Comp
+L power:GND #PWR0216
+U 1 1 624971E6
+P 2095 7515
+F 0 "#PWR0216" H 2095 7265 50  0001 C CNN
+F 1 "GND" H 2100 7342 50  0000 C CNN
+F 2 "" H 2095 7515 50  0001 C CNN
+F 3 "" H 2095 7515 50  0001 C CNN
+	1    2095 7515
+	-1   0    0    -1
+$EndComp
+Wire Wire Line
+	1640 7345 2095 7345
+Wire Wire Line
+	2095 7345 2095 7515
+Wire Wire Line
+	1640 7245 2100 7245
 Wire Bus Line
 	3075 4640 3075 5520
+Text Notes 2260 7435 0    50   ~ 0
+This connector has all the Tape and IEC\nsignals and can be used to implement\nan internal SD2IEC or Tapuino.
 $EndSCHEMATC

Commit message: Improve power zones
Parts:
- RP1: Notes (none) -> Bussed
Changed lines of the file:
@@
 F 2 "Resistor_THT:R_Array_SIP6" V 5880 4725 50  0001 C CNN
 F 3 "~" H 5950 4725 50  0001 C CNN
+F 4 "Bussed" H 5950 4725 50  0001 C CNN "Notes"
 	2    5950 4725
 	-1   0    0    -1
@@
 F 2 "Resistor_THT:R_Array_SIP6" V 5735 4725 50  0001 C CNN
 F 3 "~" H 5805 4725 50  0001 C CNN
+F 4 "Bussed" H 5805 4725 50  0001 C CNN "Notes"
 	3    5805 4725
 	-1   0    0    -1
@@
 F 2 "Resistor_THT:R_Array_SIP6" V 5585 4725 50  0001 C CNN
 F 3 "~" H 5655 4725 50  0001 C CNN
+F 4 "Bussed" H 5655 4725 50  0001 C CNN "Notes"
 	4    5655 4725
 	-1   0    0    -1
@@
 F 2 "Resistor_THT:R_Array_SIP6" V 5435 4725 50  0001 C CNN
 F 3 "~" H 5505 4725 50  0001 C CNN
+F 4 "Bussed" H 5505 4725 50  0001 C CNN "Notes"
 	5    5505 4725
 	-1   0    0    -1
