File: exp_port.sch (KiCad schematic (older format))
At the start: 4 parts, among them CN1 EXPANSION_CONNECTOR

Commit message: Add crystal
Parts:
- FB38, FB39, FB40: footprint (none) -> CSeventeen:Ferrite
Changed lines of the file:
@@
 F 0 "FB38" V 6760 3390 50  0000 C CNN
 F 1 "Ferrite_Bead_Small" V 6759 3390 50  0001 C CNN
-F 2 "" V 6835 3390 50  0001 C CNN
+F 2 "CSeventeen:Ferrite" V 6835 3390 50  0001 C CNN
 F 3 "~" H 6905 3390 50  0001 C CNN
 	1    6905 3390
@@
 F 0 "FB40" V 4625 4090 50  0000 C CNN
 F 1 "Ferrite_Bead_Small" V 4619 4090 50  0001 C CNN
-F 2 "" V 4695 4090 50  0001 C CNN
+F 2 "CSeventeen:Ferrite" V 4695 4090 50  0001 C CNN
 F 3 "~" H 4765 4090 50  0001 C CNN
 	1    4765 4090
@@
 F 0 "FB39" V 6960 3490 50  0000 C CNN
 F 1 "Ferrite_Bead_Small" V 6959 3490 50  0001 C CNN
-F 2 "" V 7035 3490 50  0001 C CNN
+F 2 "CSeventeen:Ferrite" V 7035 3490 50  0001 C CNN
 F 3 "~" H 7105 3490 50  0001 C CNN
 	1    7105 3490

Commit message: Use 3d models from github.com/StormTrooper/Commodore-Plus4
Parts:
- CN1: footprint (none) -> CommodorePlus4:50Pin_Edge_Connector
Changed lines of the file:
@@
 F 0 "CN1" H 5855 5855 50  0000 C CNN
 F 1 "EXPANSION_CONNECTOR" H 5855 5764 50  0000 C CNN
-F 2 "" H 5855 2640 50  0001 C CNN
+F 2 "CommodorePlus4:50Pin_Edge_Connector" H 5855 2640 50  0001 C CNN
 F 3 "DOCUMENTATION" H 5855 2540 50  0001 C CNN
 	1    5855 4290

Commit message: CSeventeen -> LittleSixteen (PCB)
Parts:
- FB38, FB39, FB40: footprint CSeventeen:Ferrite -> LittleSixteen:Ferrite
Changed lines of the file:
@@
 F 0 "FB38" V 6760 3390 50  0000 C CNN
 F 1 "Ferrite_Bead_Small" V 6759 3390 50  0001 C CNN
-F 2 "CSeventeen:Ferrite" V 6835 3390 50  0001 C CNN
+F 2 "LittleSixteen:Ferrite" V 6835 3390 50  0001 C CNN
 F 3 "~" H 6905 3390 50  0001 C CNN
 	1    6905 3390
@@
 F 0 "FB40" V 4625 4090 50  0000 C CNN
 F 1 "Ferrite_Bead_Small" V 4619 4090 50  0001 C CNN
-F 2 "CSeventeen:Ferrite" V 4695 4090 50  0001 C CNN
+F 2 "LittleSixteen:Ferrite" V 4695 4090 50  0001 C CNN
 F 3 "~" H 4765 4090 50  0001 C CNN
 	1    4765 4090
@@
 F 0 "FB39" V 6960 3490 50  0000 C CNN
 F 1 "Ferrite_Bead_Small" V 6959 3490 50  0001 C CNN
-F 2 "CSeventeen:Ferrite" V 7035 3490 50  0001 C CNN
+F 2 "LittleSixteen:Ferrite" V 7035 3490 50  0001 C CNN
 F 3 "~" H 7105 3490 50  0001 C CNN
 	1    7105 3490

Commit message: Working on PCB...
Parts:
- CN1: footprint CommodorePlus4:50Pin_Edge_Connector -> LittleSixteen:50Pin_Edge_Connector
Changed lines of the file:
@@
 F 0 "CN1" H 5855 5855 50  0000 C CNN
 F 1 "EXPANSION_CONNECTOR" H 5855 5764 50  0000 C CNN
-F 2 "CommodorePlus4:50Pin_Edge_Connector" H 5855 2640 50  0001 C CNN
+F 2 "LittleSixteen:50Pin_Edge_Connector" H 5855 2640 50  0001 C CNN
 F 3 "DOCUMENTATION" H 5855 2540 50  0001 C CNN
 	1    5855 4290
