File: exp_port.sch (KiCad schematic (older format))
At the start: 5 parts, among them CN1 EXPANSION_CONNECTOR

Commit message: Rationalize BOM There should be no significant changes on both schematics on PCB, just some values and something on the silkscreen
Parts:
- C94: value 100n/25V -> 100n; MouserPN (none) -> 810-FG28X7R1H104KNT0
- FB38, FB39, FB40: value Ferrite_Bead_Small -> DSS1NB32A271Q91A; footprint LittleSixteen:Ferrite -> LittleSixteen:EMI_Filter; symbol ferrite_bead_small:Ferrite_Bead_Small -> emi_filter_3pin:EMI_Filter_3Pin
Changed lines of the file:
@@
 	6700 5490 6700 3090
 $Comp
-L ferrite_bead_small:Ferrite_Bead_Small FB38
+L emi_filter_3pin:EMI_Filter_3Pin FB38
 U 1 1 5E9793EF
 P 6905 3390
 F 0 "FB38" V 6760 3390 50  0000 C CNN
-F 1 "Ferrite_Bead_Small" V 6759 3390 50  0001 C CNN
-F 2 "LittleSixteen:Ferrite" V 6835 3390 50  0001 C CNN
+F 1 "DSS1NB32A271Q91A" V 6759 3390 50  0001 C CNN
+F 2 "LittleSixteen:EMI_Filter" V 6835 3390 50  0001 C CNN
 F 3 "~" H 6905 3390 50  0001 C CNN
 	1    6905 3390
@@
 	6805 3390 6605 3390
 $Comp
-L ferrite_bead_small:Ferrite_Bead_Small FB40
+L emi_filter_3pin:EMI_Filter_3Pin FB40
 U 1 1 5E979856
 P 4765 4090
 F 0 "FB40" V 4625 4090 50  0000 C CNN
-F 1 "Ferrite_Bead_Small" V 4619 4090 50  0001 C CNN
-F 2 "LittleSixteen:Ferrite" V 4695 4090 50  0001 C CNN
+F 1 "DSS1NB32A271Q91A" V 4619 4090 50  0001 C CNN
+F 2 "LittleSixteen:EMI_Filter" V 4695 4090 50  0001 C CNN
 F 3 "~" H 4765 4090 50  0001 C CNN
 	1    4765 4090
@@
 	7440 3490 7205 3490
 $Comp
-L ferrite_bead_small:Ferrite_Bead_Small FB39
+L emi_filter_3pin:EMI_Filter_3Pin FB39
 U 1 1 5E982F3B
 P 7105 3490
 F 0 "FB39" V 6960 3490 50  0000 C CNN
-F 1 "Ferrite_Bead_Small" V 6959 3490 50  0001 C CNN
-F 2 "LittleSixteen:Ferrite" V 7035 3490 50  0001 C CNN
+F 1 "DSS1NB32A271Q91A" V 6959 3490 50  0001 C CNN
+F 2 "LittleSixteen:EMI_Filter" V 7035 3490 50  0001 C CNN
 F 3 "~" H 7105 3490 50  0001 C CNN
 	1    7105 3490
@@
 AR Path="/5E6A379E/6349BFDB" Ref="C94"  Part="1"
 F 0 "C94" H 10395 4161 50  0000 L CNN
-F 1 "100n/25V" H 10395 4070 50  0000 L CNN
+F 1 "100n" H 10395 4070 50  0000 L CNN
 F 2 "Capacitor_THT:C_Disc_D8.0mm_W2.5mm_P5.00mm" H 10318 3965 50  0001 C CNN
 F 3 "~" H 10280 4115 50  0001 C CNN
+F 4 "810-FG28X7R1H104KNT0" H 10280 4115 50  0001 C CNN "MouserPN"
 	1    10280 4115
 	1    0    0    -1

Commit message: Rationalize capacitor footprints & BOM
Parts:
- CN1: Notes (none) -> Must be recovered from an old board : (
Changed lines of the file:
@@
 F 2 "LittleSixteen:50Pin_Edge_Connector" H 5855 2640 50  0001 C CNN
 F 3 "DOCUMENTATION" H 5855 2540 50  0001 C CNN
+F 4 "Must be recovered from an old board : (" H 5855 4290 50  0001 C CNN "Notes"
 	1    5855 4290
 	1    0    0    -1

Commit message: Replace /BRESET on Expansion Port and User Port with /RESET This was an oversight we probably introduced in V3 which makes it impossible for the Expansion Port and User Port to reset the machine through the RESET pin. The /BRESET line only went to the IEC Port in the original machine, which means that "Serial button dongles" cannot reset the machine, unlike on the C64. Maybe we should introduce a jumper for that?
Connections:
- net ~BRESET renamed ~RESET
Changed lines of the file:
@@
 Sheet 8 14
 Title "LittleSixteen"
-Date "2021-12-05"
+Date "2024-07-21"
 Rev "4git"
 Comp "SukkoPera"
@@
 	6605 3290 7440 3290
 Text GLabel 7440 3290 2    50   Input ~ 0
-~BRESET
+~RESET
 Text GLabel 7230 3190 2    50   Input ~ 0
 C1_LOW

Commit message: Switch to polyfuses on userport and to ferrites for FB38/39/40
Parts:
- FB38, FB39, FB40: value DSS1NB32A271Q91A -> 28L0138-80R-10
Changed lines of the file:
@@
 P 6905 3390
 F 0 "FB38" V 6760 3390 50  0000 C CNN
-F 1 "DSS1NB32A271Q91A" V 6759 3390 50  0001 C CNN
+F 1 "28L0138-80R-10" V 6759 3390 50  0001 C CNN
 F 2 "LittleSixteen:EMI_Filter" V 6835 3390 50  0001 C CNN
 F 3 "~" H 6905 3390 50  0001 C CNN
@@
 P 4765 4090
 F 0 "FB40" V 4625 4090 50  0000 C CNN
-F 1 "DSS1NB32A271Q91A" V 4619 4090 50  0001 C CNN
+F 1 "28L0138-80R-10" V 4619 4090 50  0001 C CNN
 F 2 "LittleSixteen:EMI_Filter" V 4695 4090 50  0001 C CNN
 F 3 "~" H 4765 4090 50  0001 C CNN
@@
 P 7105 3490
 F 0 "FB39" V 6960 3490 50  0000 C CNN
-F 1 "DSS1NB32A271Q91A" V 6959 3490 50  0001 C CNN
+F 1 "28L0138-80R-10" V 6959 3490 50  0001 C CNN
 F 2 "LittleSixteen:EMI_Filter" V 7035 3490 50  0001 C CNN
 F 3 "~" H 7105 3490 50  0001 C CNN

Commit message: Fix some P/Ns
Parts:
- FB38, FB39, FB40: value 28L0138-80R-10 -> DO NOT MOUNT; MouserPN (none) -> ---
Changed lines of the file:
@@
 P 6905 3390
 F 0 "FB38" V 6760 3390 50  0000 C CNN
-F 1 "28L0138-80R-10" V 6759 3390 50  0001 C CNN
+F 1 "DO NOT MOUNT" V 6759 3390 50  0001 C CNN
 F 2 "LittleSixteen:EMI_Filter" V 6835 3390 50  0001 C CNN
 F 3 "~" H 6905 3390 50  0001 C CNN
+F 4 "---" H 6905 3390 50  0001 C CNN "MouserPN"
 	1    6905 3390
 	0    1    1    0
@@
 P 4765 4090
 F 0 "FB40" V 4625 4090 50  0000 C CNN
-F 1 "28L0138-80R-10" V 4619 4090 50  0001 C CNN
+F 1 "DO NOT MOUNT" V 4619 4090 50  0001 C CNN
 F 2 "LittleSixteen:EMI_Filter" V 4695 4090 50  0001 C CNN
 F 3 "~" H 4765 4090 50  0001 C CNN
+F 4 "---" H 4765 4090 50  0001 C CNN "MouserPN"
 	1    4765 4090
 	0    -1   1    0
@@
 P 7105 3490
 F 0 "FB39" V 6960 3490 50  0000 C CNN
-F 1 "28L0138-80R-10" V 6959 3490 50  0001 C CNN
+F 1 "DO NOT MOUNT" V 6959 3490 50  0001 C CNN
 F 2 "LittleSixteen:EMI_Filter" V 7035 3490 50  0001 C CNN
 F 3 "~" H 7105 3490 50  0001 C CNN
+F 4 "---" H 7105 3490 50  0001 C CNN "MouserPN"
 	1    7105 3490
 	0    1    1    0

Commit message: Minor fixes + P/N updates
Parts:
- CN1: MouserPN (none) -> :)
Changed lines of the file:
@@
 F 3 "DOCUMENTATION" H 5855 2540 50  0001 C CNN
 F 4 "Must be recovered from an old board : (" H 5855 4290 50  0001 C CNN "Notes"
+F 5 ":)" H 5855 4290 50  0001 C CNN "MouserPN"
 	1    5855 4290
 	1    0    0    -1
