File: misc.sch (KiCad schematic (older format))
At the start: 15 parts, among them CN8 POWER_INPUT, CN9 LED_CONNECTOR, SW1 POWER_SWITCH, U11 74LS125, U9 74LS06

Commit message: Start working on PCB
Parts:
- C2: footprint (none) -> Capacitor_THT:CP_Radial_D7.5mm_P2.50mm
- R10: footprint (none) -> Resistor_THT:R_Box_L26.0mm_W5.0mm_P20.00mm
- R14: footprint (none) -> Resistor_THT:R_Axial_DIN0207_L6.3mm_D2.5mm_P5.08mm_Vertical
Changed lines of the file:
@@
 F 0 "R14" H 10110 2651 50  0000 L CNN
 F 1 "470" H 10110 2560 50  0000 L CNN
-F 2 "" V 9970 2605 50  0001 C CNN
+F 2 "Resistor_THT:R_Axial_DIN0207_L6.3mm_D2.5mm_P5.08mm_Vertical" V 9970 2605 50  0001 C CNN
 F 3 "~" H 10040 2605 50  0001 C CNN
 	1    10040 2605
@@
 F 0 "C2" H 6650 3286 50  0000 L CNN
 F 1 "47u/25V" H 6650 3195 50  0000 L CNN
-F 2 "" H 6535 3240 50  0001 C CNN
+F 2 "Capacitor_THT:CP_Radial_D7.5mm_P2.50mm" H 6535 3240 50  0001 C CNN
 F 3 "~" H 6535 3240 50  0001 C CNN
 	1    6535 3240
@@
 F 0 "R10" V 5798 2300 50  0000 C CNN
 F 1 "20/5W" V 5889 2300 50  0000 C CNN
-F 2 "" V 5935 2300 50  0001 C CNN
+F 2 "Resistor_THT:R_Box_L26.0mm_W5.0mm_P20.00mm" V 5935 2300 50  0001 C CNN
 F 3 "~" H 6005 2300 50  0001 C CNN
 	1    6005 2300

Commit message: Add pin headers
Parts:
- CN9: footprint (none) -> Connector_PinHeader_2.54mm:PinHeader_1x03_P2.54mm_Vertical
Changed lines of the file:
@@
 F 0 "CN9" H 9708 3266 50  0000 C CNN
 F 1 "LED_CONNECTOR" H 9708 3175 50  0000 C CNN
-F 2 "" H 9600 2985 50  0001 C CNN
+F 2 "Connector_PinHeader_2.54mm:PinHeader_1x03_P2.54mm_Vertical" H 9600 2985 50  0001 C CNN
 F 3 "~" H 9600 2985 50  0001 C CNN
 	1    9600 2985

Commit message: Add ceramics
Parts:
- C1, C200, C34: footprint (none) -> Capacitor_THT:C_Disc_D8.0mm_W2.5mm_P5.00mm
Changed lines of the file:
@@
 F 0 "C1" H 5600 3286 50  0000 L CNN
 F 1 "100n" H 5600 3195 50  0000 L CNN
-F 2 "" H 5523 3090 50  0001 C CNN
+F 2 "Capacitor_THT:C_Disc_D8.0mm_W2.5mm_P5.00mm" H 5523 3090 50  0001 C CNN
 F 3 "~" H 5485 3240 50  0001 C CNN
 	1    5485 3240
@@
 F 0 "C200" H 3097 3316 50  0000 L CNN
 F 1 "220n" H 3097 3225 50  0000 L CNN
-F 2 "" H 3005 3270 50  0001 C CNN
+F 2 "Capacitor_THT:C_Disc_D8.0mm_W2.5mm_P5.00mm" H 3005 3270 50  0001 C CNN
 F 3 "~" H 3005 3270 50  0001 C CNN
 	1    3005 3270
@@
 F 0 "C34" H 4850 5831 50  0000 L CNN
 F 1 "100n" H 4850 5740 50  0000 L CNN
-F 2 "" H 4773 5635 50  0001 C CNN
+F 2 "Capacitor_THT:C_Disc_D8.0mm_W2.5mm_P5.00mm" H 4773 5635 50  0001 C CNN
 F 3 "~" H 4735 5785 50  0001 C CNN
 	1    4735 5785

Commit message: Add diodes
Parts:
- D11: footprint (none) -> Diode_THT:D_DO-41_SOD81_P5.08mm_Vertical_KathodeUp
Changed lines of the file:
@@
 F 0 "D11" H 6005 2841 50  0000 C CNN
 F 1 "1N914" H 6005 2750 50  0000 C CNN
-F 2 "" H 6005 2625 50  0001 C CNN
+F 2 "Diode_THT:D_DO-41_SOD81_P5.08mm_Vertical_KathodeUp" H 6005 2625 50  0001 C CNN
 F 3 "~" H 6005 2625 50  0001 C CNN
 	1    6005 2625

Commit message: Use 3d models from github.com/StormTrooper/Commodore-Plus4
Parts:
- SW1: footprint (none) -> CommodorePlus4:Switch-Rocker
Changed lines of the file:
@@
 F 0 "SW1" H 4305 3401 50  0000 C CNN
 F 1 "POWER_SWITCH" H 4305 3310 50  0000 C CNN
-F 2 "" H 4305 3170 60  0001 C CNN
+F 2 "CommodorePlus4:Switch-Rocker" H 4305 3170 60  0001 C CNN
 F 3 "" H 4305 3170 60  0000 C CNN
 	1    4305 3170

Commit message: Working on PCB...
Parts:
- F1: footprint (none) -> CommodorePlus4:Fuseholder_Cylinder-6.3x32mm
Changed lines of the file:
@@
 F 0 "F1" V 4673 3120 50  0000 C CNN
 F 1 "FUSE" V 4764 3120 50  0000 C CNN
-F 2 "" V 4800 3120 50  0001 C CNN
+F 2 "CommodorePlus4:Fuseholder_Cylinder-6.3x32mm" V 4800 3120 50  0001 C CNN
 F 3 "~" H 4870 3120 50  0001 C CNN
 	1    4870 3120

Commit message: Laid out data bus and muuuuch more stuff
Parts:
- CN8: footprint (none) -> Connector_BarrelJack:BarrelJack_Horizontal
Changed lines of the file:
@@
 F 0 "CN8" H 2432 2953 50  0000 C CNN
 F 1 "POWER_INPUT" H 2432 3044 50  0000 C CNN
-F 2 "" H 2425 3230 50  0001 C CNN
+F 2 "Connector_BarrelJack:BarrelJack_Horizontal" H 2425 3230 50  0001 C CNN
 F 3 "~" H 2425 3230 50  0001 C CNN
 	1    2375 3270

Commit message: One last connection missing!
Parts:
- L3: footprint (none) -> CommodorePlus4:Noise_Filter
- SW1: footprint CommodorePlus4:Switch-Rocker -> LittleSixteen:Switch-Rocker
Changed lines of the file:
@@
 F 0 "L3" H 3610 3600 50  0000 C CNN
 F 1 "LINE_FILTER" H 3610 3490 50  0000 C CNN
-F 2 "" H 3610 3310 50  0001 C CNN
+F 2 "CommodorePlus4:Noise_Filter" H 3610 3310 50  0001 C CNN
 F 3 "~" H 3610 3310 50  0001 C CNN
 	1    3610 3270
@@
 F 0 "SW1" H 4305 3401 50  0000 C CNN
 F 1 "POWER_SWITCH" H 4305 3310 50  0000 C CNN
-F 2 "CommodorePlus4:Switch-Rocker" H 4305 3170 60  0001 C CNN
+F 2 "LittleSixteen:Switch-Rocker" H 4305 3170 60  0001 C CNN
 F 3 "" H 4305 3170 60  0000 C CNN
 	1    4305 3170
