File: ted.sch (KiCad schematic (older format))
At the start: 20 parts, among them Q1 2SC1815, Q2 2SC1815, U1 MOS_7360_TED, Y1 Crystal

Commit message: Start working on PCB
Parts:
- C3: footprint (none) -> Capacitor_THT:CP_Radial_D6.3mm_P2.50mm
- R1, R2, R3, R4, R5, R6, R7: footprint (none) -> Resistor_THT:R_Axial_DIN0207_L6.3mm_D2.5mm_P5.08mm_Vertical
Changed lines of the file:
@@
 F 0 "C3" H 5871 7131 50  0000 R CNN
 F 1 "10u/25V" H 5871 7040 50  0000 R CNN
-F 2 "" H 5985 7085 50  0001 C CNN
+F 2 "Capacitor_THT:CP_Radial_D6.3mm_P2.50mm" H 5985 7085 50  0001 C CNN
 F 3 "~" H 5985 7085 50  0001 C CNN
 	1    5985 7085
@@
 F 0 "R2" H 2320 4146 50  0000 L CNN
 F 1 "4.7k" H 2320 4055 50  0000 L CNN
-F 2 "" V 2180 4100 50  0001 C CNN
+F 2 "Resistor_THT:R_Axial_DIN0207_L6.3mm_D2.5mm_P5.08mm_Vertical" V 2180 4100 50  0001 C CNN
 F 3 "~" H 2250 4100 50  0001 C CNN
 	1    2250 4100
@@
 F 0 "R1" H 2320 2666 50  0000 L CNN
 F 1 "10k" H 2320 2575 50  0000 L CNN
-F 2 "" V 2180 2620 50  0001 C CNN
+F 2 "Resistor_THT:R_Axial_DIN0207_L6.3mm_D2.5mm_P5.08mm_Vertical" V 2180 2620 50  0001 C CNN
 F 3 "~" H 2250 2620 50  0001 C CNN
 	1    2250 2620
@@
 F 0 "R4" H 3370 4146 50  0000 L CNN
 F 1 "220" H 3370 4055 50  0000 L CNN
-F 2 "" V 3230 4100 50  0001 C CNN
+F 2 "Resistor_THT:R_Axial_DIN0207_L6.3mm_D2.5mm_P5.08mm_Vertical" V 3230 4100 50  0001 C CNN
 F 3 "~" H 3300 4100 50  0001 C CNN
 	1    3300 4100
@@
 F 0 "R3" H 3370 2666 50  0000 L CNN
 F 1 "470" H 3370 2575 50  0000 L CNN
-F 2 "" V 3230 2620 50  0001 C CNN
+F 2 "Resistor_THT:R_Axial_DIN0207_L6.3mm_D2.5mm_P5.08mm_Vertical" V 3230 2620 50  0001 C CNN
 F 3 "~" H 3300 2620 50  0001 C CNN
 	1    3300 2620
@@
 F 0 "R5" H 4420 2666 50  0000 L CNN
 F 1 "18k" H 4420 2575 50  0000 L CNN
-F 2 "" V 4280 2620 50  0001 C CNN
+F 2 "Resistor_THT:R_Axial_DIN0207_L6.3mm_D2.5mm_P5.08mm_Vertical" V 4280 2620 50  0001 C CNN
 F 3 "~" H 4350 2620 50  0001 C CNN
 	1    4350 2620
@@
 F 0 "R6" H 4420 3481 50  0000 L CNN
 F 1 "1.5k" H 4420 3390 50  0000 L CNN
-F 2 "" V 4280 3435 50  0001 C CNN
+F 2 "Resistor_THT:R_Axial_DIN0207_L6.3mm_D2.5mm_P5.08mm_Vertical" V 4280 3435 50  0001 C CNN
 F 3 "~" H 4350 3435 50  0001 C CNN
 	1    4350 3435
@@
 F 0 "R7" H 4935 2666 50  0000 L CNN
 F 1 "470" H 4935 2575 50  0000 L CNN
-F 2 "" V 4795 2620 50  0001 C CNN
+F 2 "Resistor_THT:R_Axial_DIN0207_L6.3mm_D2.5mm_P5.08mm_Vertical" V 4795 2620 50  0001 C CNN
 F 3 "~" H 4865 2620 50  0001 C CNN
 	1    4865 2620

Commit message: Add pin headers
Parts:
- TP1: footprint (none) -> TestPoint:TestPoint_Pad_D2.0mm
Changed lines of the file:
@@
 F 0 "TP1" H 6000 2945 50  0000 C CNN
 F 1 "CLOCK_TESTPOINT" H 6000 2854 50  0000 C CNN
-F 2 "" H 6200 2620 50  0001 C CNN
+F 2 "TestPoint:TestPoint_Pad_D2.0mm" H 6200 2620 50  0001 C CNN
 F 3 "~" H 6200 2620 50  0001 C CNN
 	1    6000 2620

Commit message: Add ceramics
Parts:
- C12, C13, C14, C15, C21, C32: footprint (none) -> Capacitor_THT:C_Disc_D8.0mm_W2.5mm_P5.00mm
Changed lines of the file:
@@
 F 0 "C21" H 6595 7131 50  0000 L CNN
 F 1 "100n" H 6595 7040 50  0000 L CNN
-F 2 "" H 6518 6935 50  0001 C CNN
+F 2 "Capacitor_THT:C_Disc_D8.0mm_W2.5mm_P5.00mm" H 6518 6935 50  0001 C CNN
 F 3 "~" H 6480 7085 50  0001 C CNN
 	1    6480 7085
@@
 F 0 "C12" H 1855 4156 50  0000 L CNN
 F 1 "22p" H 1855 4065 50  0000 L CNN
-F 2 "" H 1778 3960 50  0001 C CNN
+F 2 "Capacitor_THT:C_Disc_D8.0mm_W2.5mm_P5.00mm" H 1778 3960 50  0001 C CNN
 F 3 "~" H 1740 4110 50  0001 C CNN
 	1    1740 4110
@@
 F 0 "C13" H 2865 3726 50  0000 L CNN
 F 1 "220p" H 2865 3635 50  0000 L CNN
-F 2 "" H 2788 3530 50  0001 C CNN
+F 2 "Capacitor_THT:C_Disc_D8.0mm_W2.5mm_P5.00mm" H 2788 3530 50  0001 C CNN
 F 3 "~" H 2750 3680 50  0001 C CNN
 	1    2750 3680
@@
 F 0 "C14" H 2865 4146 50  0000 L CNN
 F 1 "150p" H 2865 4055 50  0000 L CNN
-F 2 "" H 2788 3950 50  0001 C CNN
+F 2 "Capacitor_THT:C_Disc_D8.0mm_W2.5mm_P5.00mm" H 2788 3950 50  0001 C CNN
 F 3 "~" H 2750 4100 50  0001 C CNN
 	1    2750 4100
@@
 F 0 "C15" V 3603 3130 50  0000 C CNN
 F 1 "10p" V 3694 3130 50  0000 C CNN
-F 2 "" H 3893 2980 50  0001 C CNN
+F 2 "Capacitor_THT:C_Disc_D8.0mm_W2.5mm_P5.00mm" H 3893 2980 50  0001 C CNN
 F 3 "~" H 3855 3130 50  0001 C CNN
 	1    3855 3130
@@
 F 0 "C32" H 5685 2661 50  0000 L CNN
 F 1 "100p" H 5685 2570 50  0000 L CNN
-F 2 "" H 5608 2465 50  0001 C CNN
+F 2 "Capacitor_THT:C_Disc_D8.0mm_W2.5mm_P5.00mm" H 5608 2465 50  0001 C CNN
 F 3 "~" H 5570 2615 50  0001 C CNN
 	1    5570 2615

Commit message: Add diodes
Parts:
- Q1, Q2: footprint Package_TO_SOT_THT:TO-92_Inline -> Package_TO_SOT_THT:TO-92_Inline_Wide
Changed lines of the file:
@@
 F 0 "Q1" H 3390 3426 50  0000 L CNN
 F 1 "2SC1815" H 3390 3335 50  0000 L CNN
-F 2 "Package_TO_SOT_THT:TO-92_Inline" H 3400 3305 50  0001 L CIN
+F 2 "Package_TO_SOT_THT:TO-92_Inline_Wide" H 3400 3305 50  0001 L CIN
 F 3 "https://media.digikey.com/pdf/Data%20Sheets/Toshiba%20PDFs/2SC1815.pdf" H 3200 3380 50  0001 L CNN
 	1    3200 3380
@@
 F 0 "Q2" H 4955 3176 50  0000 L CNN
 F 1 "2SC1815" H 4955 3085 50  0000 L CNN
-F 2 "Package_TO_SOT_THT:TO-92_Inline" H 4965 3055 50  0001 L CIN
+F 2 "Package_TO_SOT_THT:TO-92_Inline_Wide" H 4965 3055 50  0001 L CIN
 F 3 "https://media.digikey.com/pdf/Data%20Sheets/Toshiba%20PDFs/2SC1815.pdf" H 4765 3130 50  0001 L CNN
 	1    4765 3130

Commit message: Laid out data bus and muuuuch more stuff
Parts:
- CT1: footprint (none) -> LittleSixteen:VariCap
Changed lines of the file:
@@
 F 0 "CT1" H 1440 4156 50  0000 L CNN
 F 1 "40p" H 1440 4065 50  0000 L CNN
-F 2 "" H 1325 4110 50  0001 C CNN
+F 2 "LittleSixteen:VariCap" H 1325 4110 50  0001 C CNN
 F 3 "~" H 1325 4110 50  0001 C CNN
 	1    1325 4110
