File: ted.sch (KiCad schematic (older format))
At the start: 22 parts, among them CN13 CONN_TED_OUTPUT, Q1 2SC1815, Q2 2SC1815, U1 MOS_7360_TED, Y1 17.734475M

Commit message: Rationalize capacitor footprints & BOM
Parts:
- C3: footprint Capacitor_THT:CP_Radial_D6.3mm_P2.50mm -> Capacitor_THT:CP_Radial_D5.0mm_P2.00mm; MouserPN (none) -> 710-860010672009
- C96: MouserPN 710-860010472002 -> 710-860010672009
- R1: MouserPN (none) -> 603-MFR-25FTF52-10K
- TP1: MouserPN (none) -> ---
- U1: MouserPN (none) -> :)
- Y1: MouserPN (none) -> 710-830003298B
Changed lines of the file:
@@
 F 2 "LittleSixteen:DIP-48_W15.24mm_Socket_LongPads" H 8185 2700 50  0001 C CNN
 F 3 "DOCUMENTATION" H 8185 2700 50  0001 C CNN
+F 4 ":)" H 8185 2700 50  0001 C CNN "MouserPN"
 	1    8185 2700
 	1    0    0    -1
@@
 F 0 "C3" H 5871 7131 50  0000 R CNN
 F 1 "10u/25V" H 5871 7040 50  0000 R CNN
-F 2 "Capacitor_THT:CP_Radial_D6.3mm_P2.50mm" H 5985 7085 50  0001 C CNN
+F 2 "Capacitor_THT:CP_Radial_D5.0mm_P2.00mm" H 5985 7085 50  0001 C CNN
 F 3 "~" H 5985 7085 50  0001 C CNN
+F 4 "710-860010672009" H 5985 7085 50  0001 C CNN "MouserPN"
 	1    5985 7085
 	1    0    0    -1
@@
 F 2 "Resistor_THT:R_Axial_DIN0207_L6.3mm_D2.5mm_P5.08mm_Vertical" V 2180 2620 50  0001 C CNN
 F 3 "~" H 2250 2620 50  0001 C CNN
+F 4 "603-MFR-25FTF52-10K" H 2250 2620 50  0001 C CNN "MouserPN"
 	1    2250 2620
 	1    0    0    -1
@@
 F 2 "TestPoint:TestPoint_Pad_D2.0mm" H 6200 2620 50  0001 C CNN
 F 3 "~" H 6200 2620 50  0001 C CNN
+F 4 "---" H 6000 2620 50  0001 C CNN "MouserPN"
 	1    6000 2620
 	1    0    0    -1
@@
 F 3 "~" H 1740 3655 50  0001 C CNN
 F 4 "Use 14.31818M for NTSC, +/- 70ppm, CL = 32p" H 1740 3655 50  0001 C CNN "Notes"
+F 5 "710-830003298B" H 1740 3655 50  0001 C CNN "MouserPN"
 	1    1740 3655
 	0    -1   1    0
@@
 F 2 "Capacitor_THT:CP_Radial_D5.0mm_P2.00mm" H 8045 5265 50  0001 C CNN
 F 3 "~" H 8045 5265 50  0001 C CNN
-F 4 "710-860010472002" H 8045 5265 50  0001 C CNN "MouserPN"
+F 4 "710-860010672009" H 8045 5265 50  0001 C CNN "MouserPN"
 F 5 "10u" H 8045 5265 50  0001 C CNN "Value"
 	1    8045 5265

Commit message: Add note on some components
Parts:
- C96: Notes (none) -> Audio cap recommended
Changed lines of the file:
@@
 F 4 "710-860010672009" H 8045 5265 50  0001 C CNN "MouserPN"
 F 5 "10u" H 8045 5265 50  0001 C CNN "Value"
+F 6 "Audio cap recommended" H 8045 5265 50  0001 C CNN "Notes"
 	1    8045 5265
 	0    -1   -1   0

Commit message: Make C83 10uF
Parts:
- C96: MouserPN 710-860010672009 -> (none)
Changed lines of the file:
@@
 F 2 "Capacitor_THT:CP_Radial_D5.0mm_P2.00mm" H 8045 5265 50  0001 C CNN
 F 3 "~" H 8045 5265 50  0001 C CNN
-F 4 "710-860010672009" H 8045 5265 50  0001 C CNN "MouserPN"
+F 4 "" H 8045 5265 50  0001 C CNN "MouserPN"
 F 5 "10u" H 8045 5265 50  0001 C CNN "Value"
 F 6 "Audio cap recommended" H 8045 5265 50  0001 C CNN "Notes"

Commit message: Add footprint for single oscillator
Parts:
- added JP2: JMP_OSC_GND, Jumper:SolderJumper-2_P1.3mm_Open_RoundedPad1.0x1.5mm, symbol Device:Jumper_NO_Small
- added X1: OSC_DIP14, LittleSixteen:Oscillator_DIP-8+14, symbol Oscillator:CXO_DIP14
Connections:
- net GND: now also JP2.1, X1.7 (GND)
- net VCC: now also X1.14 (Vcc)
- net clock_in: now reaches Q2.2 (C), R7.2, TP1.1, U1.14 (CLKIN)
- net clock_in: now also X1.8 (OUT)
- new net: JP2.2, X1.1 (EN)
Other:
- note added: "ALTERNATIVE DISCRETE OSCILLATOR"
- note added: "This can replace the whole circuit above.\n\nIf a DFO is mounted, PAL/NTSC switching\nbecomes a breeze ;)"
Changed lines of the file:
@@
 Sheet 3 14
 Title "LittleSixteen"
-Date "2020-01-03"
+Date "2024-02-05"
 Rev "4git"
 Comp "SukkoPera"
@@
 	1    0    0    -1
 $EndComp
+$Comp
+L Oscillator:CXO_DIP14 X1
+U 1 1 65CA419C
+P 3300 6040
+F 0 "X1" H 3490 6300 50  0000 R CNN
+F 1 "OSC_DIP14" H 3775 5780 50  0000 R CNN
+F 2 "LittleSixteen:Oscillator_DIP-8+14" H 3750 5690 50  0001 C CNN
+F 3 "http://cdn-reichelt.de/documents/datenblatt/B400/OSZI.pdf" H 3200 6040 50  0001 C CNN
+	1    3300 6040
+	1    0    0    -1
+$EndComp
+$Comp
+L power:GND #PWR031
+U 1 1 65CA9785
+P 3300 6385
+F 0 "#PWR031" H 3300 6135 50  0001 C CNN
+F 1 "GND" H 3305 6212 50  0000 C CNN
+F 2 "" H 3300 6385 50  0001 C CNN
+F 3 "" H 3300 6385 50  0001 C CNN
+	1    3300 6385
+	1    0    0    -1
+$EndComp
+Wire Wire Line
+	3300 6340 3300 6385
+Wire Wire Line
+	3300 5740 3300 5635
+$Comp
+L power:VCC #PWR025
+U 1 1 65CAECEF
+P 3300 5635
+F 0 "#PWR025" H 3300 5485 50  0001 C CNN
+F 1 "VCC" H 3317 5808 50  0000 C CNN
+F 2 "" H 3300 5635 50  0001 C CNN
+F 3 "" H 3300 5635 50  0001 C CNN
+	1    3300 5635
+	1    0    0    -1
+$EndComp
+Text Label 6000 2850 0    50   ~ 0
+clock_in
+Text Label 4095 6040 2    50   ~ 0
+clock_in
+Wire Wire Line
+	3600 6040 4095 6040
+$Comp
+L Device:Jumper_NO_Small JP2
+U 1 1 65CBEEFF
+P 2750 6040
+F 0 "JP2" H 2750 6225 50  0000 C CNN
+F 1 "JMP_OSC_GND" H 2750 6134 50  0000 C CNN
+F 2 "Jumper:SolderJumper-2_P1.3mm_Open_RoundedPad1.0x1.5mm" H 2750 6040 50  0001 C CNN
+F 3 "~" H 2750 6040 50  0001 C CNN
+	1    2750 6040
+	1    0    0    -1
+$EndComp
+Wire Wire Line
+	2850 6040 3000 6040
+Wire Wire Line
+	2650 6040 2485 6040
+$Comp
+L power:GND #PWR029
+U 1 1 65CCA0B2
+P 2485 6385
+F 0 "#PWR029" H 2485 6135 50  0001 C CNN
+F 1 "GND" H 2490 6212 50  0000 C CNN
+F 2 "" H 2485 6385 50  0001 C CNN
+F 3 "" H 2485 6385 50  0001 C CNN
+	1    2485 6385
+	1    0    0    -1
+$EndComp
+Wire Wire Line
+	2485 6040 2485 6385
+Text Notes 2450 7070 0    50   ~ 0
+This can replace the whole circuit above.\n\nIf a DFO is mounted, PAL/NTSC switching\nbecomes a breeze ;)
+Text Notes 2640 5305 0    50   ~ 0
+ALTERNATIVE DISCRETE OSCILLATOR
 Wire Bus Line
 	6865 885  6865 1650

Commit message: Minor fixes + P/N updates
Parts:
- C3: MouserPN 710-860010672009 -> 710-860010572002
- C96: MouserPN (none) -> 710-860010572002
- JP2: MouserPN (none) -> ---
Changed lines of the file:
@@
 F 2 "Capacitor_THT:CP_Radial_D5.0mm_P2.00mm" H 5985 7085 50  0001 C CNN
 F 3 "~" H 5985 7085 50  0001 C CNN
-F 4 "710-860010672009" H 5985 7085 50  0001 C CNN "MouserPN"
+F 4 "710-860010572002" H 5985 7085 50  0001 C CNN "MouserPN"
 	1    5985 7085
 	1    0    0    -1
@@
 F 2 "Capacitor_THT:CP_Radial_D5.0mm_P2.00mm" H 8045 5265 50  0001 C CNN
 F 3 "~" H 8045 5265 50  0001 C CNN
-F 4 "" H 8045 5265 50  0001 C CNN "MouserPN"
+F 4 "710-860010572002" H 8045 5265 50  0001 C CNN "MouserPN"
 F 5 "10u" H 8045 5265 50  0001 C CNN "Value"
 F 6 "Audio cap recommended" H 8045 5265 50  0001 C CNN "Notes"
@@
 F 2 "Jumper:SolderJumper-2_P1.3mm_Open_RoundedPad1.0x1.5mm" H 2750 6040 50  0001 C CNN
 F 3 "~" H 2750 6040 50  0001 C CNN
+F 4 "---" H 2750 6040 50  0001 C CNN "MouserPN"
 	1    2750 6040
 	1    0    0    -1
