File: joysticks.sch (KiCad schematic (older format))
At the start: 39 parts, among them CN4 JOY1, CN5 JOY2, U11 74LS125, U17 74AHCT244, U18 74AHCT244

Commit message: Add ESD protection on joystick ports
Parts:
- added U93, U94, U95: DT1042, Package_SO:TSOP-6_1.65x3.05mm_P0.95mm, symbol DT1042:DT1042
Connections:
- net labels added: f1d, f1f, f1l, f1r, f1u, f2d, f2f, f2l, f2r, f2u
- wire segments 187 -> 203
- no-connect marks 6 -> 8
Changed lines of the file:
@@
 Sheet 11 12
 Title "LittleSixteen"
-Date "2021-11-22"
+Date "2021-11-28"
 Rev "3git"
 Comp "SukkoPera"
@@
 Wire Wire Line
 	5530 1480 5530 1805
-Text Notes 3020 7615 0    50   ~ 0
+Text Notes 11095 1440 2    50   ~ 0
 This was one of the weakest spots of the C16, where the\nTED chip pins were directly exposed outside through the\njoystick ports.\n\nAdding a buffer will protect the TED from ESD, and TVS\ndiodes could do even more. This is basically Levente\nHársfalvi's design integrated into the C16. Please see:\nhttp://www.zimmers.net/anonftp/pub/cbm/documents/projects/interfaces/plus4joy/plus4joy.html\n\nWe can also consider to replace the MiniDIN-8 ports with\nD-SUB 9 ones.
 $Comp
@@
 Text GLabel 10185 1705 2    50   Output ~ 0
 k[0..7]
-Text Notes 650  7680 0    50   ~ 0
+Text Notes 555  7680 0    50   ~ 0
 Joystick Connector Pinout\nMiniDIN-8\n1 Up\n2 Down\n3 Left\n4 Right\n5 +5V\n6 Fire\n7 Ground\n8 Select\n\nAll signals are joy to C16, except Select
 Wire Wire Line
@@
 Wire Wire Line
 	3340 4040 3340 3925
+$Comp
+L DT1042:DT1042 U?
+U 1 1 61A59722
+P 3190 6910
+AR Path="/5ECB474B/61A59722" Ref="U?"  Part="1"
+AR Path="/61BCD018/61A59722" Ref="U93"  Part="1"
+F 0 "U93" H 3518 6956 50  0000 L CNN
+F 1 "DT1042" H 3518 6865 50  0000 L CNN
+F 2 "Package_SO:TSOP-6_1.65x3.05mm_P0.95mm" H 3040 6360 50  0001 C CNN
+F 3 "" H 3040 6360 50  0001 C CNN
+F 4 "Optional, protects Joystick port from ESD" H 3190 6910 50  0001 C CNN "Notes"
+	1    3190 6910
+	1    0    0    -1
+$EndComp
+Wire Wire Line
+	3190 6460 3190 6390
+Wire Wire Line
+	3190 7360 3190 7435
+$Comp
+L power:VCC #PWR?
+U 1 1 61A5972A
+P 3190 6390
+AR Path="/5ECB474B/61A5972A" Ref="#PWR?"  Part="1"
+AR Path="/61BCD018/61A5972A" Ref="#PWR0218"  Part="1"
+F 0 "#PWR0218" H 3190 6240 50  0001 C CNN
+F 1 "VCC" H 3207 6563 50  0000 C CNN
+F 2 "" H 3190 6390 50  0001 C CNN
+F 3 "" H 3190 6390 50  0001 C CNN
+	1    3190 6390
+	-1   0    0    -1
+$EndComp
+$Comp
+L power:GND #PWR?
+U 1 1 61A59730
+P 3190 7435
+AR Path="/5ECB474B/61A59730" Ref="#PWR?"  Part="1"
+AR Path="/61BCD018/61A59730" Ref="#PWR0219"  Part="1"
+F 0 "#PWR0219" H 3190 7185 50  0001 C CNN
+F 1 "GND" H 3195 7262 50  0000 C CNN
+F 2 "" H 3190 7435 50  0001 C CNN
+F 3 "" H 3190 7435 50  0001 C CNN
+	1    3190 7435
+	1    0    0    -1
+$EndComp
+Wire Wire Line
+	2590 6760 2400 6760
+Wire Wire Line
+	2590 6860 2400 6860
+Wire Wire Line
+	2590 7060 2400 7060
+Wire Wire Line
+	2590 6960 2400 6960
+$Comp
+L DT1042:DT1042 U?
+U 1 1 61A6C798
+P 6200 6920
+AR Path="/5ECB474B/61A6C798" Ref="U?"  Part="1"
+AR Path="/61BCD018/61A6C798" Ref="U94"  Part="1"
+F 0 "U94" H 6528 6966 50  0000 L CNN
+F 1 "DT1042" H 6528 6875 50  0000 L CNN
+F 2 "Package_SO:TSOP-6_1.65x3.05mm_P0.95mm" H 6050 6370 50  0001 C CNN
+F 3 "" H 6050 6370 50  0001 C CNN
+F 4 "Optional, protects Joystick port from ESD" H 6200 6920 50  0001 C CNN "Notes"
+	1    6200 6920
+	1    0    0    -1
+$EndComp
+Wire Wire Line
+	6200 6470 6200 6400
+Wire Wire Line
+	6200 7370 6200 7445
+$Comp
+L power:VCC #PWR?
+U 1 1 61A6CFAC
+P 6200 6400
+AR Path="/5ECB474B/61A6CFAC" Ref="#PWR?"  Part="1"
+AR Path="/61BCD018/61A6CFAC" Ref="#PWR0220"  Part="1"
+F 0 "#PWR0220" H 6200 6250 50  0001 C CNN
+F 1 "VCC" H 6217 6573 50  0000 C CNN
+F 2 "" H 6200 6400 50  0001 C CNN
+F 3 "" H 6200 6400 50  0001 C CNN
+	1    6200 6400
+	-1   0    0    -1
+$EndComp
+$Comp
+L power:GND #PWR?
+U 1 1 61A6CFB6
+P 6200 7445
+AR Path="/5ECB474B/61A6CFB6" Ref="#PWR?"  Part="1"
+AR Path="/61BCD018/61A6CFB6" Ref="#PWR0221"  Part="1"
+F 0 "#PWR0221" H 6200 7195 50  0001 C CNN
+F 1 "GND" H 6205 7272 50  0000 C CNN
+F 2 "" H 6200 7445 50  0001 C CNN
+F 3 "" H 6200 7445 50  0001 C CNN
+	1    6200 7445
+	1    0    0    -1
+$EndComp
+Wire Wire Line
+	5600 7070 5445 7070
+Wire Wire Line
+	5600 6970 5445 6970
+$Comp
+L DT1042:DT1042 U?
+U 1 1 61A78456
+P 4650 6915
+AR Path="/5ECB474B/61A78456" Ref="U?"  Part="1"
+AR Path="/61BCD018/61A78456" Ref="U95"  Part="1"
+F 0 "U95" H 4978 6961 50  0000 L CNN
+F 1 "DT1042" H 4978 6870 50  0000 L CNN
+F 2 "Package_SO:TSOP-6_1.65x3.05mm_P0.95mm" H 4500 6365 50  0001 C CNN
+F 3 "" H 4500 6365 50  0001 C CNN
+F 4 "Optional, protects Joystick port from ESD" H 4650 6915 50  0001 C CNN "Notes"
+	1    4650 6915
+	1    0    0    -1
+$EndComp
+Wire Wire Line
+	4650 6465 4650 6395
+Wire Wire Line
+	4650 7365 4650 7440
+$Comp
+L power:VCC #PWR?
+U 1 1 61A78C9E
+P 4650 6395
+AR Path="/5ECB474B/61A78C9E" Ref="#PWR?"  Part="1"
+AR Path="/61BCD018/61A78C9E" Ref="#PWR0222"  Part="1"
+F 0 "#PWR0222" H 4650 6245 50  0001 C CNN
+F 1 "VCC" H 4667 6568 50  0000 C CNN
+F 2 "" H 4650 6395 50  0001 C CNN
+F 3 "" H 4650 6395 50  0001 C CNN
+	1    4650 6395
+	-1   0    0    -1
+$EndComp
+$Comp
+L power:GND #PWR?
+U 1 1 61A78CA8
+P 4650 7440
+AR Path="/5ECB474B/61A78CA8" Ref="#PWR?"  Part="1"
+AR Path="/61BCD018/61A78CA8" Ref="#PWR0223"  Part="1"
+F 0 "#PWR0223" H 4650 7190 50  0001 C CNN
+F 1 "GND" H 4655 7267 50  0000 C CNN
+F 2 "" H 4650 7440 50  0001 C CNN
+F 3 "" H 4650 7440 50  0001 C CNN
+	1    4650 7440
+	1    0    0    -1
+$EndComp
+Wire Wire Line
+	4050 6765 3880 6765
+Wire Wire Line
+	4050 6865 3880 6865
+Wire Wire Line
+	4050 7065 3880 7065
+Wire Wire Line
+	4050 6965 3880 6965
+Text Label 4425 2255 0    50   ~ 0
+f1u
+Text Label 4425 2155 0    50   ~ 0
+f1l
+Text Label 4425 2355 0    50   ~ 0
+f1r
+Text Label 4425 2055 0    50   ~ 0
+f1f
+Text Label 3705 2255 0    50   ~ 0
+f1d
+Text Label 5445 6970 0    50   ~ 0
+f2d
+Text Label 2400 6760 0    50   ~ 0
+f1d
+Text Label 2400 6860 0    50   ~ 0
+f1u
+Text Label 2400 7060 0    50   ~ 0
+f1r
+Text Label 2400 6960 0    50   ~ 0
+f1f
+Text Label 4425 4930 0    50   ~ 0
+f2u
+Text Label 3705 4930 0    50   ~ 0
+f2d
+Text Label 4425 5030 0    50   ~ 0
+f2r
+Text Label 4425 4730 0    50   ~ 0
+f2f
+Text Label 4425 4830 0    50   ~ 0
+f2l
+Text Label 5445 7070 0    50   ~ 0
+f1l
+NoConn ~ 5600 6770
+NoConn ~ 5600 6870
+Text Label 3880 6765 0    50   ~ 0
+f2u
+Text Label 3880 6865 0    50   ~ 0
+f2l
+Text Label 3880 6965 0    50   ~ 0
+f2f
+Text Label 3880 7065 0    50   ~ 0
+f2r
 Wire Bus Line
 	9685 1705 9685 4880

Commit message: Tidy up silkscreen
Parts:
- U17, U18: value 74AHCT244 -> 74LS244
Changed lines of the file:
@@
 P 6705 2305
 F 0 "U17" H 6935 2960 50  0000 C CNN
-F 1 "74AHCT244" H 6975 1645 50  0000 C CNN
+F 1 "74LS244" H 6975 1645 50  0000 C CNN
 F 2 "Package_DIP:DIP-20_W7.62mm_Socket_LongPads" H 6705 2305 50  0001 C CNN
 F 3 "https://assets.nexperia.com/documents/data-sheet/74AHC_AHCT244.pdf" H 6705 2305 50  0001 C CNN
@@
 P 6700 4980
 F 0 "U18" H 6930 5635 50  0000 C CNN
-F 1 "74AHCT244" H 6970 4320 50  0000 C CNN
+F 1 "74LS244" H 6970 4320 50  0000 C CNN
 F 2 "Package_DIP:DIP-20_W7.62mm_Socket_LongPads" H 6700 4980 50  0001 C CNN
 F 3 "https://assets.nexperia.com/documents/data-sheet/74AHC_AHCT244.pdf" H 6700 4980 50  0001 C CNN

Commit message: Various minor fixes
Parts:
- renumbered JD1 to JP1, JD2 to JP2
Other:
- note added: "ADDITIONAL CURRENT-\nLIMITING RESISTOR"
- note added: "The JP1 and JP2 jumpers are not present\nin the original schematics but I have traced\nthem on my board. They are labeled "D1" and\n"D2", I have renamed them to avoid conflicts\nwith the diodes bearing the same labels.\n\nTheir purpose seems to be able to enable the\njoysticks after passing through the keyboard\ndriver. Since it seems the latter was introduced\nlate in the x264 architecture, mayb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"
- note removed: "The JD1 and JD2 jumpers are not present\nin the original schematics but I have traced\nthem on my board. They are labeled "D1" and\n"D2", I have renamed them to avoid conflicts\nwith the diodes bearing the same labels.\n\nTheir purpose seems to be able to enable the\njoysticks after passing through the keyboard\ndriver. Since it seems the latter was introduced\nlate in the x264 architecture, mayb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"
Changed lines of the file:
@@
 Sheet 11 12
 Title "LittleSixteen"
-Date "2021-11-28"
+Date "2021-11-29"
 Rev "3git"
 Comp "SukkoPera"
@@
 The (apparently)\nodd connections\nhere are to\nsimplify routing!
 $Comp
-L Jumper:Jumper_3_Bridged12 JD1
+L Jumper:Jumper_3_Bridged12 JP1
 U 1 1 61F59301
 P 2390 5480
-F 0 "JD1" V 2344 5547 50  0000 L CNN
+F 0 "JP1" V 2344 5547 50  0000 L CNN
 F 1 "JOY2_SELECT" V 2435 5547 50  0000 L CNN
 F 2 "LittleSixteen:SolderJumper2x" H 2390 5480 50  0001 C CNN
@@
 	2540 2805 2655 2805
 $Comp
-L Jumper:Jumper_3_Bridged12 JD2
+L Jumper:Jumper_3_Bridged12 JP2
 U 1 1 61F9FE8A
 P 2390 2805
-F 0 "JD2" V 2344 2872 50  0000 L CNN
+F 0 "JP2" V 2344 2872 50  0000 L CNN
 F 1 "JOY1_SELECT" V 2435 2872 50  0000 L CNN
 F 2 "LittleSixteen:SolderJumper2x" H 2390 2805 50  0001 C CNN
@@
 Wire Bus Line
 	1560 2255 1560 4930
-Text Notes 2800 2090 2    50   ~ 0
-The JD1 and JD2 jumpers are not present\nin the original schematics but I have traced\nthem on my board. They are labeled "D1" and\n"D2", I have renamed them to avoid conflicts\nwith the diodes bearing the same labels.\n\nTheir purpose seems to be able to enable the\njoysticks after passing through the keyboard\ndriver. Since it seems  the latter was introduced\nlate in the x264 architecture, maybe the\ndesigners weren't sure what was best and kept\nboth possibilities.
+Text Notes 2575 4575 2    50   ~ 0
+The JP1 and JP2 jumpers are not present\nin the original schematics but I have traced\nthem on my board. They are labeled "D1" and\n"D2", I have renamed them to avoid conflicts\nwith the diodes bearing the same labels.\n\nTheir purpose seems to be able to enable the\njoysticks after passing through the keyboard\ndriver. Since it seems  the latter was introduced\nlate in the x264 architecture, maybe the\ndesigners weren't sure what was best and kept\nboth possibilities.
 NoConn ~ 7200 4880
 Wire Wire Line
@@
 Text Label 3880 7065 0    50   ~ 0
 f2r
+Wire Notes Line
+	2890 1215 3545 1215
+Wire Notes Line
+	3545 1215 3545 1585
+Wire Notes Line
+	3545 1585 2890 1585
+Wire Notes Line
+	2890 1585 2890 1220
+Text Notes 2845 1475 2    50   ~ 0
+ADDITIONAL CURRENT-\nLIMITING RESISTOR
+Wire Notes Line
+	2880 3990 3535 3990
+Wire Notes Line
+	3535 4360 2880 4360
+Wire Notes Line
+	2880 4360 2880 3995
+Text Notes 3575 4260 0    50   ~ 0
+ADDITIONAL CURRENT-\nLIMITING RESISTOR
+Wire Notes Line
+	3535 4360 3535 3995
 Wire Bus Line
 	9685 1705 9685 4880

Commit message: Switch joystick ports to DB9 connectors Not sure the power switch still fits. Fixing screws might touch protection diodes, too.
Parts:
- removed CN4: JOY1, LittleSixteen:KMDGX-8S-BS, symbol mini-din-8:Mini-DIN-8
- removed CN5: JOY2, LittleSixteen:KMDGX-8S-BS, symbol mini-din-8:Mini-DIN-8
- added CN4: JOY1, LittleSixteen:DB_9M, symbol Connector:DB9_Male_MountingHoles
- added CN5: JOY2, LittleSixteen:DB_9M, symbol Connector:DB9_Male_MountingHoles
- added JP10: JP_J2_POW5, Connector_PinHeader_2.54mm:PinHeader_1x02_P2.54mm_Vertical, symbol Device:Jumper_NC_Small
- added JP9: JP_J1_POW5, Connector_PinHeader_2.54mm:PinHeader_1x02_P2.54mm_Vertical, symbol Device:Jumper_NC_Small
Connections:
- net labels added: b1d, b1f, b1l, b1r, b1u, b2d, b2f, b2l, b2r, b2u
- no-connect marks 8 -> 10
Other:
- moved on the sheet: D1, D10, D2, D4, D5, D6, D7, D9, FB22, FB29, FB30, FB37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

Commit message: Enlarge drill holes to 0.9mm in order to make it possible to use ZIF sockets
Parts:
- U11: footprint Package_DIP:DIP-14_W7.62mm_Socket_LongPads -> LittleSixteen:DIP-14_W7.62mm_Socket_LongPads
- U17, U18: footprint Package_DIP:DIP-20_W7.62mm_Socket_LongPads -> LittleSixteen:DIP-20_W7.62mm_Socket_LongPads
Changed lines of the file:
@@
 F 0 "U17" H 6935 2960 50  0000 C CNN
 F 1 "74LS244" H 6975 1645 50  0000 C CNN
-F 2 "Package_DIP:DIP-20_W7.62mm_Socket_LongPads" H 6705 2305 50  0001 C CNN
+F 2 "LittleSixteen:DIP-20_W7.62mm_Socket_LongPads" H 6705 2305 50  0001 C CNN
 F 3 "https://assets.nexperia.com/documents/data-sheet/74AHC_AHCT244.pdf" H 6705 2305 50  0001 C CNN
 	1    6705 2305
@@
 F 0 "U11" H 2955 5797 50  0000 C CNN
 F 1 "74LS125" H 2955 5706 50  0000 C CNN
-F 2 "Package_DIP:DIP-14_W7.62mm_Socket_LongPads" H 2955 5480 50  0001 C CNN
+F 2 "LittleSixteen:DIP-14_W7.62mm_Socket_LongPads" H 2955 5480 50  0001 C CNN
 F 3 "http://www.ti.com/lit/gpn/sn74LS125" H 2955 5480 50  0001 C CNN
 	2    2955 5480
@@
 F 0 "U11" H 2955 3122 50  0000 C CNN
 F 1 "74LS125" H 2955 3031 50  0000 C CNN
-F 2 "Package_DIP:DIP-14_W7.62mm_Socket_LongPads" H 2955 2805 50  0001 C CNN
+F 2 "LittleSixteen:DIP-14_W7.62mm_Socket_LongPads" H 2955 2805 50  0001 C CNN
 F 3 "http://www.ti.com/lit/gpn/sn74LS125" H 2955 2805 50  0001 C CNN
 	1    2955 2805
@@
 F 0 "U18" H 6930 5635 50  0000 C CNN
 F 1 "74LS244" H 6970 4320 50  0000 C CNN
-F 2 "Package_DIP:DIP-20_W7.62mm_Socket_LongPads" H 6700 4980 50  0001 C CNN
+F 2 "LittleSixteen:DIP-20_W7.62mm_Socket_LongPads" H 6700 4980 50  0001 C CNN
 F 3 "https://assets.nexperia.com/documents/data-sheet/74AHC_AHCT244.pdf" H 6700 4980 50  0001 C CNN
 	1    6700 4980

Commit message: Use local Ferrite_Bead_Small symbol
Parts:
- FB22, FB24, FB25, FB26, FB27, FB28, FB29, FB30, FB31, FB32, FB33, FB34, FB35, FB37: symbol Device:Ferrite_Bead_Small -> ferrite_bead_small:Ferrite_Bead_Small
Changed lines of the file:
@@
 	5530 1110 5530 1080
 $Comp
-L Device:Ferrite_Bead_Small FB35
+L ferrite_bead_small:Ferrite_Bead_Small FB35
 U 1 1 5E19A8AD
 P 5010 4880
@@
 	4160 3705 4160 3775
 $Comp
-L Device:Ferrite_Bead_Small FB30
+L ferrite_bead_small:Ferrite_Bead_Small FB30
 U 1 1 5E19A89F
 P 4160 3875
@@
 $EndComp
 $Comp
-L Device:Ferrite_Bead_Small FB33
+L ferrite_bead_small:Ferrite_Bead_Small FB33
 U 1 1 5E19A894
 P 5010 4680
@@
 $EndComp
 $Comp
-L Device:Ferrite_Bead_Small FB34
+L ferrite_bead_small:Ferrite_Bead_Small FB34
 U 1 1 5E19A889
 P 5215 4780
@@
 $EndComp
 $Comp
-L Device:Ferrite_Bead_Small FB32
+L ferrite_bead_small:Ferrite_Bead_Small FB32
 U 1 1 5E19A87E
 P 5210 4580
@@
 $EndComp
 $Comp
-L Device:Ferrite_Bead_Small FB31
+L ferrite_bead_small:Ferrite_Bead_Small FB31
 U 1 1 5E19A873
 P 5010 4480
@@
 $EndComp
 $Comp
-L Device:Ferrite_Bead_Small FB29
+L ferrite_bead_small:Ferrite_Bead_Small FB29
 U 1 1 5E0A3992
 P 4230 2500
@@
 $EndComp
 $Comp
-L Device:Ferrite_Bead_Small FB28
+L ferrite_bead_small:Ferrite_Bead_Small FB28
 U 1 1 5E0A2BD5
 P 4965 2205
@@
 $EndComp
 $Comp
-L Device:Ferrite_Bead_Small FB22
+L ferrite_bead_small:Ferrite_Bead_Small FB22
 U 1 1 5E094DB1
 P 4115 1200
@@
 $EndComp
 $Comp
-L Device:Ferrite_Bead_Small FB26
+L ferrite_bead_small:Ferrite_Bead_Small FB26
 U 1 1 5E09220F
 P 4965 2005
@@
 $EndComp
 $Comp
-L Device:Ferrite_Bead_Small FB27
+L ferrite_bead_small:Ferrite_Bead_Small FB27
 U 1 1 5E09163E
 P 5165 2105
@@
 $EndComp
 $Comp
-L Device:Ferrite_Bead_Small FB25
+L ferrite_bead_small:Ferrite_Bead_Small FB25
 U 1 1 5E09073A
 P 5165 1905
@@
 $EndComp
 $Comp
-L Device:Ferrite_Bead_Small FB24
+L ferrite_bead_small:Ferrite_Bead_Small FB24
 U 1 1 5E08FAD9
 P 4965 1805
@@
 $EndComp
 $Comp
-L Device:Ferrite_Bead_Small FB37
+L ferrite_bead_small:Ferrite_Bead_Small FB37
 U 1 1 5E19A8B7
 P 4275 5175

Commit message: Use clearer diode footprint
Parts:
- D1, D10, D2, D3, D4, D5, D6, D7, D8, D9: footprint Diode_THT:D_DO-35_SOD27_P5.08mm_Vertical_KathodeUp -> LittleSixteen:D_DO-35_SOD27_P5.08mm_Vertical_KathodeUp
Changed lines of the file:
@@
 F 0 "D10" H 8330 4520 50  0000 C CNN
 F 1 "1N914" H 8355 4640 50  0000 C CNN
-F 2 "Diode_THT:D_DO-35_SOD27_P5.08mm_Vertical_KathodeUp" H 8195 4305 50  0001 C CNN
+F 2 "LittleSixteen:D_DO-35_SOD27_P5.08mm_Vertical_KathodeUp" H 8195 4305 50  0001 C CNN
 F 3 "http://www.vishay.com/docs/85622/1n914.pdf" H 8195 4480 50  0001 C CNN
 	1    8195 4480
@@
 F 0 "D9" H 8625 4810 50  0000 C CNN
 F 1 "1N914" H 8510 4901 50  0001 C CNN
-F 2 "Diode_THT:D_DO-35_SOD27_P5.08mm_Vertical_KathodeUp" H 8510 4600 50  0001 C CNN
+F 2 "LittleSixteen:D_DO-35_SOD27_P5.08mm_Vertical_KathodeUp" H 8510 4600 50  0001 C CNN
 F 3 "http://www.vishay.com/docs/85622/1n914.pdf" H 8510 4775 50  0001 C CNN
 	1    8510 4775
@@
 F 0 "D8" H 8305 4720 50  0000 C CNN
 F 1 "1N914" H 8195 4455 50  0001 C CNN
-F 2 "Diode_THT:D_DO-35_SOD27_P5.08mm_Vertical_KathodeUp" H 8195 4505 50  0001 C CNN
+F 2 "LittleSixteen:D_DO-35_SOD27_P5.08mm_Vertical_KathodeUp" H 8195 4505 50  0001 C CNN
 F 3 "http://www.vishay.com/docs/85622/1n914.pdf" H 8195 4680 50  0001 C CNN
 	1    8195 4680
@@
 F 0 "D7" H 8305 5025 50  0000 C CNN
 F 1 "1N914" H 8195 5105 50  0001 C CNN
-F 2 "Diode_THT:D_DO-35_SOD27_P5.08mm_Vertical_KathodeUp" H 8195 4805 50  0001 C CNN
+F 2 "LittleSixteen:D_DO-35_SOD27_P5.08mm_Vertical_KathodeUp" H 8195 4805 50  0001 C CNN
 F 3 "http://www.vishay.com/docs/85622/1n914.pdf" H 8195 4980 50  0001 C CNN
 	1    8195 4980
@@
 F 0 "D5" H 8305 1845 50  0000 C CNN
 F 1 "1N914" H 8365 1950 50  0000 C CNN
-F 2 "Diode_THT:D_DO-35_SOD27_P5.08mm_Vertical_KathodeUp" H 8195 1630 50  0001 C CNN
+F 2 "LittleSixteen:D_DO-35_SOD27_P5.08mm_Vertical_KathodeUp" H 8195 1630 50  0001 C CNN
 F 3 "http://www.vishay.com/docs/85622/1n914.pdf" H 8195 1805 50  0001 C CNN
 	1    8195 1805
@@
 F 0 "D3" H 8305 2045 50  0000 C CNN
 F 1 "1N914" H 8195 1790 50  0001 C CNN
-F 2 "Diode_THT:D_DO-35_SOD27_P5.08mm_Vertical_KathodeUp" H 8195 1830 50  0001 C CNN
+F 2 "LittleSixteen:D_DO-35_SOD27_P5.08mm_Vertical_KathodeUp" H 8195 1830 50  0001 C CNN
 F 3 "http://www.vishay.com/docs/85622/1n914.pdf" H 8195 2005 50  0001 C CNN
 	1    8195 2005
@@
 F 0 "D1" H 8625 1940 50  0000 C CNN
 F 1 "1N914" H 8510 2025 50  0001 C CNN
-F 2 "Diode_THT:D_DO-35_SOD27_P5.08mm_Vertical_KathodeUp" H 8510 1725 50  0001 C CNN
+F 2 "LittleSixteen:D_DO-35_SOD27_P5.08mm_Vertical_KathodeUp" H 8510 1725 50  0001 C CNN
 F 3 "http://www.vishay.com/docs/85622/1n914.pdf" H 8510 1900 50  0001 C CNN
 	1    8510 1900
@@
 F 0 "D6" H 8625 4625 50  0000 C CNN
 F 1 "1N914" H 8510 4705 50  0001 C CNN
-F 2 "Diode_THT:D_DO-35_SOD27_P5.08mm_Vertical_KathodeUp" H 8510 4405 50  0001 C CNN
+F 2 "LittleSixteen:D_DO-35_SOD27_P5.08mm_Vertical_KathodeUp" H 8510 4405 50  0001 C CNN
 F 3 "http://www.vishay.com/docs/85622/1n914.pdf" H 8510 4580 50  0001 C CNN
 	1    8510 4580
@@
 F 0 "D2" H 8305 2345 50  0000 C CNN
 F 1 "1N914" H 8195 2430 50  0001 C CNN
-F 2 "Diode_THT:D_DO-35_SOD27_P5.08mm_Vertical_KathodeUp" H 8195 2130 50  0001 C CNN
+F 2 "LittleSixteen:D_DO-35_SOD27_P5.08mm_Vertical_KathodeUp" H 8195 2130 50  0001 C CNN
 F 3 "http://www.vishay.com/docs/85622/1n914.pdf" H 8195 2305 50  0001 C CNN
 	1    8195 2305
@@
 F 0 "D4" H 8625 2145 50  0000 C CNN
 F 1 "1N914" H 8510 2231 50  0001 C CNN
-F 2 "Diode_THT:D_DO-35_SOD27_P5.08mm_Vertical_KathodeUp" H 8510 1930 50  0001 C CNN
+F 2 "LittleSixteen:D_DO-35_SOD27_P5.08mm_Vertical_KathodeUp" H 8510 1930 50  0001 C CNN
 F 3 "http://www.vishay.com/docs/85622/1n914.pdf" H 8510 2105 50  0001 C CNN
 	1    8510 2105
