File: ram.sch (KiCad schematic (older format))
At the start: 14 parts, among them U12 74LS02, U5 4416, U6 4416, U7 74LS257, U8 74LS257

Commit message: Various minor fixes
Parts:
- renumbered JP1 to JP3, JP2 to JP4
Other:
- note added: "JP3/4 are a 16kB/64kB\nRAM Switch Mod. Use\n4464 chips instead of 4416."
- note removed: "JP1/2 are a 16kB/64kB\nRAM Switch Mod. Use\n4464 chips instead of 4416."
Changed lines of the file:
@@
 	3380 6525 3760 6525
 $Comp
-L Connector:Conn_01x03_Male JP2
+L Connector:Conn_01x03_Male JP4
 U 1 1 61451C3E
 P 2765 3770
-F 0 "JP2" V 2827 3582 50  0000 R CNN
+F 0 "JP4" V 2827 3582 50  0000 R CNN
 F 1 "JP_RAMSIZE2" V 2918 3582 50  0000 R CNN
 F 2 "Connector_PinHeader_2.54mm:PinHeader_1x03_P2.54mm_Vertical" H 2765 3770 50  0001 C CNN
@@
 $EndComp
 $Comp
-L Connector:Conn_01x03_Male JP1
+L Connector:Conn_01x03_Male JP3
 U 1 1 6147B280
 P 2765 1030
-F 0 "JP1" V 2827 842 50  0000 R CNN
+F 0 "JP3" V 2827 842 50  0000 R CNN
 F 1 "JP_RAMSIZE1" V 2918 842 50  0000 R CNN
 F 2 "Connector_PinHeader_2.54mm:PinHeader_1x03_P2.54mm_Vertical" H 2765 1030 50  0001 C CNN
@@
 a15
 Text Notes 3175 1230 0    50   ~ 0
-JP1/2 are a 16kB/64kB\nRAM Switch Mod. Use\n4464 chips instead of 4416.
+JP3/4 are a 16kB/64kB\nRAM Switch Mod. Use\n4464 chips instead of 4416.
 Text GLabel 5445 1540 0    50   Input ~ 0
 RAMEN

Commit message: Enlarge drill holes to 0.9mm in order to make it possible to use ZIF sockets
Parts:
- U12: footprint Package_DIP:DIP-14_W7.62mm_Socket_LongPads -> LittleSixteen:DIP-14_W7.62mm_Socket_LongPads
- U5, U6: footprint Package_DIP:DIP-18_W7.62mm_Socket_LongPads -> LittleSixteen:DIP-18_W7.62mm_Socket_LongPads
- U7, U8: footprint Package_DIP:DIP-16_W7.62mm_Socket_LongPads -> LittleSixteen:DIP-16_W7.62mm_Socket_LongPads
Changed lines of the file:
@@
 F 0 "U6" H 8710 2905 50  0000 C CNN
 F 1 "4416" H 8710 2814 50  0000 C CNN
-F 2 "Package_DIP:DIP-18_W7.62mm_Socket_LongPads" H 8710 1390 50  0001 C CNN
+F 2 "LittleSixteen:DIP-18_W7.62mm_Socket_LongPads" H 8710 1390 50  0001 C CNN
 F 3 "http://pdf.datasheetcatalog.com/datasheet_pdf/texas-instruments/TMS4416-12_to_TMS4416-20.pdf" H 8710 1490 50  0001 C CNN
 	1    8710 2140
@@
 F 0 "U5" H 8710 4605 50  0000 C CNN
 F 1 "4416" H 8710 4514 50  0000 C CNN
-F 2 "Package_DIP:DIP-18_W7.62mm_Socket_LongPads" H 8710 3090 50  0001 C CNN
+F 2 "LittleSixteen:DIP-18_W7.62mm_Socket_LongPads" H 8710 3090 50  0001 C CNN
 F 3 "http://pdf.datasheetcatalog.com/datasheet_pdf/texas-instruments/TMS4416-12_to_TMS4416-20.pdf" H 8710 3190 50  0001 C CNN
 	1    8710 3840
@@
 F 0 "U7" H 3235 7081 50  0000 L CNN
 F 1 "74LS257" H 3235 6990 50  0000 L CNN
-F 2 "Package_DIP:DIP-16_W7.62mm_Socket_LongPads" H 3005 7010 50  0001 C CNN
+F 2 "LittleSixteen:DIP-16_W7.62mm_Socket_LongPads" H 3005 7010 50  0001 C CNN
 F 3 "" H 3005 7010 50  0001 C CNN
 	2    3005 7010
@@
 F 0 "U8" H 4740 7081 50  0000 L CNN
 F 1 "74LS257" H 4740 6990 50  0000 L CNN
-F 2 "Package_DIP:DIP-16_W7.62mm_Socket_LongPads" H 4510 7010 50  0001 C CNN
+F 2 "LittleSixteen:DIP-16_W7.62mm_Socket_LongPads" H 4510 7010 50  0001 C CNN
 F 3 "" H 4510 7010 50  0001 C CNN
 	2    4510 7010
@@
 F 0 "U8" H 3420 5680 50  0000 C CNN
 F 1 "74LS257" H 3420 4060 50  0000 C CNN
-F 2 "Package_DIP:DIP-16_W7.62mm_Socket_LongPads" H 3420 4930 50  0001 C CNN
+F 2 "LittleSixteen:DIP-16_W7.62mm_Socket_LongPads" H 3420 4930 50  0001 C CNN
 F 3 "" H 3420 4930 50  0001 C CNN
 	1    3420 4930
@@
 F 0 "U7" H 3420 2940 50  0000 C CNN
 F 1 "74LS257" H 3420 1320 50  0000 C CNN
-F 2 "Package_DIP:DIP-16_W7.62mm_Socket_LongPads" H 3420 2190 50  0001 C CNN
+F 2 "LittleSixteen:DIP-16_W7.62mm_Socket_LongPads" H 3420 2190 50  0001 C CNN
 F 3 "" H 3420 2190 50  0001 C CNN
 	1    3420 2190
@@
 F 0 "U12" H 6015 1965 50  0000 C CNN
 F 1 "74LS02" H 6015 1874 50  0000 C CNN
-F 2 "Package_DIP:DIP-14_W7.62mm_Socket_LongPads" H 6015 1640 50  0001 C CNN
+F 2 "LittleSixteen:DIP-14_W7.62mm_Socket_LongPads" H 6015 1640 50  0001 C CNN
 F 3 "http://www.ti.com/lit/gpn/sn74ls02" H 6015 1640 50  0001 C CNN
 	4    6015 1640

Commit message: Add 512kB RAM expansions, Hannes-style
Parts:
- removed C10, C92: 100n, Capacitor_THT:C_Disc_D8.0mm_W2.5mm_P5.00mm, symbol Device:C
- removed C7, C8: 220n, Capacitor_THT:C_Disc_D8.0mm_W2.5mm_P5.00mm, symbol Device:C
- removed JP3: JP_RAMSIZE1, Connector_PinHeader_2.54mm:PinHeader_1x03_P2.54mm_Vertical, symbol Connector:Conn_01x03_Male
- removed JP4: JP_RAMSIZE2, Connector_PinHeader_2.54mm:PinHeader_1x03_P2.54mm_Vertical, symbol Connector:Conn_01x03_Male
- removed R99: 10k, Resistor_THT:R_Axial_DIN0207_L6.3mm_D2.5mm_P5.08mm_Vertical, symbol Device:R
- removed RP3: 68, Resistor_THT:R_Array_SIP8, symbol rp3:RPack4_RP3
- removed RP4: 68, Resistor_THT:R_Array_SIP8, symbol rp4:RPack4_RP4
- removed U12: 74LS02, LittleSixteen:DIP-14_W7.62mm_Socket_LongPads, symbol 74xx:74LS02
- removed U5, U6: 4416, LittleSixteen:DIP-18_W7.62mm_Socket_LongPads, symbol 4416:4416
- removed U7, U8: 74LS257, LittleSixteen:DIP-16_W7.62mm_Socket_LongPads, symbol 74ls157:74LS157
- added C1, C2, C27, C9: 100n, Capacitor_SMD:C_0805_2012Metric_Pad1.18x1.45mm_HandSolder, symbol Device:C
- added C56: 100n, Capacitor_THT:C_Disc_D8.0mm_W2.5mm_P5.00mm, symbol Device:C
- added RN4, RN5: 1k, Resistor_SMD:R_Array_Convex_4x0603, symbol Device:R_Pack04
- added SW3: SW_JOYSWAP, Connector_PinHeader_2.54mm:PinHeader_1x03_P2.54mm_Vertical, symbol Connector:Conn_01x03_Male
- added U25: 74LS74, Package_DIP:DIP-14_W7.62mm_Socket_LongPads, symbol 74xx:74LS74
- added U26: GAL16V8, Package_DIP:DIP-20_W7.62mm_Socket_LongPads, symbol Logic_Programmable:GAL16V8
- added U29: 74HCT245, Package_SO:SO-20_5.3x12.6mm_P1.27mm, symbol 74xx:74LS245
- added U30: AS6C4008, Package_DIP:DIP-32_W15.24mm_Socket_LongPads, symbol AS6C4008:AS6C4008
- added U5: 74HCT02, Package_SO:SOIC-14_3.9x8.7mm_P1.27mm, symbol 74xx:74HCT02
- added U6: 74HCT573, Package_SO:SO-20_5.3x12.6mm_P1.27mm, symbol 74xx:74LS573
Connections:
- net GND: now also C1.2, C2.2, C27.2, C56.2, C9.2, SW3.1 (Pin_1), U25.11 (C), U25.12 (D), U26.10 (GND), U29.10 (GND), U30.16 (GND), U5.7 (GND), U6.10 (GND)
- net R_~W: now also U30.29 (~WE), U5.9
- net VCC: now also C1.1, C2.1, C27.1, C56.1, C9.1, RN4.5 (R4.2), RN4.6 (R3.2), RN4.7 (R2.2), RN4.8 (R1.2), RN5.5 (R4.2), RN5.6 (R3.2), RN5.7 (R2.2), RN5.8 (R1.2), SW3.3 (Pin_3), U26.20 (VCC), U29.1 (A->B), U29.20 (VCC), U30.32 (VCC), U5.14 (VCC), U6.20 (VCC)
- net a0: now also U30.4 (A12)
- net a1: now also U30.3 (A14)
- net a10: now also U30.7 (A5)
- net a11: now also U30.9 (A3)
- net a12: now also U26.4 (I4), U30.10 (A2)
- net a13: now also U26.3 (I3), U30.8 (A4)
- net a14: now also U26.2 (I2), U30.11 (A1)
- net a15: now also U26.1 (I1/CLK), U30.12 (A0)
- net a2: now also U30.23 (A10)
- net a3: now also U30.31 (A15)
- net a4: now also U30.25 (A11)
- net a5: now also U30.28 (A13)
- net a6: now also U30.27 (A8)
- net a7: now also U30.26 (A9)
- net a8: now also U30.5 (A7)
- net a9: now also U30.6 (A6)
- net d0: now also U29.18 (B0), U30.15 (D2), U6.2 (D0)
- net d1: now also U26.13 (IO7), U29.17 (B1), U30.14 (D1), U6.3 (D1)
- net d2: now also U26.12 (IO8), U29.16 (B2), U30.13 (D0), U6.4 (D2)
- net d3: now also U29.15 (B3), U30.17 (D3), U6.5 (D3)
- net d4: now also U29.14 (B4), U30.18 (D4), U6.6 (D4)
- net d5: now also U29.13 (B5), U30.19 (D5), U6.7 (D5)
- net d6: now also U29.12 (B6), U30.20 (D6), U6.8 (D6)
- net d7: now also U29.11 (B7), U30.21 (D7), U6.9 (D7)
- net ~CAS: now also U5.6
- new net: U5.2, U5.3, U5.4
- new net: U5.10, U5.5
- new net AEC: U26.11 (I10/~OE~)
- new net CS_RAMWR: U5.11, U5.12, U6.11 (Load)
- new net PHI0: U5.8
- new net a16: U26.19 (IO1), U30.2 (A16)
- new net a17: U26.18 (IO2), U30.30 (A17)
- new net a18: U26.17 (I03), U30.1 (A18)
- new net joyswap: SW3.2 (Pin_2), U26.14 (IO6)
- new net r0: RN4.4 (R4.1), U26.5 (I5), U29.2 (A0), U6.19 (Q0)
- new net r1: RN4.3 (R3.1), U26.6 (I6), U29.3 (A1), U6.18 (Q1)
- new net r2: RN4.2 (R2.1), U26.7 (I7), U29.4 (A2), U6.17 (Q2)
- new net r3: RN4.1 (R1.1), U29.5 (A3), U6.16 (Q3)
- new net r4: RN5.4 (R4.1), U29.6 (A4), U6.15 (Q4)
- new net r5: RN5.3 (R3.1), U29.7 (A5), U6.14 (Q5)
- new net r6: RN5.2 (R2.1), U26.8 (I8), U29.8 (A6), U6.13 (Q6)
- new net r7: RN5.1 (R1.1), U26.9 (I9), U29.9 (A7), U6.12 (Q7)
- new net sram_ce: U30.22 (~CE), U30.24 (~OE), U5.1
- new net ~CS_RAMRD: U29.19 (CE)
- new net ~JOY1: U26.15 (IO5)
- new net ~JOY2: U26.16 (IO4)
- new net ~RESET: U25.10 (~S)
- new net ~cs_ramwr: U25.13 (~R), U5.13
- new net ~u3enable: U25.9 (Q), U6.1 (OE)
- no-connect marks 0 -> 1
Other:
- note added: "$FD16 READ"
- note added: "$FD16 WRITE\n(NOTE: ACTIVE *HIGH*!)"
- note added: "PLA - 2 -"
- note added: "THIS CIRCUIT WAS DERIVED\nFROM WORK BY ESLAPION"
- note added: "WE ALSO NEED SOMETHING ELSE TO ALLOW OUR\nRAM CONTROL REGISTER TO BE READ BACK. SINCE\nWE ARE WORKING WITH REVERSE LOGIC, WE USE\nAN INVERTING BUFFER AND... TA-DA!"
- note added: "fixme"
- note removed: "Additional\ndecoupling cap"
- note removed: "JP3/4 are a 16kB/64kB\nRAM Switch Mod. Use\n4464 chips instead of 4416."
- note removed: "U7 and U8 can either be 74x157 or 74x257,\nsince they are permanently enabled"
- note removed: "We make use of a spare gate to fix the\neternal problem of external RAM\nexpansions not working, which is due to\nthe impossibility of disabling the internal\nRAM. This should do it, just ground the Z\npin and the internal RAM will disappear."
- note removed: "Yes, RP3/4 have this\nweird pin numbering,\nmost likely in order to\nmake routing easier"

Commit message: WIP
Parts:
- removed RN4, RN5: 1k, Resistor_SMD:R_Array_Convex_4x0603, symbol Device:R_Pack04
- added RP3: 10k, Resistor_THT:R_Array_SIP9, symbol Device:R_Network08
- C7: renamed from C2; footprint Capacitor_SMD:C_0805_2012Metric_Pad1.18x1.45mm_HandSolder -> Capacitor_THT:C_Disc_D8.0mm_W2.5mm_P5.00mm
- C8: renamed from C1; footprint Capacitor_SMD:C_0805_2012Metric_Pad1.18x1.45mm_HandSolder -> Capacitor_THT:C_Disc_D8.0mm_W2.5mm_P5.00mm
- C9: footprint Capacitor_SMD:C_0805_2012Metric_Pad1.18x1.45mm_HandSolder -> Capacitor_THT:C_Disc_D8.0mm_W2.5mm_P5.00mm
- C92: renamed from C27; footprint Capacitor_SMD:C_0805_2012Metric_Pad1.18x1.45mm_HandSolder -> Capacitor_THT:C_Disc_D8.0mm_W2.5mm_P5.00mm
- U25: footprint Package_DIP:DIP-14_W7.62mm_Socket_LongPads -> LittleSixteen:DIP-14_W7.62mm_Socket_LongPads
- U26: footprint Package_DIP:DIP-20_W7.62mm_Socket_LongPads -> LittleSixteen:DIP-20_W7.62mm_Socket_LongPads
- U29, U6: footprint Package_SO:SO-20_5.3x12.6mm_P1.27mm -> LittleSixteen:DIP-20_W7.62mm_Socket_LongPads
- U5: footprint Package_SO:SOIC-14_3.9x8.7mm_P1.27mm -> LittleSixteen:DIP-14_W7.62mm_Socket_LongPads
Connections:
- net VCC: now also RP3.1 (common)
- net d0: now also U30.21 (D7); no longer U30.15 (D2)
- net d1: now also U30.13 (D0); no longer U30.14 (D1)
- net d2: now also U30.20 (D6); no longer U30.13 (D0)
- net d3: now also U30.14 (D1); no longer U30.17 (D3)
- net d4: now also U30.19 (D5); no longer U30.18 (D4)
- net d5: now also U30.15 (D2); no longer U30.19 (D5)
- net d6: now also U30.18 (D4); no longer U30.20 (D6)
- net d7: now also U30.17 (D3); no longer U30.21 (D7)
- net r0: now also RP3.2 (R1)
- net r1: now also RP3.3 (R2)
- net r2: now also RP3.4 (R3)
- net r3: now also RP3.5 (R4)
- net r4: now also RP3.6 (R5)
- net r5: now also RP3.7 (R6)
- net r6: now also RP3.8 (R7)
- net r7: now also RP3.9 (R8)
Other:
- note removed: "fixme"

Commit message: -63
Connections:
- net GND: now also C9.1; no longer C9.2
- net VCC: now also C9.2; no longer C9.1
- net ~JOY1: now also U26.16 (IO4); no longer U26.15 (IO5)
- net ~JOY2: now also U26.15 (IO5); no longer U26.16 (IO4)
Changed lines of the file:
@@
 	4665 2895 5035 2895
 Text GLabel 8060 2895 2    50   Output ~ 0
-p[0..7]
+r[0..7]
 Text Label 7630 2095 2    50   ~ 0
 r0
@@
 	7965 4175 7635 4175
 Text GLabel 7635 4175 0    50   Input ~ 0
-p[0..7]
+r[0..7]
 Entry Wire Line
 	8065 4275 7965 4175
@@
 AR Path="/5E4A465A/64E9FF4C/64F128AF" Ref="C?"  Part="1"
 AR Path="/5E4A465A/64F128AF" Ref="C9"  Part="1"
-F 0 "C9" H 10420 4301 50  0000 R CNN
-F 1 "100n" H 10420 4210 50  0000 R CNN
+F 0 "C9" H 10420 4209 50  0000 R CNN
+F 1 "100n" H 10420 4300 50  0000 R CNN
 F 2 "Capacitor_THT:C_Disc_D8.0mm_W2.5mm_P5.00mm" H 10573 4105 50  0001 C CNN
 F 3 "~" H 10535 4255 50  0001 C CNN
 	1    10535 4255
-	1    0    0    -1
+	-1   0    0    1
 $EndComp
 Wire Wire Line
@@
 Text Label 3060 2065 2    50   ~ 0
 d1
-Text GLabel 3355 1865 2    50   Output ~ 0
-~JOY1
-Text GLabel 3115 1765 2    50   Output ~ 0
-~JOY2
 Wire Wire Line
 	2855 1965 3780 1965
@@
 Wire Bus Line
 	13460 1660 13460 3305
+Text GLabel 3115 1765 2    50   Output ~ 0
+~JOY1
+Text GLabel 3355 1865 2    50   Output ~ 0
+~JOY2
 $EndSCHEMATC
