File: ram.sch (KiCad schematic (older format))
At the start: 13 parts, among them SW3 SW_JOYSWAP, U25 74LS74, U26 GAL16V8, U29 74HCT245, U30 AS6C4008, U5 74HCT02, U6 74HCT573

Commit message: -2!!!
Other:
- note added: "WE ALSO NEED SOMETHING ELSE TO ALLOW OUR\nRAM CONTROL REGISTER TO BE READ BACK..."
- note removed: "WE ALSO NEED SOMETHING ELSE TO ALLOW OUR\nRAM CONTROL REGISTER TO BE READ BACK. SINCE\nWE ARE WORKING WITH REVERSE LOGIC, WE USE\nAN INVERTING BUFFER AND... TA-DA!"
- moved on the sheet: C56, C7, C9, C92, RP3, SW3, U25B, U26, U29, U30, U5A, U5B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

Commit message: Make most ICs HCT
Parts:
- SW3: Notes For 6581 do not mount -> (none)
Changed lines of the file:
@@
 F 2 "Connector_PinHeader_2.54mm:PinHeader_1x03_P2.54mm_Vertical" H 3880 1950 50  0001 C CNN
 F 3 "~" H 3880 1950 50  0001 C CNN
-F 4 "For 6581 do not mount" H 3880 1950 50  0001 C CNN "Notes"
+F 4 "" H 3880 1950 50  0001 C CNN "Notes"
 F 5 "SW_DIGIFIX" H 3880 1950 50  0001 C CNN "Value"
 	1    3880 1950

Commit message: Switch to 2-pin header for joyswap
Parts:
- removed SW3: SW_JOYSWAP, Connector_PinHeader_2.54mm:PinHeader_1x03_P2.54mm_Vertical, symbol Connector:Conn_01x03_Male
- added R97: 10k, Resistor_THT:R_Axial_DIN0207_L6.3mm_D2.5mm_P5.08mm_Vertical, symbol Device:R
- added SW3: SW_JOYSWAP, Connector_PinHeader_2.54mm:PinHeader_1x02_P2.54mm_Vertical, symbol Connector:Conn_01x02_Male
Connections:
- net GND: now also SW3.1 (Pin_1)
- net VCC: now also R97.2
- net joyswap: now also R97.1, SW3.2 (Pin_2)
Other:
- note added: "- WE USE A SINGLE STATIC RAM CHIP\n- WE SUPPORT A HANNES-STYLE MECHANISM\n FOR RAM EXPANSION TO UP TO 512 KB"
- note added: "Another idea from Levente Hársfalvi in order to achieve the "high at reset"\nbehaviour of the MOS 6529 that was originally used in Hannes/Solder's\ndesign for the control register: keep the 74x573 in Hi-Z until the first write\nto $FD16 and use pull-ups on its output. All hail TLC!"
- note added: "Generates:\n- High RAM address bits, depending on the contents of the $FD16\n register, implementing the Hannes logic\n- ~CS~ signals for joystick buffers, adding the possibility of swapping"
- note added: "Note that address bits and data bits can be swapped freely\nhere since no refresh mechanism is involved, so let's just\nassign everything in order to simplify routing!"
- moved on the sheet: C56, C7, RP3, U25B, U26, U5D, U6

Commit message: Update schematics PDF
Other:
- note added: "Generates:\n- High RAM address bits, depending on the contents of the $FD16\n register, implementing the Hannes logic\n- ~CS~ signals for joystick buffers, with the possibility of swapping them"
- note removed: "Generates:\n- High RAM address bits, depending on the contents of the $FD16\n register, implementing the Hannes logic\n- ~CS~ signals for joystick buffers, adding the possibility of swapping"
Changed lines of the file:
@@
 Title "LittleSixteen"
 Date "2023-07-10"
-Rev "3git"
+Rev "4git"
 Comp "SukkoPera"
 Comment1 "Licensed under CC BY-NC-SA 4.0"
@@
 ~JOY2
 Text Notes 940  1135 0    50   ~ 0
-Generates:\n- High RAM address bits, depending on the contents of the $FD16\n  register, implementing the Hannes logic\n-  ~CS~ signals for joystick buffers, adding the possibility of swapping
+Generates:\n- High RAM address bits, depending on the contents of the $FD16\n  register, implementing the Hannes logic\n-  ~CS~ signals for joystick buffers, with the possibility of swapping them
 $Comp
 L AS6C4008:AS6C4008 U30

Commit message: Rationalize BOM There should be no significant changes on both schematics on PCB, just some values and something on the silkscreen
Parts:
- C7, C8, C9, C92: MouserPN (none) -> 810-FG28X7R1H104KNT0
- RP7: renamed from RP3; Notes (none) -> Bussed
- U30: MouserPN (none) -> 913-AS6C4008-55PIN; Notes (none) -> Or AS6C4008-55PCN
- renumbered SW3 to JP17
Changed lines of the file:
@@
 F 2 "Capacitor_THT:C_Disc_D8.0mm_W2.5mm_P5.00mm" H 7373 4625 50  0001 C CNN
 F 3 "~" H 7335 4775 50  0001 C CNN
+F 4 "810-FG28X7R1H104KNT0" H 7335 4775 50  0001 C CNN "MouserPN"
 	1    7335 4775
 	1    0    0    -1
@@
 F 2 "Capacitor_THT:C_Disc_D8.0mm_W2.5mm_P5.00mm" H 2018 6635 50  0001 C CNN
 F 3 "~" H 1980 6785 50  0001 C CNN
+F 4 "810-FG28X7R1H104KNT0" H 1980 6785 50  0001 C CNN "MouserPN"
 	1    1980 6785
 	1    0    0    -1
@@
 F 2 "Capacitor_THT:C_Disc_D8.0mm_W2.5mm_P5.00mm" H 6263 4700 50  0001 C CNN
 F 3 "~" H 6225 4850 50  0001 C CNN
+F 4 "810-FG28X7R1H104KNT0" H 6225 4850 50  0001 C CNN "MouserPN"
 	1    6225 4850
 	-1   0    0    1
@@
 F 2 "Capacitor_THT:C_Disc_D8.0mm_W2.5mm_P5.00mm" H 5188 1235 50  0001 C CNN
 F 3 "~" H 5150 1385 50  0001 C CNN
+F 4 "810-FG28X7R1H104KNT0" H 5150 1385 50  0001 C CNN "MouserPN"
 	1    5150 1385
 	1    0    0    -1
@@
 	1840 2655 1525 2655
 $Comp
-L Device:R_Network08 RP3
+L Device:R_Network08 RP7
 U 1 1 6475B295
 P 6755 1755
-F 0 "RP3" H 7143 1801 50  0000 L CNN
+F 0 "RP7" H 7143 1801 50  0000 L CNN
 F 1 "10k" H 7143 1710 50  0000 L CNN
 F 2 "Resistor_THT:R_Array_SIP9" V 7230 1755 50  0001 C CNN
 F 3 "http://www.vishay.com/docs/31509/csc.pdf" H 6755 1755 50  0001 C CNN
+F 4 "Bussed" H 6755 1755 50  0001 C CNN "Notes"
 	1    6755 1755
 	1    0    0    -1
@@
 F 2 "Package_DIP:DIP-32_W15.24mm_Socket_LongPads" H 9385 4830 50  0001 C CNN
 F 3 "DOCUMENTATION" H 9385 4830 50  0001 C CNN
+F 4 "913-AS6C4008-55PIN" H 9385 4830 50  0001 C CNN "MouserPN"
+F 5 "Or AS6C4008-55PCN" H 9385 4830 50  0001 C CNN "Notes"
 	1    9385 4830
 	1    0    0    -1
@@
 P 3965 2355
 AR Path="/64A6E6F3/65AA1AF3" Ref="CN?"  Part="1"
-AR Path="/5E4A465A/65AA1AF3" Ref="SW3"  Part="1"
-F 0 "SW3" H 3937 2237 50  0000 R CNN
+AR Path="/5E4A465A/65AA1AF3" Ref="JP17"  Part="1"
+F 0 "JP17" H 3937 2237 50  0000 R CNN
 F 1 "SW_JOYSWAP" H 3937 2328 50  0000 R CNN
 F 2 "Connector_PinHeader_2.54mm:PinHeader_1x02_P2.54mm_Vertical" H 3965 2355 50  0001 C CNN

Commit message: Rationalize capacitor footprints & BOM
Parts:
- R97: MouserPN (none) -> 603-MFR-25FTF52-10K
- U29: Notes (none) -> Or 595-SN74HCT245NE4
- U5: MouserPN (none) -> 595-SN74HCT02N; Notes (none) -> Or 595-SN74HC02N, 595-SN74HCT02NE4
Changed lines of the file:
@@
 F 2 "LittleSixteen:DIP-14_W7.62mm_Socket_LongPads" H 5800 7175 50  0001 C CNN
 F 3 "http://www.ti.com/lit/gpn/sn74hct02" H 5800 7175 50  0001 C CNN
+F 4 "595-SN74HCT02N" H 5800 7175 50  0001 C CNN "MouserPN"
+F 5 "Or 595-SN74HC02N, 595-SN74HCT02NE4" H 5800 7175 50  0001 C CNN "Notes"
 	1    5800 7175
 	1    0    0    -1
@@
 F 2 "LittleSixteen:DIP-14_W7.62mm_Socket_LongPads" H 4945 7175 50  0001 C CNN
 F 3 "http://www.ti.com/lit/gpn/sn74hct02" H 4945 7175 50  0001 C CNN
+F 4 "595-SN74HCT02N" H 4945 7175 50  0001 C CNN "MouserPN"
+F 5 "Or 595-SN74HC02N, 595-SN74HCT02NE4" H 4945 7175 50  0001 C CNN "Notes"
 	2    4945 7175
 	1    0    0    -1
@@
 F 2 "LittleSixteen:DIP-14_W7.62mm_Socket_LongPads" H 3885 7075 50  0001 C CNN
 F 3 "http://www.ti.com/lit/gpn/sn74hct02" H 3885 7075 50  0001 C CNN
+F 4 "595-SN74HCT02N" H 3885 7075 50  0001 C CNN "MouserPN"
+F 5 "Or 595-SN74HC02N, 595-SN74HCT02NE4" H 3885 7075 50  0001 C CNN "Notes"
 	3    3885 7075
 	1    0    0    -1
@@
 F 2 "LittleSixteen:DIP-14_W7.62mm_Socket_LongPads" H 1145 6790 50  0001 C CNN
 F 3 "http://www.ti.com/lit/gpn/sn74hct02" H 1145 6790 50  0001 C CNN
+F 4 "595-SN74HCT02N" H 1145 6790 50  0001 C CNN "MouserPN"
+F 5 "Or 595-SN74HC02N, 595-SN74HCT02NE4" H 1145 6790 50  0001 C CNN "Notes"
 	5    1145 6790
 	1    0    0    -1
@@
 F 3 "http://www.ti.com/lit/gpn/sn74LS245" H 4770 5370 50  0001 C CNN
 F 4 "595-SN74HCT245ANSR" H 4770 5370 50  0001 C CNN "MouserPN"
+F 5 "Or 595-SN74HCT245NE4" H 4770 5370 50  0001 C CNN "Notes"
 	1    4770 5370
 	1    0    0    -1
@@
 F 2 "LittleSixteen:DIP-14_W7.62mm_Socket_LongPads" H 2680 4190 50  0001 C CNN
 F 3 "http://www.ti.com/lit/gpn/sn74hct02" H 2680 4190 50  0001 C CNN
+F 4 "595-SN74HCT02N" H 2680 4190 50  0001 C CNN "MouserPN"
+F 5 "Or 595-SN74HC02N, 595-SN74HCT02NE4" H 2680 4190 50  0001 C CNN "Notes"
 	4    2680 4190
 	1    0    0    -1
@@
 F 2 "Resistor_THT:R_Axial_DIN0207_L6.3mm_D2.5mm_P5.08mm_Vertical" V 3630 1940 50  0001 C CNN
 F 3 "~" H 3700 1940 50  0001 C CNN
+F 4 "603-MFR-25FTF52-10K" H 3700 1940 50  0001 C CNN "MouserPN"
 	1    3700 1940
 	-1   0    0    1

Commit message: Add RAM size jumper So we no longer need to reflash PLA2 to change it!
Parts:
- added JP4: SW_RAMSIZE, Connector_PinHeader_2.54mm:PinHeader_1x03_P2.54mm_Vertical, symbol Jumper:Jumper_3_Bridged12
Connections:
- net GND: now also JP4.3 (B)
- net a18: now also JP4.2 (C); no longer U26.17 (I03)
- new net a18_from_pla: JP4.1 (A), U26.17 (I03)
Other:
- note added: "- WE USE A SINGLE STATIC RAM CHIP\n- WE SUPPORT A HANNES-STYLE MECHANISM\n FOR RAM EXPANSION TO UP TO 512 KB\n- WE PROVIDE A SWITCH TO LIMIT THE RAM\n TO 256 KB FOR COMPATIBLITY"
- note added: "256\nkB"
- note added: "512\nkB"
- note removed: "- WE USE A SINGLE STATIC RAM CHIP\n- WE SUPPORT A HANNES-STYLE MECHANISM\n FOR RAM EXPANSION TO UP TO 512 KB"
- moved on the sheet: JP17, R97
Changed lines of the file:
@@
 Sheet 4 14
 Title "LittleSixteen"
-Date "2023-07-10"
+Date "2024-11-13"
 Rev "4git"
 Comp "SukkoPera"
@@
 Entry Wire Line
 	10680 4480 10580 4580
-Entry Wire Line
-	10680 4380 10580 4480
 Wire Wire Line
 	10135 4080 10315 4080
-Entry Wire Line
-	10680 4080 10580 4180
 Text Label 10580 4180 2    50   ~ 0
 a16
@@
 Text Label 3340 1855 2    50   ~ 0
 a17
-Text Label 3340 1955 2    50   ~ 0
-a18
+Text Label 3335 1955 2    50   ~ 0
+a18_from_pla
 Wire Wire Line
 	3045 2455 2840 2455
@@
 joyswap
 Wire Wire Line
-	3700 1790 3700 1690
-Wire Wire Line
-	3765 2355 3700 2355
-Wire Wire Line
-	3700 2355 3700 2455
+	4090 1790 4090 1690
+Wire Wire Line
+	4155 2355 4090 2355
+Wire Wire Line
+	4090 2355 4090 2455
 $Comp
 L power:GND #PWR?
 U 1 1 6616A4EF
-P 3700 2455
+P 4090 2455
 AR Path="/6616A4EF" Ref="#PWR?"  Part="1"
 AR Path="/62E48B71/6616A4EF" Ref="#PWR?"  Part="1"
@@
 AR Path="/5E4A465A/64E9FF4C/6616A4EF" Ref="#PWR?"  Part="1"
 AR Path="/5E4A465A/6616A4EF" Ref="#PWR0291"  Part="1"
-F 0 "#PWR0291" H 3700 2205 50  0001 C CNN
-F 1 "GND" H 3705 2282 50  0000 C CNN
-F 2 "" H 3700 2455 50  0001 C CNN
-F 3 "" H 3700 2455 50  0001 C CNN
-	1    3700 2455
+F 0 "#PWR0291" H 4090 2205 50  0001 C CNN
+F 1 "GND" H 4095 2282 50  0000 C CNN
+F 2 "" H 4090 2455 50  0001 C CNN
+F 3 "" H 4090 2455 50  0001 C CNN
+	1    4090 2455
 	1    0    0    -1
 $EndComp
@@
 d1
 Wire Wire Line
-	2840 2255 3700 2255
+	2840 2255 4090 2255
 $Comp
 L power:VCC #PWR?
@@
 L power:VCC #PWR?
 U 1 1 6630FA01
-P 3700 1690
+P 4090 1690
 AR Path="/5E6A379E/6630FA01" Ref="#PWR?"  Part="1"
 AR Path="/5E4A465A/6630FA01" Ref="#PWR0137"  Part="1"
-F 0 "#PWR0137" H 3700 1540 50  0001 C CNN
-F 1 "VCC" H 3717 1863 50  0000 C CNN
-F 2 "" H 3700 1690 50  0001 C CNN
-F 3 "" H 3700 1690 50  0001 C CNN
-	1    3700 1690
+F 0 "#PWR0137" H 4090 1540 50  0001 C CNN
+F 1 "VCC" H 4107 1863 50  0000 C CNN
+F 2 "" H 4090 1690 50  0001 C CNN
+F 3 "" H 4090 1690 50  0001 C CNN
+	1    4090 1690
 	1    0    0    -1
 $EndComp
@@
 Text Notes 7635 2560 0    50   ~ 0
 Another idea from Levente Hársfalvi in order to achieve the "high at reset"\nbehaviour of the MOS 6529 that was originally used in Hannes/Solder's\ndesign for the control register: keep the 74x573 in Hi-Z until the first write\nto $FD16 and use pull-ups on its output. All hail TLC!
-Text Notes 11095 1105 2    118  ~ 0
-- WE USE A SINGLE STATIC RAM CHIP\n- WE SUPPORT A HANNES-STYLE MECHANISM\n  FOR RAM EXPANSION TO UP TO 512 KB
+Text Notes 11100 1455 2    118  ~ 0
+- WE USE A SINGLE STATIC RAM CHIP\n- WE SUPPORT A HANNES-STYLE MECHANISM\n  FOR RAM EXPANSION TO UP TO 512 KB\n- WE PROVIDE A SWITCH TO LIMIT THE RAM\n  TO 256 KB FOR COMPATIBLITY
 $Comp
 L Device:R R?
 U 1 1 65A92B25
-P 3700 1940
+P 4090 1940
 AR Path="/5E019FCB/65A92B25" Ref="R?"  Part="1"
 AR Path="/5E4A465A/65A92B25" Ref="R97"  Part="1"
-F 0 "R97" H 3630 1894 50  0000 R CNN
-F 1 "10k" H 3630 1985 50  0000 R CNN
-F 2 "Resistor_THT:R_Axial_DIN0207_L6.3mm_D2.5mm_P5.08mm_Vertical" V 3630 1940 50  0001 C CNN
-F 3 "~" H 3700 1940 50  0001 C CNN
-F 4 "603-MFR-25FTF52-10K" H 3700 1940 50  0001 C CNN "MouserPN"
-	1    3700 1940
+F 0 "R97" H 4020 1894 50  0000 R CNN
+F 1 "10k" H 4020 1985 50  0000 R CNN
+F 2 "Resistor_THT:R_Axial_DIN0207_L6.3mm_D2.5mm_P5.08mm_Vertical" V 4020 1940 50  0001 C CNN
+F 3 "~" H 4090 1940 50  0001 C CNN
+F 4 "603-MFR-25FTF52-10K" H 4090 1940 50  0001 C CNN "MouserPN"
+	1    4090 1940
 	-1   0    0    1
 $EndComp
@@
 L Connector:Conn_01x02_Male CN?
 U 1 1 65AA1AF3
-P 3965 2355
+P 4355 2355
 AR Path="/64A6E6F3/65AA1AF3" Ref="CN?"  Part="1"
 AR Path="/5E4A465A/65AA1AF3" Ref="JP17"  Part="1"
-F 0 "JP17" H 3937 2237 50  0000 R CNN
-F 1 "SW_JOYSWAP" H 3937 2328 50  0000 R CNN
-F 2 "Connector_PinHeader_2.54mm:PinHeader_1x02_P2.54mm_Vertical" H 3965 2355 50  0001 C CNN
-F 3 "~" H 3965 2355 50  0001 C CNN
-	1    3965 2355
+F 0 "JP17" H 4530 2415 50  0000 R CNN
+F 1 "SW_JOYSWAP" H 4535 2495 50  0000 R CNN
+F 2 "Connector_PinHeader_2.54mm:PinHeader_1x02_P2.54mm_Vertical" H 4355 2355 50  0001 C CNN
+F 3 "~" H 4355 2355 50  0001 C CNN
+	1    4355 2355
 	-1   0    0    1
 $EndComp
 Wire Wire Line
-	3700 2090 3700 2255
-Connection ~ 3700 2255
-Wire Wire Line
-	3700 2255 3765 2255
+	4090 2090 4090 2255
+Connection ~ 4090 2255
+Wire Wire Line
+	4090 2255 4155 2255
+$Comp
+L Jumper:Jumper_3_Bridged12 JP?
+U 1 1 6758122B
+P 3590 1955
+AR Path="/5EE476E1/6758122B" Ref="JP?"  Part="1"
+AR Path="/5E4A465A/6758122B" Ref="JP4"  Part="1"
+F 0 "JP4" H 3590 1650 50  0000 C CNN
+F 1 "SW_RAMSIZE" H 3590 1565 50  0000 C CNN
+F 2 "Connector_PinHeader_2.54mm:PinHeader_1x03_P2.54mm_Vertical" H 3590 1955 50  0001 C CNN
+F 3 "~" H 3590 1955 50  0001 C CNN
+F 4 "---" H 3590 1955 50  0001 C CNN "MouserPN"
+	1    3590 1955
+	1    0    0    1
+$EndComp
+Wire Wire Line
+	3590 1805 3590 1755
+Wire Wire Line
+	3590 1755 3790 1755
+Wire Wire Line
+	3840 1955 3910 1955
+Wire Wire Line
+	3910 1955 3910 2055
+$Comp
+L power:GND #PWR?
+U 1 1 675B33AC
+P 3910 2055
+AR Path="/675B33AC" Ref="#PWR?"  Part="1"
+AR Path="/62E48B71/675B33AC" Ref="#PWR?"  Part="1"
+AR Path="/63A22C28/675B33AC" Ref="#PWR?"  Part="1"
+AR Path="/5E4A465A/64E9FF4C/675B33AC" Ref="#PWR?"  Part="1"
+AR Path="/5E4A465A/675B33AC" Ref="#PWR039"  Part="1"
+F 0 "#PWR039" H 3910 1805 50  0001 C CNN
+F 1 "GND" H 3910 1900 50  0000 C CNN
+F 2 "" H 3910 2055 50  0001 C CNN
+F 3 "" H 3910 2055 50  0001 C CNN
+	1    3910 2055
+	-1   0    0    -1
+$EndComp
+Text Label 3790 1755 2    50   ~ 0
+a18
+Text Notes 3410 1920 0    50   ~ 0
+512\nkB
+Text Notes 3875 1920 2    50   ~ 0
+256\nkB
 Wire Bus Line
 	8090 5180 8090 6210
@@
 	1240 2255 1240 2655
 Wire Bus Line
+	10680 3435 10680 4880
+Wire Bus Line
 	10680 5080 10680 6210
 Wire Bus Line
-	10680 3435 10680 4880
-Wire Bus Line
 	3655 4770 3655 5470
