File: userport.sch (KiCad schematic (older format))
At the start: 25 parts, among them CN10 USERPORT, U122 74LS654, U21 74LS04, U22 MOS_6529, U23 MOS_6551_ACIA, U28 GAL16V8, Y2 1.8432M

Commit message: WIP
Parts:
- U21: footprint Package_DIP:DIP-14_W7.62mm_Socket_LongPads -> LittleSixteen:DIP-14_W7.62mm_Socket_LongPads
- U22, U28: footprint Package_DIP:DIP-20_W7.62mm_Socket_LongPads -> LittleSixteen:DIP-20_W7.62mm_Socket_LongPads
- U23: footprint Package_DIP:DIP-28_W15.24mm_Socket_LongPads -> LittleSixteen:DIP-28_W15.24mm_Socket_LongPads
Changed lines of the file:
@@
 F 0 "U22" H 12650 2615 50  0000 C CNN
 F 1 "MOS_6529" H 12650 2524 50  0000 C CNN
-F 2 "Package_DIP:DIP-20_W7.62mm_Socket_LongPads" H 12650 1800 50  0001 C CNN
+F 2 "LittleSixteen:DIP-20_W7.62mm_Socket_LongPads" H 12650 1800 50  0001 C CNN
 F 3 "DOCUMENTATION" H 12650 1800 50  0001 C CNN
 	1    12650 1800
@@
 F 0 "U23" H 4490 3990 50  0000 C CNN
 F 1 "MOS_6551_ACIA" H 4490 3899 50  0000 C CNN
-F 2 "Package_DIP:DIP-28_W15.24mm_Socket_LongPads" H 4490 2975 50  0001 C CNN
+F 2 "LittleSixteen:DIP-28_W15.24mm_Socket_LongPads" H 4490 2975 50  0001 C CNN
 F 3 "DOCUMENTATION" H 4490 2975 50  0001 C CNN
 	1    4490 2975
@@
 F 0 "U22" H 1703 10086 50  0000 L CNN
 F 1 "MOS_6529" H 1703 9995 50  0000 L CNN
-F 2 "Package_DIP:DIP-20_W7.62mm_Socket_LongPads" H 1435 10040 50  0001 C CNN
+F 2 "LittleSixteen:DIP-20_W7.62mm_Socket_LongPads" H 1435 10040 50  0001 C CNN
 F 3 "DOCUMENTATION" H 1435 10040 50  0001 C CNN
 	2    1435 10040
@@
 F 0 "U21" H 8690 3062 50  0000 C CNN
 F 1 "74LS04" H 8690 2971 50  0000 C CNN
-F 2 "Package_DIP:DIP-14_W7.62mm_Socket_LongPads" H 8690 2745 50  0001 C CNN
+F 2 "LittleSixteen:DIP-14_W7.62mm_Socket_LongPads" H 8690 2745 50  0001 C CNN
 F 3 "http://www.ti.com/lit/gpn/sn74LS04" H 8690 2745 50  0001 C CNN
 	1    8690 2745
@@
 F 0 "U21" H 8690 2565 50  0000 C CNN
 F 1 "74LS04" H 8690 2566 50  0001 C CNN
-F 2 "Package_DIP:DIP-14_W7.62mm_Socket_LongPads" H 8690 2340 50  0001 C CNN
+F 2 "LittleSixteen:DIP-14_W7.62mm_Socket_LongPads" H 8690 2340 50  0001 C CNN
 F 3 "http://www.ti.com/lit/gpn/sn74LS04" H 8690 2340 50  0001 C CNN
 	2    8690 2340
@@
 F 0 "U21" H 8690 3435 50  0000 C CNN
 F 1 "74LS04" H 8690 3436 50  0001 C CNN
-F 2 "Package_DIP:DIP-14_W7.62mm_Socket_LongPads" H 8690 3210 50  0001 C CNN
+F 2 "LittleSixteen:DIP-14_W7.62mm_Socket_LongPads" H 8690 3210 50  0001 C CNN
 F 3 "http://www.ti.com/lit/gpn/sn74LS04" H 8690 3210 50  0001 C CNN
 	3    8690 3210
@@
 F 0 "U21" H 8690 3880 50  0000 C CNN
 F 1 "74LS04" H 8690 3881 50  0001 C CNN
-F 2 "Package_DIP:DIP-14_W7.62mm_Socket_LongPads" H 8690 3655 50  0001 C CNN
+F 2 "LittleSixteen:DIP-14_W7.62mm_Socket_LongPads" H 8690 3655 50  0001 C CNN
 F 3 "http://www.ti.com/lit/gpn/sn74LS04" H 8690 3655 50  0001 C CNN
 	4    8690 3655
@@
 F 0 "U21" H 11070 11087 50  0000 C CNN
 F 1 "74LS04" H 11070 10996 50  0000 C CNN
-F 2 "Package_DIP:DIP-14_W7.62mm_Socket_LongPads" H 11070 10770 50  0001 C CNN
+F 2 "LittleSixteen:DIP-14_W7.62mm_Socket_LongPads" H 11070 10770 50  0001 C CNN
 F 3 "http://www.ti.com/lit/gpn/sn74LS04" H 11070 10770 50  0001 C CNN
 	5    11070 10770
@@
 F 0 "U21" H 3205 10066 50  0000 L CNN
 F 1 "74LS04" H 3205 9975 50  0000 L CNN
-F 2 "Package_DIP:DIP-14_W7.62mm_Socket_LongPads" H 2975 10020 50  0001 C CNN
+F 2 "LittleSixteen:DIP-14_W7.62mm_Socket_LongPads" H 2975 10020 50  0001 C CNN
 F 3 "http://www.ti.com/lit/gpn/sn74LS04" H 2975 10020 50  0001 C CNN
 	7    2975 10020
@@
 F 0 "U28" H 3060 7395 50  0000 C CNN
 F 1 "GAL16V8" H 2985 6190 50  0000 C CNN
-F 2 "Package_DIP:DIP-20_W7.62mm_Socket_LongPads" H 2795 6795 50  0001 C CNN
+F 2 "LittleSixteen:DIP-20_W7.62mm_Socket_LongPads" H 2795 6795 50  0001 C CNN
 F 3 "" H 2795 6795 50  0001 C CNN
 F 4 "556-AF16V8B15PU" H 2795 6795 50  0001 C CNN "MouserPN"

Commit message: SID Power is almost there
Connections:
- no-connect marks 0 -> 2
Changed lines of the file:
@@
 Text Notes 4755 6680 0    50   ~ 0
 512KB RAM EXPANSION\nCONTROL SIGNALS
+NoConn ~ 10770 10770
+NoConn ~ 11370 10770
 Wire Bus Line
 	9765 6730 9765 8260
