File: sid.sch (KiCad schematic (older format))
At the start: 41 parts, among them CN11 CONN_SID_OUTPUT, CN12 CONN_SID_INPUT, J1 CONN_JOY3, Q6 2SC1815, SW2 SW_DIGIFIX, U21 74LS04, U24 MOS_8580, U25 74LS74, U26 GAL16V8, U27 74HCT245

Commit message: Routing in progress
Connections:
- net down: now also RN3.4 (R2.2); no longer RN3.3 (R2.1)
- net left: now also RN3.7 (R4.1); no longer RN3.6 (R3.2)
- net right: now also RN3.2 (R1.2); no longer RN3.7 (R4.1)
- net up: now also RN3.6 (R3.2); no longer RN3.1 (R1.1)
- net at RN2.2 (R1), U27.2 (A0): now also RN3.5 (R3.1); no longer RN3.2 (R1.2)
- net at RN2.3 (R2), U27.3 (A1): now also RN3.3 (R2.1); no longer RN3.4 (R2.2)
- net at RN2.4 (R3), U27.4 (A2): now also RN3.8 (R4.2); no longer RN3.5 (R3.1)
- net at RN2.5 (R4), U27.5 (A3): now also RN3.1 (R1.1); no longer RN3.8 (R4.2)
Other:
- moved on the sheet: RN3A, RN3C, RN3D
Changed lines of the file:
@@
 L Device:R_Pack05_SIP_Split RN3
 U 4 1 63A29AC0
-P 11920 6755
-F 0 "RN3" V 11880 7020 50  0000 C CNN
-F 1 "100" H 12008 6710 50  0001 L CNN
-F 2 "Resistor_THT:R_Array_SIP10" V 11840 6755 50  0001 C CNN
-F 3 "http://www.vishay.com/docs/31509/csc.pdf" H 11920 6755 50  0001 C CNN
-F 4 "652-4610X-2LF-100" H 11920 6755 50  0001 C CNN "MouserPN"
-F 5 "100" H 11920 6755 50  0001 C CNN "Value"
-	4    11920 6755
-	0    1    1    0
+P 10620 6755
+F 0 "RN3" V 10580 7020 50  0000 C CNN
+F 1 "100" H 10708 6710 50  0001 L CNN
+F 2 "Resistor_THT:R_Array_SIP10" V 10540 6755 50  0001 C CNN
+F 3 "http://www.vishay.com/docs/31509/csc.pdf" H 10620 6755 50  0001 C CNN
+F 4 "652-4610X-2LF-100" H 10620 6755 50  0001 C CNN "MouserPN"
+F 5 "100" H 10620 6755 50  0001 C CNN "Value"
+	4    10620 6755
+	0    -1   -1   0
 $EndComp
 $Comp
@@
 U 5 1 63A26FF8
 P 11920 6855
-F 0 "RN3" V 11880 7120 50  0000 C CNN
+F 0 "RN3" V 11880 7115 50  0000 C CNN
 F 1 "100" V 12030 6855 50  0000 C CNN
 F 2 "Resistor_THT:R_Array_SIP10" V 11840 6855 50  0001 C CNN
@@
 L Device:R_Pack05_SIP_Split RN3
 U 3 1 63A27F03
-P 10620 6755
-F 0 "RN3" V 10753 6755 50  0000 C CNN
-F 1 "100" V 10504 6755 50  0001 C CNN
-F 2 "Resistor_THT:R_Array_SIP10" V 10540 6755 50  0001 C CNN
-F 3 "http://www.vishay.com/docs/31509/csc.pdf" H 10620 6755 50  0001 C CNN
-F 4 "652-4610X-2LF-100" H 10620 6755 50  0001 C CNN "MouserPN"
-F 5 "100" H 10620 6755 50  0001 C CNN "Value"
-	3    10620 6755
+P 10620 6655
+F 0 "RN3" V 10505 6655 50  0000 C CNN
+F 1 "100" V 10504 6655 50  0001 C CNN
+F 2 "Resistor_THT:R_Array_SIP10" V 10540 6655 50  0001 C CNN
+F 3 "http://www.vishay.com/docs/31509/csc.pdf" H 10620 6655 50  0001 C CNN
+F 4 "652-4610X-2LF-100" H 10620 6655 50  0001 C CNN "MouserPN"
+F 5 "100" H 10620 6655 50  0001 C CNN "Value"
+	3    10620 6655
 	0    1    1    0
 $EndComp
@@
 U 2 1 63A28C60
 P 11920 6655
-F 0 "RN3" V 11880 6920 50  0000 C CNN
+F 0 "RN3" V 11880 6395 50  0000 C CNN
 F 1 "100" V 11804 6655 50  0001 C CNN
 F 2 "Resistor_THT:R_Array_SIP10" V 11840 6655 50  0001 C CNN
@@
 F 5 "100" H 11920 6655 50  0001 C CNN "Value"
 	2    11920 6655
-	0    1    1    0
+	0    -1   1    0
 $EndComp
 $Comp
 L Device:R_Pack05_SIP_Split RN3
 U 1 1 63A2AA82
-P 10620 6655
-F 0 "RN3" V 10753 6655 50  0000 C CNN
-F 1 "100" H 10708 6610 50  0001 L CNN
-F 2 "Resistor_THT:R_Array_SIP10" V 10540 6655 50  0001 C CNN
-F 3 "http://www.vishay.com/docs/31509/csc.pdf" H 10620 6655 50  0001 C CNN
-F 4 "652-4610X-2LF-100" H 10620 6655 50  0001 C CNN "MouserPN"
-F 5 "100" H 10620 6655 50  0001 C CNN "Value"
-	1    10620 6655
+P 11920 6755
+F 0 "RN3" V 11955 6495 50  0000 C CNN
+F 1 "100" H 12008 6710 50  0001 L CNN
+F 2 "Resistor_THT:R_Array_SIP10" V 11840 6755 50  0001 C CNN
+F 3 "http://www.vishay.com/docs/31509/csc.pdf" H 11920 6755 50  0001 C CNN
+F 4 "652-4610X-2LF-100" H 11920 6755 50  0001 C CNN "MouserPN"
+F 5 "100" H 11920 6755 50  0001 C CNN "Value"
+	1    11920 6755
 	0    -1   -1   0
 $EndComp
@@
 	7135 2495 7135 2895
 Wire Bus Line
+	9620 2095 9620 2795
+Wire Bus Line
+	15380 6155 15380 6855
+Wire Bus Line
 	6450 5890 6450 6845
-Wire Bus Line
-	15380 6155 15380 6855
-Wire Bus Line
-	9620 2095 9620 2795
 $EndSCHEMATC

Commit message: WIP
Connections:
- net at RN3.5 (R3.1), U27.2 (A0): now also RN2.5 (R4); no longer RN2.2 (R1)
- net at RN3.8 (R4.2), U27.4 (A2): now also RN2.8 (R7); no longer RN2.4 (R3)
- net at RN3.1 (R1.1), U27.5 (A3): now also RN2.2 (R1); no longer RN2.5 (R4)
- net at RN3.10 (R5.2), U27.6 (A4): now also RN2.9 (R8); no longer RN2.6 (R5)
- net at U27.7 (A5): now also RN2.4 (R3); no longer RN2.9 (R8)
- net at U27.8 (A6): now also RN2.6 (R5); no longer RN2.8 (R7)
Changed lines of the file:
@@
 	15590 7135 15590 7035
 Wire Wire Line
-	13875 6255 12590 6255
-Wire Wire Line
 	13875 6355 12690 6355
 Wire Wire Line
-	13875 6455 12790 6455
+	13875 6455 13190 6455
 Wire Wire Line
 	11050 6855 10800 6855
@@
 	9245 2095 9520 2095
 Wire Wire Line
-	12590 6085 12590 6255
-Connection ~ 12590 6255
-Wire Wire Line
-	12690 6355 12690 6085
-Wire Wire Line
-	12790 6085 12790 6455
-Connection ~ 12790 6455
-Wire Wire Line
-	13875 6655 12990 6655
-Wire Wire Line
-	12990 6085 12990 6655
-Connection ~ 12990 6655
-Wire Wire Line
-	13875 6555 12890 6555
-Wire Wire Line
-	12890 6555 12890 6085
+	13875 6655 13290 6655
 Wire Wire Line
 	1320 10315 1320 10410
@@
 	13090 6955 13875 6955
 Wire Wire Line
-	13190 6855 13190 6085
-Wire Wire Line
-	13190 6855 13875 6855
-Wire Wire Line
-	13290 6085 13290 6755
-Wire Wire Line
-	13290 6755 13875 6755
+	13290 6085 13290 6655
 Text GLabel 15580 6155 2    50   BiDi ~ 0
 d[0..7]
@@
 $EndComp
 Wire Wire Line
-	12590 6255 10355 6255
-Wire Wire Line
 	10355 6255 10355 6655
 Wire Wire Line
 	10355 6655 10470 6655
 Wire Wire Line
-	12790 6455 10255 6455
-Wire Wire Line
 	10255 6455 10255 6755
 Wire Wire Line
 	10255 6755 10470 6755
-Connection ~ 12690 6355
-Connection ~ 12890 6555
-Wire Wire Line
-	12990 6645 12990 6655
 Wire Wire Line
 	12990 6655 12990 6855
 Wire Wire Line
-	12890 6555 12890 6755
-Wire Wire Line
-	12070 6755 12890 6755
+	12070 6755 12590 6755
 Wire Wire Line
 	12070 6855 12990 6855
-Wire Wire Line
-	12690 6355 12690 6655
 Wire Wire Line
 	12070 6655 12690 6655
@@
 	1    0    0    -1
 $EndComp
+Wire Wire Line
+	12690 6085 12690 6355
+Connection ~ 12590 6755
+Wire Wire Line
+	12590 6755 12890 6755
+Wire Wire Line
+	10355 6255 12890 6255
+Wire Wire Line
+	12590 6085 12590 6755
+Connection ~ 12690 6355
+Wire Wire Line
+	12690 6355 12690 6655
+Wire Wire Line
+	12890 6085 12890 6255
+Connection ~ 12890 6255
+Wire Wire Line
+	12890 6255 13875 6255
+Wire Wire Line
+	13875 6555 12890 6555
+Wire Wire Line
+	12890 6555 12890 6755
+Connection ~ 13190 6455
+Wire Wire Line
+	13190 6455 13190 6085
+Wire Wire Line
+	10255 6455 13190 6455
+Connection ~ 13290 6655
+Wire Wire Line
+	13290 6655 12990 6655
+Wire Wire Line
+	12790 6085 12790 6705
+Wire Wire Line
+	12790 6705 13190 6705
+Wire Wire Line
+	13190 6705 13190 6755
+Wire Wire Line
+	13190 6755 13875 6755
+Wire Wire Line
+	12990 6085 12990 6605
+Wire Wire Line
+	12990 6605 13140 6605
+Wire Wire Line
+	13140 6605 13140 6855
+Wire Wire Line
+	13140 6855 13875 6855
 Wire Bus Line
 	8650 5890 8650 6745

Commit message: Well yeah maybe
Connections:
- no-connect marks 10 -> 12
Changed lines of the file:
@@
 Wire Wire Line
 	13140 6855 13875 6855
+NoConn ~ 8050 6345
+NoConn ~ 8050 6445
 Wire Bus Line
 	8650 5890 8650 6745
