File: sid.sch (KiCad schematic (older format))
At the start: 40 parts, among them CN11 CONN_SID_OUTPUT, CN12 CONN_SID_INPUT, CN14 CONN_JOY3, Q6 2SC1815, U21 74HCT04, U24 MOS_8580, U25 74LS74, U27 74HCT245

Commit message: Make C83 10uF
Parts:
- C52: MouserPN 710-860010672009 -> (none)
Changed lines of the file:
@@
 F 2 "Capacitor_THT:CP_Radial_D5.0mm_P2.00mm" H 14195 1800 50  0001 C CNN
 F 3 "~" H 14195 1800 50  0001 C CNN
-F 4 "710-860010672009" H 14195 1800 50  0001 C CNN "MouserPN"
+F 4 "" H 14195 1800 50  0001 C CNN "MouserPN"
 F 5 "10u" H 14195 1800 50  0001 C CNN "Value"
 F 6 "Audio cap recommended" H 14195 1800 50  0001 C CNN "Notes"
