File: sid.sch (KiCad schematic (older format))
At the start: 40 parts, among them CN11 CONN_SID_OUTPUT, CN12 CONN_SID_INPUT, CN14 CONN_JOY3, Q6 2SC1815, U21 74HCT04, U24 MOS_8580, U25 74LS74, U27 74HCT245

Commit message: VTED -> VSID, sigh...
Connections:
- net VTED renamed VSID
Changed lines of the file:
@@
 $EndComp
 $Comp
-L Power:VTED #PWR0258
+L Power:VSID #PWR0258
 U 1 1 64314574
 P 8965 1360
+AR Path="/64314574" Ref="#PWR0258"  Part="1"
+AR Path="/64A6E6F3/64314574" Ref="#PWR0258"  Part="1"
 F 0 "#PWR0258" H 8965 1210 50  0001 C CNN
-F 1 "VTED" H 8980 1533 50  0000 C CNN
+F 1 "VSID" H 8980 1533 50  0000 C CNN
 F 2 "" H 8965 1360 50  0001 C CNN
 F 3 "" H 8965 1360 50  0001 C CNN
@@
 $EndComp
 $Comp
-L Power:VTED #PWR0273
+L Power:VSID #PWR0273
 U 1 1 643169AD
 P 5860 4045
+AR Path="/643169AD" Ref="#PWR0273"  Part="1"
+AR Path="/64A6E6F3/643169AD" Ref="#PWR0273"  Part="1"
 F 0 "#PWR0273" H 5860 3895 50  0001 C CNN
-F 1 "VTED" H 5875 4218 50  0000 C CNN
+F 1 "VSID" H 5875 4218 50  0000 C CNN
 F 2 "" H 5860 4045 50  0001 C CNN
 F 3 "" H 5860 4045 50  0001 C CNN
@@
 $EndComp
 $Comp
-L Power:VTED #PWR0274
+L Power:VSID #PWR0274
 U 1 1 6432A2C4
 P 12830 830
+AR Path="/6432A2C4" Ref="#PWR0274"  Part="1"
+AR Path="/64A6E6F3/6432A2C4" Ref="#PWR0274"  Part="1"
 F 0 "#PWR0274" H 12830 680 50  0001 C CNN
-F 1 "VTED" H 12845 1003 50  0000 C CNN
+F 1 "VSID" H 12845 1003 50  0000 C CNN
 F 2 "" H 12830 830 50  0001 C CNN
 F 3 "" H 12830 830 50  0001 C CNN

Commit message: Fix all points from #15
Parts:
- R32: Notes For 6581 do not mount -> For 8580 do not mount
Changed lines of the file:
@@
 F 3 "~" H 10720 1775 50  0001 C CNN
 F 4 "603-MFR-25FBF52-1K" H 10720 1775 50  0001 C CNN "MouserPN"
-F 5 "For 6581 do not mount" H 10720 1775 50  0001 C CNN "Notes"
+F 5 "For 8580 do not mount" H 10720 1775 50  0001 C CNN "Notes"
 F 6 "1k" H 10720 1775 50  0001 C CNN "Value"
 	1    10720 1775

Commit message: Fix some P/Ns
Parts:
- U25: value 74LS74 -> 74HCT74; MouserPN (none) -> 595-SN74HC74N
- U27: MouserPN 595-SN74HCT245ANSR -> 595-SN74HCT245N
Changed lines of the file:
@@
 P 1625 9725
 F 0 "U25" H 1855 9771 50  0000 L CNN
-F 1 "74LS74" H 1855 9680 50  0000 L CNN
+F 1 "74HCT74" H 1855 9680 50  0000 L CNN
 F 2 "LittleSixteen:DIP-14_W7.62mm_Socket_LongPads" H 1625 9725 50  0001 C CNN
 F 3 "74xx/74hc_hct74.pdf" H 1625 9725 50  0001 C CNN
+F 4 "595-SN74HC74N" H 1625 9725 50  0001 C CNN "MouserPN"
 	3    1625 9725
 	1    0    0    -1
@@
 P 3215 6470
 F 0 "U25" H 3350 6730 50  0000 C CNN
-F 1 "74LS74" H 3395 6210 50  0000 C CNN
+F 1 "74HCT74" H 3395 6210 50  0000 C CNN
 F 2 "LittleSixteen:DIP-14_W7.62mm_Socket_LongPads" H 3215 6470 50  0001 C CNN
 F 3 "74xx/74hc_hct74.pdf" H 3215 6470 50  0001 C CNN
+F 4 "595-SN74HC74N" H 3215 6470 50  0001 C CNN "MouserPN"
 	1    3215 6470
 	1    0    0    -1
@@
 F 2 "LittleSixteen:DIP-20_W7.62mm_Socket_LongPads" H 14375 6755 50  0001 C CNN
 F 3 "http://www.ti.com/lit/gpn/sn74LS245" H 14375 6755 50  0001 C CNN
-F 4 "595-SN74HCT245ANSR" H 14375 6755 50  0001 C CNN "MouserPN"
+F 4 "595-SN74HCT245N" H 14375 6755 50  0001 C CNN "MouserPN"
 F 5 "74HCT245" H 14375 6755 50  0001 C CNN "Value"
 F 6 "Or 595-SN74HCT245NE4" H 14375 6755 50  0001 C CNN "Notes"

Commit message: R37 -> 220
Parts:
- R37: value 100 -> 220
Changed lines of the file:
@@
 Sheet 14 14
 Title "LittleSixteen"
-Date "2023-02-16"
+Date "2025-06-22"
 Rev "4git"
 Comp "SukkoPera"
@@
 P 3970 6370
 F 0 "R37" V 3763 6370 50  0000 C CNN
-F 1 "100" V 3854 6370 50  0000 C CNN
+F 1 "220" V 3854 6370 50  0000 C CNN
 F 2 "Resistor_THT:R_Axial_DIN0207_L6.3mm_D2.5mm_P5.08mm_Vertical" V 3900 6370 50  0001 C CNN
 F 3 "~" H 3970 6370 50  0001 C CNN

Commit message: Minor fixes + P/N updates
Parts:
- C52: MouserPN (none) -> 710-860010572002
- R37: MouserPN 708-RNF14FTD100R -> (none)
- U21: MouserPN (none) -> 595-SN74HCT04N
Changed lines of the file:
@@
 F 2 "Capacitor_THT:CP_Radial_D5.0mm_P2.00mm" H 14195 1800 50  0001 C CNN
 F 3 "~" H 14195 1800 50  0001 C CNN
-F 4 "" H 14195 1800 50  0001 C CNN "MouserPN"
+F 4 "710-860010572002" H 14195 1800 50  0001 C CNN "MouserPN"
 F 5 "10u" H 14195 1800 50  0001 C CNN "Value"
 F 6 "Audio cap recommended" H 14195 1800 50  0001 C CNN "Notes"
@@
 F 2 "Resistor_THT:R_Axial_DIN0207_L6.3mm_D2.5mm_P5.08mm_Vertical" V 3900 6370 50  0001 C CNN
 F 3 "~" H 3970 6370 50  0001 C CNN
-F 4 "708-RNF14FTD100R" H 3970 6370 50  0001 C CNN "MouserPN"
+F 4 "" H 3970 6370 50  0001 C CNN "MouserPN"
 F 5 "" H 3970 6370 50  0001 C CNN "Notes"
 F 6 "100" H 3970 6370 50  0001 C CNN "Value"
@@
 F 2 "LittleSixteen:DIP-14_W7.62mm_Socket_LongPads" H 1765 6470 50  0001 C CNN
 F 3 "http://www.ti.com/lit/gpn/sn74LS04" H 1765 6470 50  0001 C CNN
+F 4 "595-SN74HCT04N" H 1765 6470 50  0001 C CNN "MouserPN"
 	6    1765 6470
 	1    0    0    -1
