File: keyboard.sch (KiCad schematic (older format))
At the start: 28 parts, among them CN2 KEYBOARD_HEADER, U13 MOS_6529, U20 74HCT273

Commit message: Add 512kB RAM expansions, Hannes-style
Connections:
- net D1_LATCHED: no longer names the net of D71.2 (A), FB42.1, U13.3 (P1)
- net D2_LATCHED: no longer names the net of D72.2 (A), FB43.1, U13.4 (P2)
Changed lines of the file:
@@
 Wire Wire Line
 	5830 2215 6005 2215
-Wire Wire Line
-	6005 2215 6005 830
-Wire Wire Line
-	6005 830  6800 830
 Connection ~ 6005 2215
 Wire Wire Line
 	6005 2215 7965 2215
-Text GLabel 6800 945  2    50   Output ~ 0
-D2_LATCHED
-Text GLabel 6800 830  2    50   Output ~ 0
-D1_LATCHED
 Connection ~ 4275 1775
 Wire Wire Line
@@
 	5915 2115 7590 2115
 Wire Wire Line
-	6085 2315 6085 945
-Wire Wire Line
-	6085 945  6800 945
-Wire Wire Line
 	6085 2315 6085 3435

Commit message: Rationalize BOM There should be no significant changes on both schematics on PCB, just some values and something on the silkscreen
Parts:
- C33: MouserPN (none) -> 810-FG28X7R1H104KNT0
- FB41, FB42, FB43, FB44, FB45, FB46, FB47, FB48, FB49, FB50, FB51, FB52, FB53, FB54, FB55, FB56: value Ferrite_Bead_Small -> DSS1NB32A271Q91A; footprint LittleSixteen:Ferrite -> LittleSixteen:EMI_Filter; symbol ferrite_bead_small:Ferrite_Bead_Small -> emi_filter_3pin:EMI_Filter_3Pin
Changed lines of the file:
@@
 F 2 "Capacitor_THT:C_Disc_D8.0mm_W2.5mm_P5.00mm" H 1978 6420 50  0001 C CNN
 F 3 "~" H 1940 6570 50  0001 C CNN
+F 4 "810-FG28X7R1H104KNT0" H 1940 6570 50  0001 C CNN "MouserPN"
 	1    1940 6570
 	1    0    0    -1
@@
 	8235 2315 8730 2315
 $Comp
-L ferrite_bead_small:Ferrite_Bead_Small FB46
+L emi_filter_3pin:EMI_Filter_3Pin FB46
 U 1 1 5E275829
 P 8810 1515
 F 0 "FB46" V 8665 1515 50  0000 C CNN
-F 1 "Ferrite_Bead_Small" V 8664 1515 50  0001 C CNN
-F 2 "LittleSixteen:Ferrite" V 8740 1515 50  0001 C CNN
+F 1 "DSS1NB32A271Q91A" V 8664 1515 50  0001 C CNN
+F 2 "LittleSixteen:EMI_Filter" V 8740 1515 50  0001 C CNN
 F 3 "~" H 8810 1515 50  0001 C CNN
 	1    8810 1515
@@
 	8910 1515 9420 1515
 $Comp
-L ferrite_bead_small:Ferrite_Bead_Small FB56
+L emi_filter_3pin:EMI_Filter_3Pin FB56
 U 1 1 5E277735
 P 8820 1715
 F 0 "FB56" V 8675 1715 50  0000 C CNN
-F 1 "Ferrite_Bead_Small" V 8674 1715 50  0001 C CNN
-F 2 "LittleSixteen:Ferrite" V 8750 1715 50  0001 C CNN
+F 1 "DSS1NB32A271Q91A" V 8674 1715 50  0001 C CNN
+F 2 "LittleSixteen:EMI_Filter" V 8750 1715 50  0001 C CNN
 F 3 "~" H 8820 1715 50  0001 C CNN
 	1    8820 1715
@@
 	9420 1915 9155 1915
 $Comp
-L ferrite_bead_small:Ferrite_Bead_Small FB53
+L emi_filter_3pin:EMI_Filter_3Pin FB53
 U 1 1 5E279505
 P 8820 2115
 F 0 "FB53" V 8675 2115 50  0000 C CNN
-F 1 "Ferrite_Bead_Small" V 8674 2115 50  0001 C CNN
-F 2 "LittleSixteen:Ferrite" V 8750 2115 50  0001 C CNN
+F 1 "DSS1NB32A271Q91A" V 8674 2115 50  0001 C CNN
+F 2 "LittleSixteen:EMI_Filter" V 8750 2115 50  0001 C CNN
 F 3 "~" H 8820 2115 50  0001 C CNN
 	1    8820 2115
@@
 	8920 2115 9420 2115
 $Comp
-L ferrite_bead_small:Ferrite_Bead_Small FB54
+L emi_filter_3pin:EMI_Filter_3Pin FB54
 U 1 1 5E27AC84
 P 8830 2315
 F 0 "FB54" V 8685 2315 50  0000 C CNN
-F 1 "Ferrite_Bead_Small" V 8684 2315 50  0001 C CNN
-F 2 "LittleSixteen:Ferrite" V 8760 2315 50  0001 C CNN
+F 1 "DSS1NB32A271Q91A" V 8684 2315 50  0001 C CNN
+F 2 "LittleSixteen:EMI_Filter" V 8760 2315 50  0001 C CNN
 F 3 "~" H 8830 2315 50  0001 C CNN
 	1    8830 2315
@@
 	8930 2315 9420 2315
 $Comp
-L ferrite_bead_small:Ferrite_Bead_Small FB44
+L emi_filter_3pin:EMI_Filter_3Pin FB44
 U 1 1 5E27B4EF
 P 8805 2515
 F 0 "FB44" V 8660 2515 50  0000 C CNN
-F 1 "Ferrite_Bead_Small" V 8659 2515 50  0001 C CNN
-F 2 "LittleSixteen:Ferrite" V 8735 2515 50  0001 C CNN
+F 1 "DSS1NB32A271Q91A" V 8659 2515 50  0001 C CNN
+F 2 "LittleSixteen:EMI_Filter" V 8735 2515 50  0001 C CNN
 F 3 "~" H 8805 2515 50  0001 C CNN
 	1    8805 2515
@@
 	8905 2515 9420 2515
 $Comp
-L ferrite_bead_small:Ferrite_Bead_Small FB45
+L emi_filter_3pin:EMI_Filter_3Pin FB45
 U 1 1 5E27BE11
 P 8805 2715
 F 0 "FB45" V 8660 2715 50  0000 C CNN
-F 1 "Ferrite_Bead_Small" V 8659 2715 50  0001 C CNN
-F 2 "LittleSixteen:Ferrite" V 8735 2715 50  0001 C CNN
+F 1 "DSS1NB32A271Q91A" V 8659 2715 50  0001 C CNN
+F 2 "LittleSixteen:EMI_Filter" V 8735 2715 50  0001 C CNN
 F 3 "~" H 8805 2715 50  0001 C CNN
 	1    8805 2715
@@
 	8905 2715 9420 2715
 $Comp
-L ferrite_bead_small:Ferrite_Bead_Small FB50
+L emi_filter_3pin:EMI_Filter_3Pin FB50
 U 1 1 5E27C5F0
 P 8815 2915
 F 0 "FB50" V 8670 2915 50  0000 C CNN
-F 1 "Ferrite_Bead_Small" V 8669 2915 50  0001 C CNN
-F 2 "LittleSixteen:Ferrite" V 8745 2915 50  0001 C CNN
+F 1 "DSS1NB32A271Q91A" V 8669 2915 50  0001 C CNN
+F 2 "LittleSixteen:EMI_Filter" V 8745 2915 50  0001 C CNN
 F 3 "~" H 8815 2915 50  0001 C CNN
 	1    8815 2915
@@
 	8915 2915 9420 2915
 $Comp
-L ferrite_bead_small:Ferrite_Bead_Small FB52
+L emi_filter_3pin:EMI_Filter_3Pin FB52
 U 1 1 5E27CC99
 P 8815 3115
 F 0 "FB52" V 8670 3115 50  0000 C CNN
-F 1 "Ferrite_Bead_Small" V 8669 3115 50  0001 C CNN
-F 2 "LittleSixteen:Ferrite" V 8745 3115 50  0001 C CNN
+F 1 "DSS1NB32A271Q91A" V 8669 3115 50  0001 C CNN
+F 2 "LittleSixteen:EMI_Filter" V 8745 3115 50  0001 C CNN
 F 3 "~" H 8815 3115 50  0001 C CNN
 	1    8815 3115
@@
 	8915 3115 9420 3115
 $Comp
-L ferrite_bead_small:Ferrite_Bead_Small FB41
+L emi_filter_3pin:EMI_Filter_3Pin FB41
 U 1 1 5E27D4CD
 P 8810 3315
 F 0 "FB41" V 8955 3315 50  0000 C CNN
-F 1 "Ferrite_Bead_Small" V 8664 3315 50  0001 C CNN
-F 2 "LittleSixteen:Ferrite" V 8740 3315 50  0001 C CNN
+F 1 "DSS1NB32A271Q91A" V 8664 3315 50  0001 C CNN
+F 2 "LittleSixteen:EMI_Filter" V 8740 3315 50  0001 C CNN
 F 3 "~" H 8810 3315 50  0001 C CNN
 	1    8810 3315
@@
 	8910 3315 9420 3315
 $Comp
-L ferrite_bead_small:Ferrite_Bead_Small FB48
+L emi_filter_3pin:EMI_Filter_3Pin FB48
 U 1 1 5E27E7DF
 P 9030 2015
 F 0 "FB48" V 8885 2015 50  0000 C CNN
-F 1 "Ferrite_Bead_Small" V 8884 2015 50  0001 C CNN
-F 2 "LittleSixteen:Ferrite" V 8960 2015 50  0001 C CNN
+F 1 "DSS1NB32A271Q91A" V 8884 2015 50  0001 C CNN
+F 2 "LittleSixteen:EMI_Filter" V 8960 2015 50  0001 C CNN
 F 3 "~" H 9030 2015 50  0001 C CNN
 	1    9030 2015
@@
 	9130 2015 9420 2015
 $Comp
-L ferrite_bead_small:Ferrite_Bead_Small FB42
+L emi_filter_3pin:EMI_Filter_3Pin FB42
 U 1 1 5E27ED7A
 P 9050 2215
 F 0 "FB42" V 8905 2215 50  0000 C CNN
-F 1 "Ferrite_Bead_Small" V 8904 2215 50  0001 C CNN
-F 2 "LittleSixteen:Ferrite" V 8980 2215 50  0001 C CNN
+F 1 "DSS1NB32A271Q91A" V 8904 2215 50  0001 C CNN
+F 2 "LittleSixteen:EMI_Filter" V 8980 2215 50  0001 C CNN
 F 3 "~" H 9050 2215 50  0001 C CNN
 	1    9050 2215
@@
 	9150 2215 9420 2215
 $Comp
-L ferrite_bead_small:Ferrite_Bead_Small FB55
+L emi_filter_3pin:EMI_Filter_3Pin FB55
 U 1 1 5E27F5BE
 P 9040 2415
 F 0 "FB55" V 8895 2415 50  0000 C CNN
-F 1 "Ferrite_Bead_Small" V 8894 2415 50  0001 C CNN
-F 2 "LittleSixteen:Ferrite" V 8970 2415 50  0001 C CNN
+F 1 "DSS1NB32A271Q91A" V 8894 2415 50  0001 C CNN
+F 2 "LittleSixteen:EMI_Filter" V 8970 2415 50  0001 C CNN
 F 3 "~" H 9040 2415 50  0001 C CNN
 	1    9040 2415
@@
 	9140 2415 9420 2415
 $Comp
-L ferrite_bead_small:Ferrite_Bead_Small FB43
+L emi_filter_3pin:EMI_Filter_3Pin FB43
 U 1 1 5E27FD6B
 P 9020 2615
 F 0 "FB43" V 8875 2615 50  0000 C CNN
-F 1 "Ferrite_Bead_Small" V 8874 2615 50  0001 C CNN
-F 2 "LittleSixteen:Ferrite" V 8950 2615 50  0001 C CNN
+F 1 "DSS1NB32A271Q91A" V 8874 2615 50  0001 C CNN
+F 2 "LittleSixteen:EMI_Filter" V 8950 2615 50  0001 C CNN
 F 3 "~" H 9020 2615 50  0001 C CNN
 	1    9020 2615
@@
 	9120 2615 9420 2615
 $Comp
-L ferrite_bead_small:Ferrite_Bead_Small FB51
+L emi_filter_3pin:EMI_Filter_3Pin FB51
 U 1 1 5E280D1A
 P 9045 2815
 F 0 "FB51" V 8900 2815 50  0000 C CNN
-F 1 "Ferrite_Bead_Small" V 8899 2815 50  0001 C CNN
-F 2 "LittleSixteen:Ferrite" V 8975 2815 50  0001 C CNN
+F 1 "DSS1NB32A271Q91A" V 8899 2815 50  0001 C CNN
+F 2 "LittleSixteen:EMI_Filter" V 8975 2815 50  0001 C CNN
 F 3 "~" H 9045 2815 50  0001 C CNN
 	1    9045 2815
@@
 	9145 2815 9420 2815
 $Comp
-L ferrite_bead_small:Ferrite_Bead_Small FB47
+L emi_filter_3pin:EMI_Filter_3Pin FB47
 U 1 1 5E281382
 P 9045 3015
 F 0 "FB47" V 8900 3015 50  0000 C CNN
-F 1 "Ferrite_Bead_Small" V 8899 3015 50  0001 C CNN
-F 2 "LittleSixteen:Ferrite" V 8975 3015 50  0001 C CNN
+F 1 "DSS1NB32A271Q91A" V 8899 3015 50  0001 C CNN
+F 2 "LittleSixteen:EMI_Filter" V 8975 3015 50  0001 C CNN
 F 3 "~" H 9045 3015 50  0001 C CNN
 	1    9045 3015
@@
 	9145 3015 9420 3015
 $Comp
-L ferrite_bead_small:Ferrite_Bead_Small FB49
+L emi_filter_3pin:EMI_Filter_3Pin FB49
 U 1 1 5E2818F5
 P 9030 3215
 F 0 "FB49" V 9150 3215 50  0000 C CNN
-F 1 "Ferrite_Bead_Small" V 8884 3215 50  0001 C CNN
-F 2 "LittleSixteen:Ferrite" V 8960 3215 50  0001 C CNN
+F 1 "DSS1NB32A271Q91A" V 8884 3215 50  0001 C CNN
+F 2 "LittleSixteen:EMI_Filter" V 8960 3215 50  0001 C CNN
 F 3 "~" H 9030 3215 50  0001 C CNN
 	1    9030 3215

Commit message: Rationalize capacitor footprints & BOM
Parts:
- U13: MouserPN (none) -> :)
Changed lines of the file:
@@
 F 2 "LittleSixteen:DIP-20_W7.62mm_Socket_LongPads" H 5080 2295 50  0001 C CNN
 F 3 "DOCUMENTATION" H 5080 2295 50  0001 C CNN
+F 4 ":)" H 5080 2295 50  0001 C CNN "MouserPN"
 	1    5080 2295
 	-1   0    0    -1
@@
 F 2 "LittleSixteen:DIP-20_W7.62mm_Socket_LongPads" H 1345 6580 50  0001 C CNN
 F 3 "DOCUMENTATION" H 1345 6580 50  0001 C CNN
+F 4 ":)" H 1345 6580 50  0001 C CNN "MouserPN"
 	2    1345 6580
 	1    0    0    -1

Commit message: Add keyboard power jumper and remove pin 2 from keyboard connector
Parts:
- added JP1: JMP_KBD_POWER, Jumper:SolderJumper-2_P1.3mm_Open_RoundedPad1.0x1.5mm, symbol Device:Jumper_NO_Small
- CN2: footprint Connector_PinHeader_2.54mm:PinHeader_1x20_P2.54mm_Vertical -> LittleSixteen:PinHeader_1x20_P2.54mm_NoPin2
Connections:
- net VCC: now also JP1.1
- net at CN2.5 (Pin_5): now also JP1.2
- no-connect marks 3 -> 2
Other:
- note added: "Male\nPin 2: Key (Missing)\nPin 5: NC on original board,\n optional power for\n MechBoard16 for us\nPin 20: NC"
- note removed: "Pin 2: Key (Missing)\nPins 5, 20: NC\nMale"
Changed lines of the file:
@@
 Sheet 6 14
 Title "LittleSixteen"
-Date "2022-08-17"
+Date "2024-02-05"
 Rev "4git"
 Comp "SukkoPera"
@@
 U 1 1 5DED69BA
 P 9620 2415
-F 0 "CN2" H 9728 3496 50  0000 C CNN
-F 1 "KEYBOARD_HEADER" H 9728 3405 50  0000 C CNN
-F 2 "Connector_PinHeader_2.54mm:PinHeader_1x20_P2.54mm_Vertical" H 9620 2415 50  0001 C CNN
+F 0 "CN2" H 9592 2389 50  0000 R CNN
+F 1 "KEYBOARD_HEADER" H 9592 2298 50  0000 R CNN
+F 2 "LittleSixteen:PinHeader_1x20_P2.54mm_NoPin2" H 9620 2415 50  0001 C CNN
 F 3 "~" H 9620 2415 50  0001 C CNN
 	1    9620 2415
@@
 Text Label 8485 2915 2    50   ~ 0
 k1
-Text Notes 9685 2535 0    50   ~ 0
-Pin 2: Key (Missing)\nPins 5, 20: NC\nMale
+Text Notes 9645 3055 0    50   ~ 0
+Male\nPin 2: Key (Missing)\nPin 5: NC on original board,\n       optional power for\n       MechBoard16 for us\nPin 20: NC
 Text Label 8485 3215 2    50   ~ 0
 k0
@@
 $EndComp
 Wire Wire Line
-	9420 1915 9155 1915
+	9420 1915 9185 1915
 $Comp
 L emi_filter_3pin:EMI_Filter_3Pin FB53
@@
 Wire Wire Line
 	8235 2015 8930 2015
-NoConn ~ 9155 1915
 NoConn ~ 9155 3415
 Wire Wire Line
@@
 Wire Wire Line
 	6520 4595 6520 3485
+$Comp
+L Device:Jumper_NO_Small JP1
+U 1 1 65C514B9
+P 9185 1120
+F 0 "JP1" V 9139 1168 50  0000 L CNN
+F 1 "JMP_KBD_POWER" V 9230 1168 50  0000 L CNN
+F 2 "Jumper:SolderJumper-2_P1.3mm_Open_RoundedPad1.0x1.5mm" H 9185 1120 50  0001 C CNN
+F 3 "~" H 9185 1120 50  0001 C CNN
+	1    9185 1120
+	0    1    1    0
+$EndComp
+Wire Wire Line
+	9185 1915 9185 1220
+$Comp
+L power:VCC #PWR024
+U 1 1 65C61E3F
+P 9185 925
+F 0 "#PWR024" H 9185 775 50  0001 C CNN
+F 1 "VCC" H 9202 1098 50  0000 C CNN
+F 2 "" H 9185 925 50  0001 C CNN
+F 3 "" H 9185 925 50  0001 C CNN
+	1    9185 925
+	1    0    0    -1
+$EndComp
+Wire Wire Line
+	9185 925  9185 1020
 Wire Bus Line
 	3090 2015 3090 2720
