File: keyboard.sch (KiCad schematic (older format))
At the start: 30 parts, among them CN2 KEYBOARD_HEADER, U13 MOS_6529, U20 74HCT273

Commit message: Minor fixes + P/N updates
Parts:
- JP1: MouserPN (none) -> ---
- U20: MouserPN (none) -> 595-CD74HCT273E
Changed lines of the file:
@@
 F 2 "LittleSixteen:DIP-20_W7.62mm_Socket_LongPads" H 5070 4795 50  0001 C CNN
 F 3 "https://assets.nexperia.com/documents/data-sheet/74HC_HCT273.pdf" H 5070 4795 50  0001 C CNN
+F 4 "595-CD74HCT273E" H 5070 4795 50  0001 C CNN "MouserPN"
 	1    5070 4795
 	1    0    0    -1
@@
 F 2 "Jumper:SolderJumper-2_P1.3mm_Open_RoundedPad1.0x1.5mm" H 9185 1120 50  0001 C CNN
 F 3 "~" H 9185 1120 50  0001 C CNN
+F 4 "---" H 9185 1120 50  0001 C CNN "MouserPN"
 	1    9185 1120
 	0    1    1    0
