File: pla.sch (KiCad schematic (older format))
At the start: 17 parts, among them U12 74HCT02, U14 74HCT139, U15 74LS175, U19 GAL16V8

Commit message: Rationalize BOM There should be no significant changes on both schematics on PCB, just some values and something on the silkscreen
Parts:
- C28, C30, C90, C91: MouserPN (none) -> 810-FG28X7R1H104KNT0
- R80: Notes Only mount if using PLA16V8 -> (none)
Changed lines of the file:
@@
 F 2 "Capacitor_THT:C_Disc_D8.0mm_W2.5mm_P5.00mm" H 9813 5330 50  0001 C CNN
 F 3 "~" H 9775 5480 50  0001 C CNN
+F 4 "810-FG28X7R1H104KNT0" H 9775 5480 50  0001 C CNN "MouserPN"
 	1    9775 5480
 	1    0    0    -1
@@
 F 2 "Capacitor_THT:C_Disc_D8.0mm_W2.5mm_P5.00mm" H 8028 5330 50  0001 C CNN
 F 3 "~" H 7990 5480 50  0001 C CNN
+F 4 "810-FG28X7R1H104KNT0" H 7990 5480 50  0001 C CNN "MouserPN"
 	1    7990 5480
 	1    0    0    -1
@@
 F 2 "Capacitor_THT:C_Disc_D8.0mm_W2.5mm_P5.00mm" H 10458 5330 50  0001 C CNN
 F 3 "~" H 10420 5480 50  0001 C CNN
+F 4 "810-FG28X7R1H104KNT0" H 10420 5480 50  0001 C CNN "MouserPN"
 	1    10420 5480
 	1    0    0    -1
@@
 F 2 "Resistor_THT:R_Axial_DIN0207_L6.3mm_D2.5mm_P5.08mm_Vertical" V 1640 4660 50  0001 C CNN
 F 3 "~" H 1710 4660 50  0001 C CNN
-F 4 "Only mount if using PLA16V8" H 1710 4660 50  0001 C CNN "Notes"
 	1    1710 4660
 	-1   0    0    1
@@
 F 2 "Capacitor_THT:C_Disc_D8.0mm_W2.5mm_P5.00mm" H 1858 6335 50  0001 C CNN
 F 3 "~" H 1820 6485 50  0001 C CNN
+F 4 "810-FG28X7R1H104KNT0" H 1820 6485 50  0001 C CNN "MouserPN"
 	1    1820 6485
 	1    0    0    -1

Commit message: Rationalize capacitor footprints & BOM
Parts:
- TP6, TP7: MouserPN (none) -> ---
- U12: MouserPN (none) -> 595-SN74HCT02N; Notes (none) -> Or 595-SN74HC02N, 595-SN74HCT02NE4
Changed lines of the file:
@@
 F 2 "LittleSixteen:DIP-14_W7.62mm_Socket_LongPads" H 7265 5485 50  0001 C CNN
 F 3 "http://www.ti.com/lit/gpn/sn74ls02" H 7265 5485 50  0001 C CNN
+F 4 "595-SN74HCT02N" H 7265 5485 50  0001 C CNN "MouserPN"
+F 5 "Or 595-SN74HC02N, 595-SN74HCT02NE4" H 7265 5485 50  0001 C CNN "Notes"
 	5    7265 5485
 	1    0    0    -1
@@
 F 2 "LittleSixteen:DIP-14_W7.62mm_Socket_LongPads" H 8105 2750 50  0001 C CNN
 F 3 "http://www.ti.com/lit/gpn/sn74ls02" H 8105 2750 50  0001 C CNN
+F 4 "595-SN74HCT02N" H 8105 2750 50  0001 C CNN "MouserPN"
+F 5 "Or 595-SN74HC02N, 595-SN74HCT02NE4" H 8105 2750 50  0001 C CNN "Notes"
 	3    8105 2750
 	1    0    0    -1
@@
 F 2 "LittleSixteen:DIP-14_W7.62mm_Socket_LongPads" H 8105 2050 50  0001 C CNN
 F 3 "http://www.ti.com/lit/gpn/sn74ls02" H 8105 2050 50  0001 C CNN
+F 4 "595-SN74HCT02N" H 8105 2050 50  0001 C CNN "MouserPN"
+F 5 "Or 595-SN74HC02N, 595-SN74HCT02NE4" H 8105 2050 50  0001 C CNN "Notes"
 	2    8105 2050
 	1    0    0    -1
@@
 F 2 "LittleSixteen:DIP-14_W7.62mm_Socket_LongPads" H 4660 1985 50  0001 C CNN
 F 3 "http://www.ti.com/lit/gpn/sn74ls02" H 4660 1985 50  0001 C CNN
+F 4 "595-SN74HCT02N" H 4660 1985 50  0001 C CNN "MouserPN"
+F 5 "Or 595-SN74HC02N, 595-SN74HCT02NE4" H 4660 1985 50  0001 C CNN "Notes"
 	1    4660 1985
 	1    0    0    -1
@@
 F 2 "TestPoint:TestPoint_Pad_D2.0mm" H 4635 6640 50  0001 C CNN
 F 3 "~" H 4635 6640 50  0001 C CNN
+F 4 "---" H 4435 6640 50  0001 C CNN "MouserPN"
 	1    4435 6640
 	-1   0    0    1
@@
 F 2 "TestPoint:TestPoint_Pad_D2.0mm" H 3175 6865 50  0001 C CNN
 F 3 "~" H 3175 6865 50  0001 C CNN
+F 4 "---" H 2975 6865 50  0001 C CNN "MouserPN"
 	1    2975 6865
 	-1   0    0    1

Commit message: Fix some P/Ns
Parts:
- U15: value 74LS175 -> 74HCT175; MouserPN (none) -> 595-CD74HCT175E
Changed lines of the file:
@@
 P 6165 1585
 F 0 "U15" H 6380 2135 50  0000 C CNN
-F 1 "74LS175" H 6435 930 50  0000 C CNN
+F 1 "74HCT175" H 6435 930 50  0000 C CNN
 F 2 "LittleSixteen:DIP-16_W7.62mm_Socket_LongPads" H 6165 1585 50  0001 C CNN
 F 3 "http://www.ti.com/lit/gpn/sn74LS175" H 6165 1585 50  0001 C CNN
+F 4 "595-CD74HCT175E" H 6165 1585 50  0001 C CNN "MouserPN"
 	1    6165 1585
 	1    0    0    -1
