File: cpu.sch (KiCad schematic (older format))
At the start: 5 parts, among them U102 MOS_6510, U2 MOS_8501

Commit message: Enlarge drill holes to 0.9mm in order to make it possible to use ZIF sockets
Parts:
- U102, U2: footprint Package_DIP:DIP-40_W15.24mm_Socket_LongPads -> LittleSixteen:DIP-40_W15.24mm_Socket_LongPads
Changed lines of the file:
@@
 F 0 "U2" H 3615 3780 50  0000 C CNN
 F 1 "MOS_8501" H 3615 3689 50  0000 C CNN
-F 2 "Package_DIP:DIP-40_W15.24mm_Socket_LongPads" H 3615 2465 50  0001 C CNN
+F 2 "LittleSixteen:DIP-40_W15.24mm_Socket_LongPads" H 3615 2465 50  0001 C CNN
 F 3 "DOCUMENTATION" H 3615 2465 50  0001 C CNN
 	1    3615 2465
@@
 F 0 "U102" H 3615 7145 50  0000 C CNN
 F 1 "MOS_6510" H 3615 7054 50  0000 C CNN
-F 2 "Package_DIP:DIP-40_W15.24mm_Socket_LongPads" H 3615 5830 50  0001 C CNN
+F 2 "LittleSixteen:DIP-40_W15.24mm_Socket_LongPads" H 3615 5830 50  0001 C CNN
 F 3 "DOCUMENTATION" H 3615 5830 50  0001 C CNN
 	1    3615 5830

Commit message: Rationalize BOM There should be no significant changes on both schematics on PCB, just some values and something on the silkscreen
Parts:
- C22: MouserPN (none) -> 810-FG28X7R1H104KNT0
Changed lines of the file:
@@
 F 2 "Capacitor_THT:C_Disc_D8.0mm_W2.5mm_P5.00mm" H 1558 6940 50  0001 C CNN
 F 3 "~" H 1520 7090 50  0001 C CNN
+F 4 "810-FG28X7R1H104KNT0" H 1520 7090 50  0001 C CNN "MouserPN"
 	1    1520 7090
 	1    0    0    -1

Commit message: Rationalize capacitor footprints & BOM
Parts:
- C4: footprint Capacitor_THT:CP_Radial_D6.3mm_P2.50mm -> Capacitor_THT:CP_Radial_D5.0mm_P2.00mm; MouserPN (none) -> 710-860010672009
- U102, U2: MouserPN (none) -> :)
Changed lines of the file:
@@
 F 2 "LittleSixteen:DIP-40_W15.24mm_Socket_LongPads" H 3615 2465 50  0001 C CNN
 F 3 "DOCUMENTATION" H 3615 2465 50  0001 C CNN
+F 4 ":)" H 3615 2465 50  0001 C CNN "MouserPN"
 	1    3615 2465
 	1    0    0    -1
@@
 F 0 "C4" H 911 7136 50  0000 R CNN
 F 1 "10u/25V" H 911 7045 50  0000 R CNN
-F 2 "Capacitor_THT:CP_Radial_D6.3mm_P2.50mm" H 1025 7090 50  0001 C CNN
+F 2 "Capacitor_THT:CP_Radial_D5.0mm_P2.00mm" H 1025 7090 50  0001 C CNN
 F 3 "~" H 1025 7090 50  0001 C CNN
+F 4 "710-860010672009" H 1025 7090 50  0001 C CNN "MouserPN"
 	1    1025 7090
 	1    0    0    -1
@@
 F 2 "LittleSixteen:DIP-40_W15.24mm_Socket_LongPads" H 3615 5830 50  0001 C CNN
 F 3 "DOCUMENTATION" H 3615 5830 50  0001 C CNN
+F 4 ":)" H 3615 5830 50  0001 C CNN "MouserPN"
 	1    3615 5830
 	1    0    0    -1

Commit message: Minor fixes + P/N updates
Parts:
- C4: MouserPN 710-860010672009 -> 710-860010572002
Changed lines of the file:
@@
 F 2 "Capacitor_THT:CP_Radial_D5.0mm_P2.00mm" H 1025 7090 50  0001 C CNN
 F 3 "~" H 1025 7090 50  0001 C CNN
-F 4 "710-860010672009" H 1025 7090 50  0001 C CNN "MouserPN"
+F 4 "710-860010572002" H 1025 7090 50  0001 C CNN "MouserPN"
 	1    1025 7090
 	1    0    0    -1
